File: 12V.kicad_sch (KiCad schematic)
At the start: 0 parts

Commit message: Added cap to output of lines
based on LTSpice Simulation
Parts:
- added C77: 0.1 uF, symbol Device:C
- added C79: 6.8nF, symbol Device:C
- added C91: 100pF, symbol Device:C
- added R76: 10k, symbol Device:R
- added R77: 15.4k, symbol Device:R
- added U20: LTC3786EMSE_PBF, LTC3786EMSE_PBF:MSOP-16_MSE, symbol LTC3786EMSE_PBF:LTC3786EMSE_PBF
Connections:
- new net: C77.2, C79.1, C91.1, U20.5 (SS)
- new net: C79.2, R77.1
- new net: C91.2, R77.2, U20.4 (ITH)
- new net +3.3V: R76.1
- new net GND: C77.1, U20.17 (EPAD), U20.9 (GND)
- new net INTVCC: U20.11 (INTVCC), U20.6 (PLLIN/MODE), U20.7 (FREQ)
- new net PGOOD 12V Line: R76.2, U20.16 (PGOOD)
- new net Sense+: U20.2 (SENSE+)
- new net Sense-: U20.3 (SENSE-)
Other:
- company: (none) -> QSET (Jaron Cyna)
