File: MPPT.kicad_sch (KiCad schematic)
At the start: 41 parts, among them Q1 NMOS, Q2 NMOS, Q4 NMOS, Q5 NMOS

Commit message: Added cap to output of lines
based on LTSpice Simulation
Other:
- company: (none) -> QSET (Jaron Cyna)
Changed lines of the file:
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@@
 	(generator_version "9.0")
 	(paper "A4")
+	(title_block
+		(company "QSET (Jaron Cyna)")
+	)
 	(rectangle
 		(start 22.86 163.83)
