File: MPPT_STM32.kicad_sch (KiCad schematic)
At the start: 26 parts, among them J1 Conn_01x04_Pin, J2 Conn_01x03_Pin, U1 STM32G474RETx, U8 TCAN334

Commit message: Added cap to output of lines
based on LTSpice Simulation
Other:
- company: (none) -> QSET (Jaron Cyna)
Changed lines of the file:
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@@
 	(generator_version "9.0")
 	(paper "A4")
+	(title_block
+		(company "QSET (Jaron Cyna)")
+	)
 	(rectangle
 		(start 233.68 113.03)
