File: MPPT_WatchDog.kicad_sch (KiCad schematic)
At the start: 9 parts, among them IC1 AP54RHC705ALT-R, U2 74HC00, U3 74HC00, U4 ICM7555xB

Commit message: Added cap to output of lines
based on LTSpice Simulation
Other:
- company: (none) -> QSET (Jaron Cyna)
Changed lines of the file:
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@@
 	(generator_version "9.0")
 	(paper "A4")
+	(title_block
+		(company "QSET (Jaron Cyna)")
+	)
 	(text_box "Notes for later: \n- Check all parts are 3.3V compatible\n- look at rad hardened and non rad hardened parts and pick, as currently I have both"
 		(exclude_from_sim no)
