File: EPS_mppt_board.kicad_sch (KiCad schematic)
At the start: 0 parts

Commit message: Added connectors to schematic
Other:
- sheet External Watchdog IC ports: added none; removed RESET_TIME_2
- sheet MPPT IC ports: added Thermistor_+X, Thermistor_+Y, Thermistor_-X, Thermistor_-Y; removed none
- sheet PC104 ports: added +X_Solar_IN, +Y_Solar_IN, -X_Solar_IN, -Y_Solar_IN; removed none
- sheet STM32L4 ports: added CRIT_IN, PV_IN, WAR_IN; removed RESET_TIME_2

Commit message: A bunch of misc schematic changes
Other:
- sheet MPPT IC ports: added MPPT_SYNC_1.5MHz; removed none
- sheet STM32L4 ports: added CAN_H2, CAN_L2, I2C_MUX_RESET, MPPT_SYNC; removed I2C_Mult_RESET
Changed lines of the file:
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@@
+	(wire
+		(pts
+			(xy 227.33 158.75) (xy 334.01 158.75)
+		)
+		(stroke
+			(width 0)
+			(type default)
+		)
+	)
 	(wire
 		(pts
@@
 		)
 		(pin "CAN_H" input
-			(at 179.07 156.21 180)
+			(at 179.07 167.64 180)
 			(effects
 				(font
@@
 		)
 		(pin "CAN_L" input
-			(at 179.07 158.75 180)
+			(at 179.07 170.18 180)
 			(effects
 				(font
@@
 			)
 		)
-		(pin "I2C_Mult_RESET" input
-			(at 227.33 143.51 0)
-			(effects
-				(font
-					(size 1.27 1.27)
-				)
-				(justify right)
-			)
-		)
 		(pin "ADCS_3V3_SD" output
 			(at 227.33 102.87 0)
@@
 		(pin "CRIT_IN" input
 			(at 218.44 175.26 270)
+			(effects
+				(font
+					(size 1.27 1.27)
+				)
+				(justify left)
+			)
+		)
+		(pin "I2C_MUX_RESET" input
+			(at 227.33 143.51 0)
+			(effects
+				(font
+					(size 1.27 1.27)
+				)
+				(justify right)
+			)
+		)
+		(pin "MPPT_SYNC" output
+			(at 227.33 158.75 0)
+			(effects
+				(font
+					(size 1.27 1.27)
+				)
+				(justify right)
+			)
+		)
+		(pin "CAN_H2" input
+			(at 179.07 158.75 180)
+			(effects
+				(font
+					(size 1.27 1.27)
+				)
+				(justify left)
+			)
+		)
+		(pin "CAN_L2" input
+			(at 179.07 161.29 180)
 			(effects
 				(font
@@
 			)
 		)
+		(pin "MPPT_SYNC_1.5MHz" input
+			(at 334.01 158.75 180)
+			(effects
+				(font
+					(size 1.27 1.27)
+				)
+				(justify left)
+			)
+		)
