File: MPPT_3.3V_logic.kicad_sch (KiCad schematic)
At the start: 41 parts, among them Q1 SIR5607DP-T1-RE3, Q2 SIR5607DP-T1-RE3, Q3 SIR5607DP-T1-RE3, Q4 SIR5607DP-T1-RE3, U1 LTC4417HUF, U2 TPS259470ARPWR, U3 TPS62177DQCR

Commit message: small changes
Parts:
- removed R3: 60.4k, Resistor_SMD:R_0603_1608Metric, symbol Device:R
- added C94: 6.8nF, Capacitor_SMD:C_0603_1608Metric, symbol Device:C
- added R106: 2.21k, Resistor_SMD:R_0603_1608Metric, symbol Device:R
- C4: value 1uF -> 100nF; MANUFACTURER_PART_NUMBER CL10B105KQ8NNNC -> 06035C104K4T2A
- C5: value 6.8nF -> 1uF; MANUFACTURER (none) -> DigiKey; MANUFACTURER_PART_NUMBER KAM15AR71H682JT -> CL10B105KQ8NNNC
- R10: value 2.21k -> 60.4k; MANUFACTURER_PART_NUMBER RMCF0603FT2K21 -> RT0603FRE0760K4L
Connections:
- net GND: now also C5.1, R2.2
- net OV1: now also R10.2, R2.1; no longer R2.2
- net Solar_+X: no longer U1.16 (VS2)
- net UV1: now also R10.1; no longer R2.1
- net at C6.1, C7.1, Q1.5 (D)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: now also C94.1; no longer C5.2
- net at Q3.1 (S), Q3.2 (S), Q3.3 (S)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: now also C5.2, U1.16 (VS2)
- net at Q3.4 (G), Q4.4 (G): now also D1.1 (K), C94.2, R106.2; no longer U1.15 (G2)
- new net: Q1.4 (G), Q2.4 (G), U1.17 (G1)
- new net: D1.2 (A), R106.1, U1.15 (G2)
Other:
- moved on the sheet: C3, D1, Q3, Q4, R2
