File: MPPT_3.3V_logic.kicad_sch (KiCad schematic)
At the start: 42 parts, among them Q1 SIR5607DP-T1-RE3, Q2 SIR5607DP-T1-RE3, Q3 SIR5607DP-T1-RE3, Q4 SIR5607DP-T1-RE3, U1 LTC4417HUF, U2 TPS259470ARPWR, U3 TPS62177DQCR

Commit message: Started PCB layout
Parts:
- renumbered C9 to C10, C10 to C11, C11 to C12, C12 to C13, C13 to C14, C14 to C15, C94 to C6, C6 to C7, C7 to C8, C8 to C9, R4 to R1, R106 to R10, R5 to R2, R6 to R3, R1 to R4, R10 to R5, R2 to R6
Other:
- moved on the sheet: Q4
