File: EPS_mppt_board.kicad_pcb (KiCad board)
At the start: 6 copper layers, 90 x 96 mm, 243 parts, among them J1 Conn_01x04_Pin, J2 ESQT-126-X-X-Q-X, J3 M80-5400642, J4 M80-5400642, J5 M80-5400642, J6 M80-5400642, Q10 NMOS, Q11 NMOS, Q12 NMOS, Q13 NMOS, Q14 NMOS, Q15 SIR5607DP-T1-RE3, Q16 SIR5607DP-T1-RE3, Q17 SIR5607DP-T1-RE3, Q4 NMOS, Q5 NMOS, Q6 NMOS, Q7 NMOS, Q8 NMOS, Q9 NMOS, U1 LTC4412xS6, U10 LTC4162IUFD-LADM_PBF, U11 MR20H40, U12 TCAN334, U13 TCA9548AMRGER, U15 INA3221, U16 TPS259470ARPWR, U17 TPS259470ARPWR, U18 TPS259470ARPWR, U19 LTC3633AIUFDPBF, U2 TPS259470ARPWR, U20 STM32L476RGTx, U3 TPS62177DQCR, U4 LTC4412xS6, U5 LTC2965HDD-PBF, U6 TPS3823A-33DBVR, U7 LTC4162IUFD-LADM_PBF, U8 LTC4162IUFD-LADM_PBF, U9 LTC4162IUFD-LADM_PBF, Y1 8 MHZ Oscillator

Commit message: A bunch of misc schematic changes
Parts:
- removed the C14 at (-22.0, 54.0)
- removed the C15 at (-22.0, 56.5)
- removed the C16 at (-47.5, 48.0)
- removed the C17 at (-22.0, 59.0)
- removed the C18 at (-22.0, 61.5)
- removed the C19 at (51.3, 66.1)
- removed the C20 at (-39.0, 49.2)
- removed the C21 at (-28.9, 48.6)
- removed the C22 at (-47.5, 53.1)
- removed the C23 at (-22.0, 64.0)
- removed the C24 at (-22.0, 66.5)
- removed the C25 at (-47.5, 58.2)
- removed the C26 at (-22.0, 69.0)
- removed the C27 at (-22.0, 71.5)
- removed the C28 at (51.3, 68.6)
- removed the C29 at (-39.0, 56.9)
- removed the C30 at (-28.9, 57.0)
- removed the C31 at (-47.5, 63.3)
- removed the C32 at (-18.0, 54.0)
- removed the C33 at (-18.0, 56.5)
- removed the C34 at (-47.5, 68.4)
- removed the C35 at (-18.0, 59.0)
- removed the C36 at (-18.0, 61.5)
- removed the C37 at (51.3, 71.1)
- removed the C38 at (-39.0, 64.5)
- removed the C39 at (-28.9, 64.7)
- removed the C40 at (-47.5, 73.5)
- removed the C41 at (-18.0, 64.0)
- removed the C42 at (-18.0, 66.5)
- removed the C43 at (-47.5, 78.7)
- removed the C44 at (-18.0, 69.0)
- removed the C45 at (-18.0, 71.5)
- removed the C46 at (51.3, 73.6)
- removed the C47 at (-39.0, 72.2)
- removed the C48 at (-28.9, 72.5)
- removed the C49 at (-47.5, 83.8)
- removed D1: D_Schottky, Diode_SMD:D_SOD-323F
- removed D10, D11, D12, D9: SMAJ22A, Diode_SMD:D_SMA
- removed the L2 at (53.3, 84.3)
- removed the L3 at (53.3, 93.4)
- removed the Q4 at (66.2, 71.3)
- removed the Q5 at (66.2, 78.0)
- removed the Q6 at (66.2, 84.7)
- removed the R12 at (-21.8, 79.9)
- removed the R13 at (-14.0, 54.0)
- removed the R14 at (-14.0, 56.5)
- removed the R15 at (-21.8, 82.8)
- removed the R16 at (-21.8, 75.6)
- removed the R17 at (-21.8, 85.8)
- removed the R18 at (-14.0, 59.0)
- removed the R19 at (-21.8, 88.7)
- removed the R20 at (-14.0, 61.5)
- removed the R21 at (-14.0, 64.0)
- removed the R22 at (-17.4, 79.9)
- removed the R23 at (-17.3, 75.6)
- removed the R24 at (-17.4, 82.8)
- removed the R25 at (-14.0, 66.5)
- removed the R26 at (-17.4, 85.8)
- removed the R27 at (-14.0, 69.0)
- removed the R28 at (-14.0, 71.5)
- removed the R29 at (-17.4, 88.7)
- removed the R30 at (-12.9, 75.6)
- removed the R31 at (-13.0, 79.9)
- removed the R32 at (-9.95, 54.0)
- removed the R33 at (-13.0, 82.8)
- removed the R34 at (-9.95, 56.5)
- removed the R35 at (-9.95, 59.0)
- removed the R36 at (-13.0, 85.8)
- removed the R37 at (-8.40, 75.6)
- removed the R38 at (-13.0, 88.7)
- removed the R39 at (-9.95, 61.5)
- removed the U10 at (-1.90, 49.1)
- removed U7: LTC4162IUFD-LADM_PBF, Package_DFN_QFN:QFN-28-1EP_4x5mm_P0.5mm_EP2.65x3.65mm_ThermalVias
- removed the U8 at (-14.5, 49.1)
- removed the U9 at (-8.21, 49.1)
- added C54: 1 uF, Capacitor_SMD:C_0603_1608Metric, F.Cu at (-66.7, 9.50)
- added C55: 4.7 uF, Capacitor_SMD:C_0603_1608Metric, F.Cu at (-66.7, 12.0)
- added C56: 10 uF, zLibrary:CAP_C1210C_X7R_2S_FW_KEM-M, F.Cu at (-60.8, 24.2)
- added C57: 100n, Capacitor_SMD:C_0603_1608Metric, F.Cu at (-66.7, 14.5)
- added C58: 100n, Capacitor_SMD:C_0603_1608Metric, F.Cu at (-66.7, 17.0)
- added C59: 22nF, Capacitor_SMD:C_0603_1608Metric, F.Cu at (-66.7, 19.5)
- added C60: 100uF, Capacitor_Tantalum_SMD:CP_EIA-7361-38_AVX-V, F.Cu at (-51.4, 28.9)
- added C61: 22 uF, zLibrary:CAP_C2220C_2S_KEM-M, F.Cu at (-51.0, 21.2)
- added C62: 10 uF, zLibrary:CAP_C1210C_X7R_2S_FW_KEM-M, F.Cu at (-60.8, 29.3)
- added C63: 1 uF, Capacitor_SMD:C_0603_1608Metric, F.Cu at (-36.2, 9.50)
- added C64: 4.7 uF, Capacitor_SMD:C_0603_1608Metric, F.Cu at (-36.2, 12.0)
- added C65: 10 uF, zLibrary:CAP_C1210C_X7R_2S_FW_KEM-M, F.Cu at (-30.3, 24.2)
- added C66: 100n, Capacitor_SMD:C_0603_1608Metric, F.Cu at (-36.2, 14.5)
- added C67: 100n, Capacitor_SMD:C_0603_1608Metric, F.Cu at (-36.2, 17.0)
- added C68: 22nF, Capacitor_SMD:C_0603_1608Metric, F.Cu at (-36.2, 19.5)
- added C69: 100uF, Capacitor_Tantalum_SMD:CP_EIA-7361-38_AVX-V, F.Cu at (-20.9, 28.9)
- added C70: 22 uF, zLibrary:CAP_C2220C_2S_KEM-M, F.Cu at (-20.5, 21.2)
- added C71: 10 uF, zLibrary:CAP_C1210C_X7R_2S_FW_KEM-M, F.Cu at (-30.3, 29.3)
- added C72: 1 uF, Capacitor_SMD:C_0603_1608Metric, F.Cu at (-66.7, 39.6)
- added C73: 4.7 uF, Capacitor_SMD:C_0603_1608Metric, F.Cu at (-66.7, 42.1)
- added C74: 10 uF, zLibrary:CAP_C1210C_X7R_2S_FW_KEM-M, F.Cu at (-60.8, 54.3)
- added C75: 100n, Capacitor_SMD:C_0603_1608Metric, F.Cu at (-66.7, 44.7)
- added C76: 100n, Capacitor_SMD:C_0603_1608Metric, F.Cu at (-66.7, 47.2)
- added C77: 22nF, Capacitor_SMD:C_0603_1608Metric, F.Cu at (-66.7, 49.7)
- added C78: 100uF, Capacitor_Tantalum_SMD:CP_EIA-7361-38_AVX-V, F.Cu at (-51.4, 59.0)
- added C79: 22 uF, zLibrary:CAP_C2220C_2S_KEM-M, F.Cu at (-51.0, 51.3)
- added C80: 10 uF, zLibrary:CAP_C1210C_X7R_2S_FW_KEM-M, F.Cu at (-60.8, 59.4)
- added C81: 1 uF, Capacitor_SMD:C_0603_1608Metric, F.Cu at (-36.2, 39.6)
- added C82: 4.7 uF, Capacitor_SMD:C_0603_1608Metric, F.Cu at (-36.2, 42.1)
- added C83: 10 uF, zLibrary:CAP_C1210C_X7R_2S_FW_KEM-M, F.Cu at (-30.3, 54.3)
- added C84: 100n, Capacitor_SMD:C_0603_1608Metric, F.Cu at (-36.2, 44.7)
- added C85: 100n, Capacitor_SMD:C_0603_1608Metric, F.Cu at (-36.2, 47.2)
- added C86: 22nF, Capacitor_SMD:C_0603_1608Metric, F.Cu at (-36.2, 49.7)
- added C87: 100uF, Capacitor_Tantalum_SMD:CP_EIA-7361-38_AVX-V, F.Cu at (-20.9, 59.0)
- added C88: 22 uF, zLibrary:CAP_C2220C_2S_KEM-M, F.Cu at (-20.5, 51.3)
- added C89: 10 uF, zLibrary:CAP_C1210C_X7R_2S_FW_KEM-M, F.Cu at (-30.3, 59.4)
- added C90: 100n, Capacitor_SMD:C_0603_1608Metric, F.Cu at (-4.76, 80.5)
- added D5: SMAJ22A, Diode_SMD:D_SMA, F.Cu at (-60.6, 34.1)
- added D6: SMAJ22A, Diode_SMD:D_SMA, F.Cu at (-30.1, 34.1)
- added D7: SMAJ22A, Diode_SMD:D_SMA, F.Cu at (-60.6, 64.2)
- added D8: SMAJ22A, Diode_SMD:D_SMA, F.Cu at (-30.1, 64.2)
- added JP4: S_Jumper, Jumper:SolderJumper-2_P1.3mm_Open_TrianglePad1.0x1.5mm, F.Cu at (-9.48, 95.4)
- added L6: 4.7uH, zLibrary:IND_SRP7028A-4R7M_BRN-M, F.Cu at (-50.7, 42.9)
- added L7: 4.7uH, zLibrary:IND_SRP7028A-4R7M_BRN-M, F.Cu at (-20.2, 42.9)
- added Q12: NMOS, Package_TO_SOT_SMD:LFPAK56, F.Cu at (-60.7, 48.5)
- added Q13: NMOS, Package_TO_SOT_SMD:LFPAK56, F.Cu at (-30.2, 41.8)
- added Q14: NMOS, Package_TO_SOT_SMD:LFPAK56, F.Cu at (-30.2, 48.5)
- added R68: 2.5, Resistor_SMD:R_0805_2012Metric, F.Cu at (-43.5, 9.72)
- added R69: 4.7k, Resistor_SMD:R_0603_1608Metric, F.Cu at (-66.7, 22.1)
- added R70: 4.7k, Resistor_SMD:R_0603_1608Metric, F.Cu at (-66.7, 24.6)
- added R71: 10k, Resistor_SMD:R_0805_2012Metric, F.Cu at (-43.5, 12.7)
- added R72: 25m, Resistor_SMD:R_0815_2038Metric, F.Cu at (-43.9, 20.1)
- added R73: 10k, Resistor_SMD:R_0805_2012Metric, F.Cu at (-43.5, 15.6)
- added R74: 63.4k, Resistor_SMD:R_0603_1608Metric, F.Cu at (-66.7, 27.1)
- added R75: 2.5, Resistor_SMD:R_0805_2012Metric, F.Cu at (-13.0, 9.72)
- added R76: 4.7k, Resistor_SMD:R_0603_1608Metric, F.Cu at (-36.2, 22.1)
- added R77: 4.7k, Resistor_SMD:R_0603_1608Metric, F.Cu at (-36.2, 24.6)
- added R78: 10k, Resistor_SMD:R_0805_2012Metric, F.Cu at (-13.0, 12.7)
- added R79: 25m, Resistor_SMD:R_0815_2038Metric, F.Cu at (-13.4, 20.1)
- added R80: 10k, Resistor_SMD:R_0805_2012Metric, F.Cu at (-13.0, 15.6)
- added R81: 63.4k, Resistor_SMD:R_0603_1608Metric, F.Cu at (-36.2, 27.1)
- added R82: 2.5, Resistor_SMD:R_0805_2012Metric, F.Cu at (-43.5, 39.9)
- added R83: 4.7k, Resistor_SMD:R_0603_1608Metric, F.Cu at (-66.7, 52.2)
- added R84: 4.7k, Resistor_SMD:R_0603_1608Metric, F.Cu at (-66.7, 54.7)
- added R85: 10k, Resistor_SMD:R_0805_2012Metric, F.Cu at (-43.5, 42.8)
- added R86: 25m, Resistor_SMD:R_0815_2038Metric, F.Cu at (-43.9, 50.3)
- added R87: 10k, Resistor_SMD:R_0805_2012Metric, F.Cu at (-43.5, 45.8)
- added R88: 63.4k, Resistor_SMD:R_0603_1608Metric, F.Cu at (-66.7, 57.2)
- added R89: 2.5, Resistor_SMD:R_0805_2012Metric, F.Cu at (-13.0, 39.9)
- added R90: 4.7k, Resistor_SMD:R_0603_1608Metric, F.Cu at (-36.2, 52.2)
- added R91: 4.7k, Resistor_SMD:R_0603_1608Metric, F.Cu at (-36.2, 54.7)
- added R92: 10k, Resistor_SMD:R_0805_2012Metric, F.Cu at (-13.0, 42.8)
- added R93: 25m, Resistor_SMD:R_0815_2038Metric, F.Cu at (-13.4, 50.3)
- added R94: 10k, Resistor_SMD:R_0805_2012Metric, F.Cu at (-13.0, 45.8)
- added R95: 63.4k, Resistor_SMD:R_0603_1608Metric, F.Cu at (-36.2, 57.2)
- added R96: 10k, Resistor_SMD:R_0805_2012Metric, F.Cu at (-13.9, 95.1)
- added R97: 120, Resistor_SMD:R_0603_1608Metric, F.Cu at (-4.76, 83.0)
- added U16: LTC4162IUFD-LADM_PBF, Package_DFN_QFN:QFN-28-1EP_4x5mm_P0.5mm_EP2.65x3.65mm_ThermalVias, F.Cu at (-43.4, 28.7)
- added U17: LTC4162IUFD-LADM_PBF, Package_DFN_QFN:QFN-28-1EP_4x5mm_P0.5mm_EP2.65x3.65mm_ThermalVias, F.Cu at (-12.9, 28.7)
- added U18: LTC4162IUFD-LADM_PBF, Package_DFN_QFN:QFN-28-1EP_4x5mm_P0.5mm_EP2.65x3.65mm_ThermalVias, F.Cu at (-43.4, 58.8)
- added U19: LTC4162IUFD-LADM_PBF, Package_DFN_QFN:QFN-28-1EP_4x5mm_P0.5mm_EP2.65x3.65mm_ThermalVias, F.Cu at (-12.9, 58.8)
- added U21: STM32L496RGTx, Package_QFP:LQFP-64_10x10mm_P0.5mm, F.Cu at (-14.0, 86.4)
- U20: value STM32L476RGTx -> TCAN334GDCNT; footprint Package_QFP:LQFP-64_10x10mm_P0.5mm -> Package_TO_SOT_SMD:SOT-23-8
- U8: renamed from U12; value TCAN334 -> TCAN334GDCNT; footprint Package_SO:SOIC-8_3.9x4.9mm_P1.27mm -> Package_TO_SOT_SMD:SOT-23-8
- moved Q7 149.9 mm to (-60.7, 11.7)
- moved Q8 149.9 mm to (-60.7, 18.3)
- moved Q11 142.0 mm to (-60.7, 41.8)
- moved L4 137.3 mm to (-50.7, 12.8)
- moved L5 123.1 mm to (-20.2, 12.8)
- moved Q10 120.6 mm to (-30.2, 18.3)
- moved Q9 120.6 mm to (-30.2, 11.7)
- moved U20 18.2 mm to (-18.6, 96.0)
- moved Q6 1.02 mm to (85.0, 83.6)
- renumbered C50 to C14, C51 to C15, C52 to C16, C53 to C17, C54 to C18, C55 to C19, C56 to C20, C57 to C21, C58 to C22, C59 to C23, C60 to C24, C61 to C25, C62 to C26, C63 to C27, C64 to C28, C65 to C29, C66 to C30, C67 to C31, C68 to C32, C69 to C33, C70 to C34, C71 to C35, C72 to C36, C73 to C37, C74 to C38, C75 to C39, C76 to C40, C77 to C41, C78 to C42, C79 to C43, C80 to C44, C81 to C45, C82 to C46, C83 to C47, C84 to C48, C85 to C49, C86 to C50, C87 to C51, C88 to C52, C89 to C53, D6 to D2, D7 to D3, D8 to D4, J4 to J3, J3 to J4, L6 to L2, L7 to L3, Q16 to Q1, Q15 to Q2, Q17 to Q3, Q12 to Q4, Q13 to Q5, Q14 to Q6, R40 to R12, R41 to R13, R42 to R14, R43 to R15, R44 to R16, R45 to R17, R46 to R18, R47 to R19, R48 to R20, R49 to R21, R50 to R22, R51 to R23, R52 to R24, R53 to R25, R54 to R26, R55 to R27, R56 to R28, R57 to R29, R58 to R30, R59 to R31, R60 to R32, R61 to R33, R62 to R34, R63 to R35, R64 to R36, R65 to R37, R66 to R38, R67 to R39, R68 to R40, R69 to R41, R70 to R42, R71 to R43, R72 to R44, R73 to R45, R74 to R46, R75 to R47, R76 to R48, R77 to R49, R78 to R50, R79 to R51, R80 to R52, R81 to R53, R82 to R54, R83 to R55, R84 to R56, R85 to R57, R86 to R58, R87 to R59, R88 to R60, R89 to R61, R90 to R62, R91 to R63, R92 to R64, R93 to R65, R94 to R66, R95 to R67, U13 to U10, U15 to U11, U16 to U12, U17 to U13, U18 to U14, U19 to U15, U11 to U9
Connections:
- net Net-(U16-OUT) renamed /Current Sensing and Fault Detection/OBC_3V3_Line_Out
- net Net-(U17-OUT) renamed /Current Sensing and Fault Detection/ADCS_5V_Line_Out
- net Net-(U18-OUT) renamed /Current Sensing and Fault Detection/ADCS_3V3_Line_Out
- C21 pad 1: Net-(U20-VDDA) -> Net-(U21-VDDA)
- C22 pad 1: Net-(U20-VDDA) -> Net-(U21-VDDA)
- FB1 pad 1: Net-(U20-VDDA) -> Net-(U21-VDDA)
- J2 pad 02: unconnected-(J2-Pad02) -> unconnected-(J2-Pad01)
- J2 pad 04: unconnected-(J2-Pad04) -> unconnected-(J2-Pad03)
- J2 pad 05: unconnected-(J2-Pad05) -> unconnected-(J2-Pad01)
- J2 pad 06: unconnected-(J2-Pad06) -> unconnected-(J2-Pad01)
- J2 pad 07: unconnected-(J2-Pad07) -> unconnected-(J2-Pad03)
- J2 pad 08: unconnected-(J2-Pad08) -> unconnected-(J2-Pad03)
- J2 pad 09: unconnected-(J2-Pad09) -> unconnected-(J2-Pad01)
- J2 pad 10: unconnected-(J2-Pad10) -> unconnected-(J2-Pad01)
- J2 pad 100: unconnected-(J2-Pad100) -> unconnected-(J2-Pad03)
- J2 pad 101: unconnected-(J2-Pad101) -> unconnected-(J2-Pad01)
- J2 pad 102: unconnected-(J2-Pad102) -> unconnected-(J2-Pad01)
- J2 pad 103: unconnected-(J2-Pad103) -> unconnected-(J2-Pad03)
- J2 pad 104: unconnected-(J2-Pad104) -> unconnected-(J2-Pad03)
- J2 pad 11: unconnected-(J2-Pad11) -> unconnected-(J2-Pad03)
- J2 pad 12: unconnected-(J2-Pad12) -> unconnected-(J2-Pad03)
- J2 pad 13: unconnected-(J2-Pad13) -> unconnected-(J2-Pad01)
- J2 pad 14: unconnected-(J2-Pad14) -> unconnected-(J2-Pad01)
- J2 pad 15: unconnected-(J2-Pad15) -> unconnected-(J2-Pad03)
- J2 pad 16: unconnected-(J2-Pad16) -> unconnected-(J2-Pad03)
- J2 pad 17: unconnected-(J2-Pad17) -> unconnected-(J2-Pad01)
- J2 pad 18: unconnected-(J2-Pad18) -> unconnected-(J2-Pad01)
- J2 pad 19: unconnected-(J2-Pad19) -> unconnected-(J2-Pad03)
- J2 pad 20: unconnected-(J2-Pad20) -> unconnected-(J2-Pad03)
- J2 pad 21: unconnected-(J2-Pad21) -> unconnected-(J2-Pad01)
- J2 pad 22: unconnected-(J2-Pad22) -> unconnected-(J2-Pad01)
- J2 pad 23: unconnected-(J2-Pad23) -> unconnected-(J2-Pad03)
- J2 pad 24: unconnected-(J2-Pad24) -> unconnected-(J2-Pad03)
- J2 pad 25: unconnected-(J2-Pad25) -> unconnected-(J2-Pad01)
- J2 pad 26: unconnected-(J2-Pad26) -> unconnected-(J2-Pad01)
- J2 pad 27: unconnected-(J2-Pad27) -> unconnected-(J2-Pad03)
- J2 pad 28: unconnected-(J2-Pad28) -> unconnected-(J2-Pad03)
- J2 pad 29: unconnected-(J2-Pad29) -> unconnected-(J2-Pad01)
- J2 pad 30: unconnected-(J2-Pad30) -> unconnected-(J2-Pad01)
- J2 pad 31: unconnected-(J2-Pad31) -> unconnected-(J2-Pad03)
- J2 pad 32: unconnected-(J2-Pad32) -> unconnected-(J2-Pad03)
- J2 pad 33: unconnected-(J2-Pad33) -> unconnected-(J2-Pad01)
- J2 pad 34: unconnected-(J2-Pad34) -> unconnected-(J2-Pad01)
- J2 pad 35: unconnected-(J2-Pad35) -> unconnected-(J2-Pad03)
- J2 pad 36: unconnected-(J2-Pad36) -> unconnected-(J2-Pad03)
- J2 pad 37: unconnected-(J2-Pad37) -> unconnected-(J2-Pad01)
- J2 pad 38: unconnected-(J2-Pad38) -> unconnected-(J2-Pad01)
- J2 pad 39: unconnected-(J2-Pad39) -> unconnected-(J2-Pad03)
- J2 pad 40: unconnected-(J2-Pad40) -> unconnected-(J2-Pad03)
- J2 pad 41: unconnected-(J2-Pad41) -> unconnected-(J2-Pad01)
- J2 pad 42: unconnected-(J2-Pad42) -> unconnected-(J2-Pad01)
- J2 pad 43: unconnected-(J2-Pad43) -> unconnected-(J2-Pad03)
- J2 pad 44: unconnected-(J2-Pad44) -> unconnected-(J2-Pad03)
- J2 pad 45: unconnected-(J2-Pad45) -> unconnected-(J2-Pad01)
- J2 pad 46: unconnected-(J2-Pad46) -> unconnected-(J2-Pad01)
- J2 pad 47: unconnected-(J2-Pad47) -> unconnected-(J2-Pad03)
- J2 pad 48: unconnected-(J2-Pad48) -> unconnected-(J2-Pad03)
- J2 pad 49: unconnected-(J2-Pad49) -> unconnected-(J2-Pad01)
- J2 pad 50: unconnected-(J2-Pad50) -> unconnected-(J2-Pad01)
- J2 pad 51: unconnected-(J2-Pad51) -> unconnected-(J2-Pad03)
- J2 pad 52: unconnected-(J2-Pad52) -> unconnected-(J2-Pad03)
- J2 pad 53: unconnected-(J2-Pad53) -> unconnected-(J2-Pad01)
- J2 pad 54: unconnected-(J2-Pad54) -> unconnected-(J2-Pad01)
- J2 pad 55: unconnected-(J2-Pad55) -> unconnected-(J2-Pad03)
- J2 pad 56: unconnected-(J2-Pad56) -> unconnected-(J2-Pad03)
- J2 pad 57: unconnected-(J2-Pad57) -> unconnected-(J2-Pad01)
- J2 pad 58: unconnected-(J2-Pad58) -> unconnected-(J2-Pad01)
- J2 pad 59: unconnected-(J2-Pad59) -> unconnected-(J2-Pad03)
- J2 pad 60: unconnected-(J2-Pad60) -> unconnected-(J2-Pad03)
- J2 pad 61: unconnected-(J2-Pad61) -> unconnected-(J2-Pad01)
- J2 pad 62: unconnected-(J2-Pad62) -> unconnected-(J2-Pad01)
- J2 pad 63: unconnected-(J2-Pad63) -> unconnected-(J2-Pad03)
- J2 pad 64: unconnected-(J2-Pad64) -> unconnected-(J2-Pad03)
- J2 pad 65: unconnected-(J2-Pad65) -> unconnected-(J2-Pad01)
- J2 pad 66: unconnected-(J2-Pad66) -> unconnected-(J2-Pad01)
- J2 pad 67: unconnected-(J2-Pad67) -> unconnected-(J2-Pad03)
- J2 pad 68: unconnected-(J2-Pad68) -> unconnected-(J2-Pad03)
- J2 pad 69: unconnected-(J2-Pad69) -> unconnected-(J2-Pad01)
- J2 pad 70: unconnected-(J2-Pad70) -> unconnected-(J2-Pad01)
- J2 pad 71: unconnected-(J2-Pad71) -> unconnected-(J2-Pad03)
- J2 pad 72: unconnected-(J2-Pad72) -> unconnected-(J2-Pad03)
- J2 pad 73: unconnected-(J2-Pad73) -> unconnected-(J2-Pad01)
- J2 pad 74: unconnected-(J2-Pad74) -> unconnected-(J2-Pad01)
- J2 pad 75: unconnected-(J2-Pad75) -> unconnected-(J2-Pad03)
- J2 pad 76: unconnected-(J2-Pad76) -> unconnected-(J2-Pad03)
- J2 pad 77: unconnected-(J2-Pad77) -> unconnected-(J2-Pad01)
- J2 pad 78: unconnected-(J2-Pad78) -> unconnected-(J2-Pad01)
- J2 pad 79: unconnected-(J2-Pad79) -> unconnected-(J2-Pad03)
- J2 pad 80: unconnected-(J2-Pad80) -> unconnected-(J2-Pad03)
- J2 pad 81: unconnected-(J2-Pad81) -> unconnected-(J2-Pad01)
- J2 pad 82: unconnected-(J2-Pad82) -> unconnected-(J2-Pad01)
- J2 pad 83: unconnected-(J2-Pad83) -> unconnected-(J2-Pad03)
- J2 pad 84: unconnected-(J2-Pad84) -> unconnected-(J2-Pad03)
- J2 pad 85: unconnected-(J2-Pad85) -> unconnected-(J2-Pad01)
- J2 pad 86: unconnected-(J2-Pad86) -> unconnected-(J2-Pad01)
- J2 pad 87: unconnected-(J2-Pad87) -> unconnected-(J2-Pad03)
- J2 pad 88: unconnected-(J2-Pad88) -> unconnected-(J2-Pad03)
- J2 pad 89: unconnected-(J2-Pad89) -> unconnected-(J2-Pad01)
- J2 pad 90: unconnected-(J2-Pad90) -> unconnected-(J2-Pad01)
- J2 pad 91: unconnected-(J2-Pad91) -> unconnected-(J2-Pad03)
- J2 pad 92: unconnected-(J2-Pad92) -> unconnected-(J2-Pad03)
- J2 pad 93: unconnected-(J2-Pad93) -> unconnected-(J2-Pad01)
- J2 pad 94: unconnected-(J2-Pad94) -> unconnected-(J2-Pad01)
- J2 pad 95: unconnected-(J2-Pad95) -> unconnected-(J2-Pad03)
- J2 pad 96: unconnected-(J2-Pad96) -> unconnected-(J2-Pad03)
- J2 pad 97: unconnected-(J2-Pad97) -> unconnected-(J2-Pad01)
- J2 pad 98: unconnected-(J2-Pad98) -> unconnected-(J2-Pad01)
- J2 pad 99: unconnected-(J2-Pad99) -> unconnected-(J2-Pad03)
- J3 pad 1: unconnected-(J4-Pad1) -> GND
- J4 pad 1: unconnected-(J3-Pad1) -> GND
- J5 pad 1: unconnected-(J5-Pad1) -> GND
- J6 pad 1: unconnected-(J6-Pad1) -> GND
- L4 pad 2: Net-(Q9-S) -> Net-(Q8-S)
- L5 pad 2: Net-(Q11-S) -> Net-(Q10-S)
- Q10 pad 1: /MPPT IC/VOUT_-Y -> /MPPT IC/+X_MPPT/VOUT_+X
- Q10 pad 3: /MPPT IC/SOLAR_-Y -> Net-(Q10-S)
- Q11 pad 1: /MPPT IC/VOUT_-Y -> /MPPT IC/+Y_MPPT/VOUT_+X
- Q11 pad 3: Net-(Q11-S) -> /MPPT IC/SOLAR_+Y
- Q7 pad 1: /MPPT IC/VOUT_-X -> /MPPT IC/-X_MPPT/VOUT_+X
- Q7 pad 3: Net-(Q7-S) -> /MPPT IC/SOLAR_-X
- Q8 pad 1: /MPPT IC/VOUT_+Y -> /MPPT IC/-X_MPPT/VOUT_+X
- Q8 pad 3: /MPPT IC/SOLAR_+Y -> Net-(Q8-S)
- Q9 pad 1: /MPPT IC/VOUT_+Y -> /MPPT IC/+X_MPPT/VOUT_+X
- Q9 pad 3: Net-(Q9-S) -> /3.3V Logic/Solar_+X
- R12 pad 1: Net-(U20-NRST) -> Net-(U21-NRST)
- R13 pad 2: Net-(U20-NRST) -> Net-(U21-NRST)
- R14 pad 1: Net-(U20-BOOT0) -> Net-(U21-PH3)
- U20 pad 1: +3.3V -> /STM32L4/CANTX2
- U20 pad 2: /Current Sensing and Fault Detection/WAR_INA3221 -> GND
- U20 pad 3: /Current Sensing and Fault Detection/CRIT_INA3221 -> +3.3V
- U20 pad 4: unconnected-(U20-PC15-Pad4) -> /STM32L4/CANRX2
- U20 pad 5: /STM32L4/OSC_In -> /STM32L4/C_SHDN2
- U20 pad 6: /STM32L4/OSC_Out -> /STM32L4/CAN_L2
- U20 pad 7: Net-(U20-NRST) -> /STM32L4/CAN_H2
- U20 pad 8: unconnected-(U20-PC0-Pad8) -> Net-(U20-STB)

Commit message: Small schematic changes
Parts:
- moved L1 197.1 mm to (-151.7, 45.6)
- moved U2 191.9 mm to (-136.4, 45.5)
- moved U3 191.9 mm to (-140.7, 45.6)
- moved C10 185.4 mm to (-126.5, 41.5)
- moved C12 185.4 mm to (-126.5, 44.0)
- moved C2 137.5 mm to (-135.2, 19.0)
- moved C4 137.5 mm to (-135.2, 21.5)
- moved C6 137.5 mm to (-150.6, 26.9)
- moved C7 137.5 mm to (-150.6, 34.6)
- moved C8 137.5 mm to (-135.2, 26.6)
- moved C9 137.5 mm to (-135.2, 29.1)
- moved Q1 137.5 mm to (-141.3, 25.1)
- moved Q2 137.5 mm to (-141.3, 18.5)
- moved Q3 137.5 mm to (-141.3, 31.6)
- moved R1 137.5 mm to (-131.2, 19.0)
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
Commit message: Changed LTC 4412 to 4417, still kinks to work out
Parts:
- removed the C11 at (-131.2, 16.5)
- removed the C12 at (-126.5, 44.0)
- removed the C8 at (-135.2, 26.6)
- removed the U4 at (-134.6, 37.4)
- removed the U5 at (-129.2, 32.7)
- added C2: 100nF, Capacitor_SMD:C_0603_1608Metric, F.Cu at (-144.8, 93.6)
- added C3: 100nF, Capacitor_SMD:C_0603_1608Metric, F.Cu at (-144.8, 96.1)
- added C4: 1uF, Capacitor_SMD:C_0603_1608Metric, F.Cu at (-144.8, 103.7)
- added C5: 6.8nF, Capacitor_SMD:C_0603_1608Metric, F.Cu at (-144.8, 101.2)
- added C6: 100uF, Capacitor_Tantalum_SMD:CP_EIA-7361-38_AVX-V, F.Cu at (-141.9, 113.8)
- added D1: BAT54J, Diode_SMD:D_SOD-323F, F.Cu at (-132.7, 93.9)
- added D10: D_Schottky, Diode_SMD:D_0603_1608Metric, F.Cu at (-64.5, 118.5)
- added Q4: SIR5607DP-T1-RE3, Package_SO:PowerPAK_SO-8_Single, F.Cu at (-150.9, 102.2)
- added R1: 1M, Resistor_SMD:R_0603_1608Metric, F.Cu at (-136.8, 101.2)
- added R11: 100k, Resistor_SMD:R_0603_1608Metric, F.Cu at (-144.8, 106.2)
- added R12: 100k, Resistor_SMD:R_0603_1608Metric, F.Cu at (-144.8, 108.7)
- added R13: 100k, Resistor_SMD:R_0603_1608Metric, F.Cu at (-140.8, 93.6)
- added R2: 140k, Resistor_SMD:R_0603_1608Metric, F.Cu at (-140.8, 103.7)
- added R4: 1M, Resistor_SMD:R_0603_1608Metric, F.Cu at (-136.8, 98.7)
- added R5: 57.6k, Resistor_SMD:R_0603_1608Metric, F.Cu at (-140.8, 98.7)
- added R6: 52.3k, Resistor_SMD:R_0603_1608Metric, F.Cu at (-140.8, 101.2)
- Q10: renamed from Q11; footprint Package_TO_SOT_SMD:LFPAK56 -> Package_TO_SOT_SMD:TSOT-23
- Q11: renamed from Q12; footprint Package_TO_SOT_SMD:LFPAK56 -> Package_TO_SOT_SMD:TSOT-23
- Q12: renamed from Q7; footprint Package_TO_SOT_SMD:LFPAK56 -> Package_TO_SOT_SMD:TSOT-23
- Q13: renamed from Q8; footprint Package_TO_SOT_SMD:LFPAK56 -> Package_TO_SOT_SMD:TSOT-23
- Q14: renamed from Q13; footprint Package_TO_SOT_SMD:LFPAK56 -> Package_TO_SOT_SMD:TSOT-23
- Q15: renamed from Q14; footprint Package_TO_SOT_SMD:LFPAK56 -> Package_TO_SOT_SMD:TSOT-23
- Q5: renamed from Q4; footprint Package_TO_SOT_SMD:LFPAK56 -> Package_TO_SOT_SMD:TSOT-23
- Q6: footprint Package_TO_SOT_SMD:LFPAK56 -> Package_TO_SOT_SMD:TSOT-23
- Q7: renamed from Q5; footprint Package_TO_SOT_SMD:LFPAK56 -> Package_TO_SOT_SMD:TSOT-23
- Q8: renamed from Q9; footprint Package_TO_SOT_SMD:LFPAK56 -> Package_TO_SOT_SMD:TSOT-23
- Q9: renamed from Q10; footprint Package_TO_SOT_SMD:LFPAK56 -> Package_TO_SOT_SMD:TSOT-23
- R10: value 499k -> 2.21k
- R3: value 470k -> 60.4k
- R7: value 470k -> 1M
- R8: value 665k -> 82.5k
- R9: value 165k -> 412k
- U1: value LTC4412xS6 -> LTC4417HUF; footprint Package_TO_SOT_SMD:TSOT-23-6 -> Package_DFN_QFN:QFN-24-1EP_4x4mm_P0.5mm_EP2.6x2.6mm
- moved Q1 90.7 mm to (-150.9, 115.3)
- moved Q2 90.7 mm to (-150.9, 108.8)
- moved R7 90.7 mm to (-140.8, 108.7)
- moved C1 82.7 mm to (-144.8, 98.7)
- moved R3 82.7 mm to (-140.8, 106.2)
- moved U1 73.8 mm to (-136.2, 106.6)
- moved R8 72.7 mm to (-136.8, 93.6)
- moved R9 72.7 mm to (-136.8, 96.1)
- moved R10 70.9 mm to (-140.8, 96.1)
- moved Q3 64.7 mm to (-150.9, 95.7)
- moved U6 3.75 mm to (-111.0, 100.5), turned to 180 degrees
- moved C68 1.12 mm to (-96.0, 43.3)
- moved C69 1.12 mm to (-96.0, 45.9)
- moved C70 1.12 mm to (-96.0, 40.8)
- moved C71 1.12 mm to (-96.0, 38.3)
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- renumbered C2 to C10, C3 to C11, C4 to C12, C6 to C13, C7 to C14, C13 to C15, C14 to C16, C24 to C17, C15 to C18, C26 to C19, C16 to C20, C25 to C21, C17 to C22, C18 to C23, C19 to C24, C20 to C25, C21 to C26, C22 to C27, C23 to C28, C90 to C29, C27 to C30, C28 to C31, C29 to C32, C37 to C33, C41 to C34, C42 to C35, C35 to C36, C40 to C37, C33 to C38, C32 to C39, C34 to C40, C45 to C41, C46 to C42, C30 to C43, C31 to C44, C39 to C45, C38 to C46, C43 to C47, C44 to C48, C36 to C49, C53 to C50, C49 to C51, C51 to C52, C47 to C53, C48 to C54, C50 to C55, C52 to C56, C69 to C57, C70 to C58, C67 to C59, C68 to C60, C66 to C61, C64 to C62, C71 to C63, C63 to C64, C78 to C66, C79 to C67, C76 to C68, C77 to C69, C5 to C7, C75 to C70, C73 to C71, C80 to C72, C72 to C73, C60 to C75, C61 to C76, C58 to C77, C59 to C78, C57 to C79, C9 to C8, C55 to C80, C62 to C81, C54 to C82, C56 to C83, C87 to C84, C88 to C85, C85 to C86, C86 to C87, C84 to C88, C82 to C89, C10 to C9, C89 to C90, C81 to C91, C83 to C92, D2 to D3, D3 to D4, D4 to D5, D5 to D8, D8 to D9, J4 to J2, J5 to J3, J2 to J4, J3 to J5, L3 to L2, L2 to L3, L5 to L4, L6 to L5, L4 to L6, R90 to R100, R91 to R101, R92 to R102, R95 to R103, R93 to R104, R94 to R105, R4 to R14, R1 to R15, R6 to R16, R2 to R17, R5 to R18, R11 to R19, R13 to R21, R14 to R22, R12 to R23, R15 to R24, R19 to R25, R96 to R26, R16 to R27, R17 to R28, R18 to R29, R97 to R30, R21 to R31, R22 to R32, R23 to R33, R24 to R34, R25 to R35, R26 to R36, R27 to R37, R28 to R38, R58 to R39, R46 to R40, R49 to R41, R54 to R42, R52 to R44, R38 to R45, R36 to R46, R39 to R47, R41 to R48, R60 to R49, R30 to R50, R48 to R51, R51 to R52, R57 to R53, R29 to R54, R37 to R55, R40 to R56, R42 to R57, R45 to R58, R31 to R59, R55 to R60, R32 to R61, R33 to R62, R34 to R63, R35 to R64, R59 to R65, R47 to R66, R50 to R67, R56 to R68, R44 to R69, R53 to R70, R63 to R71, R65 to R72, R66 to R73, R61 to R74, R62 to R75, R64 to R76, R67 to R77, R75 to R78, R76 to R79, R77 to R80, R78 to R81, R81 to R82, R79 to R83, R80 to R84, R82 to R85, R83 to R86, R84 to R87, R85 to R88, R88 to R89, R86 to R90, R87 to R91, R68 to R92, R69 to R93, R70 to R94, R71 to R95, R74 to R96, R72 to R97, R73 to R98, R89 to R99, U12 to U10, U14 to U11, U11 to U12, U15 to U14, U17 to U15, U18 to U16, U16 to U17, U19 to U18, U6 to U4, U9 to U5, U21 to U6, U8 to U7, U20 to U8, U10 to U9
Connections:
- net /3.3V and 5V Line/VOUT1 renamed /3.3V and 5V Line/5V_Line
- net /3.3V and 5V Line/VOUT2 renamed /3.3V and 5V Line/3.3V_Line
- net /STM32L4/CAN_H renamed /PC104/CAN2+
- net /STM32L4/CAN_H2 renamed /PC104/CAN+
- net /STM32L4/CAN_L renamed /PC104/CAN-
- net /STM32L4/CAN_L2 renamed /PC104/CAN2-
- net Net-(U1-STAT) renamed /3.3V Logic/OV1
- C1 pad 1: /3.3V Logic/Solar_+X -> BATT
- C16 pad 1: /MPPT IC/MPPT_CAP -> BATT
- C33 pad 1: /Current Sensing and Fault Detection/OBC3V3 -> /Current Sensing and Fault Detection/OBC_3V3
- C63 pad 2: /MPPT IC/MPPT_CAP -> BATT
- C7 pad 1: Net-(U1-SENSE) -> Net-(Q1-D)
- C72 pad 2: /MPPT IC/MPPT_CAP -> BATT
- C81 pad 2: /MPPT IC/MPPT_CAP -> BATT
- C90 pad 2: /MPPT IC/MPPT_CAP -> BATT
- Q1 pad 1: /3.3V Logic/Solar_+X -> Net-(U1-VS1)
- Q1 pad 2: /3.3V Logic/Solar_+X -> Net-(U1-VS1)
- Q1 pad 3: /3.3V Logic/Solar_+X -> Net-(U1-VS1)
- Q1 pad 4: Net-(Q1-G) -> Net-(D1-K)
- Q2 pad 1: Net-(U1-SENSE) -> Net-(U1-VS1)
- Q2 pad 2: Net-(U1-SENSE) -> Net-(U1-VS1)
- Q2 pad 3: Net-(U1-SENSE) -> Net-(U1-VS1)
- Q2 pad 4: Net-(Q1-G) -> Net-(D1-K)
- Q2 pad 5: Net-(Q1-D) -> BATT
- Q3 pad 1: Net-(U1-SENSE) -> Net-(Q3-S-Pad1)
- Q3 pad 2: Net-(U1-SENSE) -> Net-(Q3-S-Pad1)
- Q3 pad 3: Net-(U1-SENSE) -> Net-(Q3-S-Pad1)
- Q3 pad 5: /3.3V Logic/Battery -> /3.3V Logic/Solar_+X
- Q7 pad 2: /Current Sensing and Fault Detection/ADCS_3V3_ShutDown -> /Current Sensing and Fault Detection/ADCS_5V_ShutDown
- R10 pad 1: Net-(U5-INL) -> Net-(D1-A)
- R10 pad 2: GND -> Net-(D1-K)
- R104 pad 2: /MPPT IC/MPPT_CAP -> BATT
- R14 pad 1: Net-(U1-SENSE) -> Net-(Q1-D)
- R21 pad 1: /External Watchdog IC/OBC_Notif -> /External Watchdog IC/Reset
- R3 pad 2: +3.3V -> GND
- R40 pad 1: /Current Sensing and Fault Detection/OBC3V3 -> /Current Sensing and Fault Detection/OBC_3V3
- R65 pad 1: /Current Sensing and Fault Detection/ADCS_3V3_ShutDown -> /Current Sensing and Fault Detection/ADCS_5V_ShutDown
- R7 pad 1: Net-(U4-STAT) -> +3.3V
- R7 pad 2: +3.3V -> /3.3V Logic/UV3
- R8 pad 1: Net-(U5-PS) -> /3.3V Logic/UV3
- R8 pad 2: Net-(U5-INH) -> /3.3V Logic/OV3
- R83 pad 2: /MPPT IC/MPPT_CAP -> BATT
- R9 pad 1: Net-(U5-INH) -> /3.3V Logic/OV3
- R9 pad 2: Net-(U5-INL) -> GND
- R90 pad 2: /MPPT IC/MPPT_CAP -> BATT
- R97 pad 2: /MPPT IC/MPPT_CAP -> BATT
- U1 pad 1: /3.3V Logic/Solar_+X -> /3.3V Logic/UV2
- U1 pad 2: GND -> /3.3V Logic/OV2
- U1 pad 3: /3.3V Logic/Cont -> /3.3V Logic/UV1
- U1 pad 5: Net-(Q1-G) -> /3.3V Logic/UV3
- U1 pad 6: Net-(U1-SENSE) -> /3.3V Logic/OV3
- U10 pad 5: /Current Sensing and Fault Detection/OBC3V3 -> /Current Sensing and Fault Detection/OBC_3V3
- U14 pad 15: /3.3V Logic/Battery -> BATT
- U14 pad 16: /3.3V Logic/Battery -> BATT
- U14 pad 21: /3.3V Logic/Battery -> BATT
- U14 pad 22: /3.3V Logic/Battery -> BATT
- U15 pad 19: /MPPT IC/MPPT_CAP -> BATT
- U15 pad 20: /MPPT IC/MPPT_CAP -> BATT
- U16 pad 19: /MPPT IC/MPPT_CAP -> BATT
- U16 pad 20: /MPPT IC/MPPT_CAP -> BATT
- U17 pad 19: /MPPT IC/MPPT_CAP -> BATT
- U17 pad 20: /MPPT IC/MPPT_CAP -> BATT
- U18 pad 19: /MPPT IC/MPPT_CAP -> BATT
- U18 pad 20: /MPPT IC/MPPT_CAP -> BATT
- U2 pad 5: Net-(U1-SENSE) -> Net-(Q1-D)
- U6 pad 23: /Current Sensing and Fault Detection/ADCS_3V3_ShutDown -> /Current Sensing and Fault Detection/ADCS_5V_ShutDown
- U6 pad 57: unconnected-(U21-PB5-Pad57) -> /3.3V Logic/!VAL1
- U6 pad 58: unconnected-(U21-PB6-Pad58) -> /3.3V Logic/!VAL2

Commit message: Started PCB layout
Parts:
- removed the C16 at (-91.5, 71.5)
- removed J4: ESQT-126-X-X-Q-X, zLibrary:SAMTEC_ESQT-126-X-X-Q-X
- removed the R3 at (-140.8, 106.2)
- added C6: 6.8nF, Capacitor_SMD:C_0603_1608Metric, F.Cu at (-168.9, 137.3)
- added C93: 56n, Capacitor_SMD:C_0603_1608Metric, F.Cu at (-200.3, 139.1)
- added C94: 56n, Capacitor_SMD:C_0603_1608Metric, F.Cu at (-200.3, 141.7)
- added C95: 100n, Capacitor_SMD:C_0603_1608Metric, F.Cu at (-200.3, 144.2)
- added C96: 100 uF, Capacitor_Tantalum_SMD:CP_EIA-7361-38_AVX-V, F.Cu at (-93.2, 20.8)
- added C97: 56n, Capacitor_SMD:C_0603_1608Metric, F.Cu at (-188.2, 139.1)
- added C98: 56n, Capacitor_SMD:C_0603_1608Metric, F.Cu at (-188.2, 141.7)
- added C99: 100n, Capacitor_SMD:C_0603_1608Metric, F.Cu at (-188.2, 144.2)
- added H1: MountingHole_Pad, MountingHole:MountingHole_3.2mm_M3_Pad, F.Cu at (183.8, 136.9)
- added H2: MountingHole_Pad, MountingHole:MountingHole_3.2mm_M3_Pad, F.Cu at (103.8, 136.9)
- added H3: MountingHole_Pad, MountingHole:MountingHole_3.2mm_M3_Pad, F.Cu at (180.0, 51.2)
- added H4: MountingHole_Pad, MountingHole:MountingHole_3.2mm_M3_Pad, F.Cu at (106.4, 51.2)
- added J7: ESQ-126-39-G-D, zLibrary:SAMTEC_ESQ-126-39-G-D, F.Cu at (111.4, 56.2)
- added J8: ESQ-126-39-G-D, zLibrary:SAMTEC_ESQ-126-39-G-D, F.Cu at (111.4, 51.2)
- added R106: 10m, Resistor_SMD:R_0815_2038Metric, F.Cu at (-84.1, 36.4)
- added R110: 100k, Resistor_SMD:R_0603_1608Metric, F.Cu at (-195.2, 157.0)
- added R111: 100k, Resistor_SMD:R_0603_1608Metric, F.Cu at (-189.2, 157.0)
- added R112: 100k, Resistor_SMD:R_0603_1608Metric, F.Cu at (-195.2, 159.5)
- added R113: 100k, Resistor_SMD:R_0603_1608Metric, F.Cu at (-189.2, 159.5)
- added R5: 60.4k, Resistor_SMD:R_0603_1608Metric, F.Cu at (-168.9, 139.8)
- added R82: 10m, Resistor_SMD:R_0815_2038Metric, F.Cu at (124.8, 73.4)
- added R90: 10m, Resistor_SMD:R_0815_2038Metric, F.Cu at (-84.1, 24.3)
- added R98: 10m, Resistor_SMD:R_0815_2038Metric, F.Cu at (-95.9, 33.9)
- added U19: LTC4353IDE-PBF, zLibrary:DFN-16_DE_LIT-M, F.Cu at (-195.2, 141.0)
- added U20: LTC4353IDE-PBF, zLibrary:DFN-16_DE_LIT-M, F.Cu at (-183.2, 141.0)
- added U21: ~, Package_TO_SOT_SMD:LFPAK33, F.Cu at (-196.1, 128.9)
- added U22: ~, Package_TO_SOT_SMD:LFPAK33, F.Cu at (-188.7, 128.9)
- added U23: ~, Package_TO_SOT_SMD:LFPAK33, F.Cu at (-196.1, 133.8)
- added U24: ~, Package_TO_SOT_SMD:LFPAK33, F.Cu at (-188.7, 133.8)
- C4: value 1uF -> 100nF
- C5: value 6.8nF -> 1uF
- R107: renamed from R103; value 63.4k -> 44.2k
- R73: value 320k -> 215k
- R83: renamed from R82; value 63.4k -> 44.2k
- R91: renamed from R89; value 63.4k -> 44.2k
- R99: renamed from R96; value 63.4k -> 44.2k
- moved C59 202.6 mm to (126.0, 76.0), turned to 180 degrees
- moved U15 180.5 mm to (130.2, 74.8)
- moved C57 179.4 mm to (118.5, 82.8), turned to -90 degrees
- moved C58 175.4 mm to (111.8, 82.8), turned to -90 degrees
- moved D6 175.1 mm to (109.8, 71.2), turned to 90 degrees
- moved R78 168.7 mm to (109.8, 76.7), turned to -90 degrees
- moved J2 95.8 mm to (101.7, 73.3), turned to -90 degrees
- moved J6 95.2 mm to (185.9, 73.3), turned to 90 degrees
- moved J5 93.6 mm to (101.7, 114.7), turned to -90 degrees
- moved J3 92.4 mm to (185.9, 114.7), turned to 90 degrees
- moved C60 55.9 mm to (-77.4, 70.6)
- moved C67 55.9 mm to (-92.2, 102.4)
- moved C69 55.9 mm to (-106.8, 100.7)
- moved C75 55.9 mm to (-92.6, 79.9)
- moved C76 55.9 mm to (-92.2, 72.2)
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- renumbered C9 to C10, C10 to C11, C11 to C12, C12 to C13, C13 to C14, C14 to C15, C15 to C16, C6 to C7, C7 to C8, C8 to C9, D10 to D2, R4 to R1, R97 to R100, R98 to R101, R99 to R102, R100 to R103, R101 to R104, R102 to R105, R104 to R108, R105 to R109, R5 to R2, R6 to R3, R1 to R4, R2 to R6, R83 to R84, R84 to R85, R85 to R86, R86 to R87, R87 to R88, R88 to R89, R90 to R92, R91 to R93, R92 to R94, R93 to R95, R94 to R96, R95 to R97
Connections:
- C5 pad 1: Net-(D1-K) -> GND
- C5 pad 2: Net-(Q1-D) -> Net-(U1-VS2)
- C51 pad 2: GND -> GNDS
- C63 pad 2: BATT -> /MPPT IC/+X_OUT
- C72 pad 2: BATT -> /MPPT IC/+Y_OUT
- C81 pad 2: BATT -> /MPPT IC/-X_OUT
- C90 pad 2: BATT -> /MPPT IC/-Y_OUT
- Q1 pad 4: Net-(D1-K) -> Net-(Q1-G)
- Q10 pad 1: /MPPT IC/+Y_MPPT/VOUT_+X -> Net-(Q10-D)
- Q12 pad 1: /MPPT IC/-X_MPPT/VOUT_+X -> Net-(Q12-D)
- Q14 pad 1: /MPPT IC/-Y_MPPT/VOUT_+X -> Net-(Q14-D)
- Q2 pad 4: Net-(D1-K) -> Net-(Q1-G)
- Q3 pad 1: Net-(Q3-S-Pad1) -> Net-(U1-VS2)
- Q3 pad 2: Net-(Q3-S-Pad1) -> Net-(U1-VS2)
- Q3 pad 3: Net-(Q3-S-Pad1) -> Net-(U1-VS2)
- Q3 pad 4: Net-(Q3-G) -> Net-(D1-K)
- Q4 pad 1: Net-(Q3-S-Pad1) -> Net-(U1-VS2)
- Q4 pad 2: Net-(Q3-S-Pad1) -> Net-(U1-VS2)
- Q4 pad 3: Net-(Q3-S-Pad1) -> Net-(U1-VS2)
- Q4 pad 4: Net-(Q3-G) -> Net-(D1-K)
- Q8 pad 1: /MPPT IC/+X_MPPT/VOUT_+X -> Net-(Q8-D)
- R1 pad 1: BATT -> /3.3V Logic/Solar_+X
- R100 pad 2: BATT -> /MPPT IC/-X_OUT
- R108 pad 2: BATT -> /MPPT IC/-Y_OUT
- R4 pad 1: /3.3V Logic/Solar_+X -> BATT
- R6 pad 1: /3.3V Logic/UV1 -> /3.3V Logic/OV1
- R6 pad 2: /3.3V Logic/OV1 -> GND
- R72 pad 2: GND -> GNDS
- R73 pad 2: GND -> GNDS
- R77 pad 2: GND -> GNDS
- R84 pad 2: BATT -> /MPPT IC/+X_OUT
- R92 pad 2: BATT -> /MPPT IC/+Y_OUT
- U1 pad 1: /3.3V Logic/UV2 -> /3.3V Logic/UV1
- U1 pad 15: Net-(Q3-G) -> Net-(D1-A)
- U1 pad 16: /3.3V Logic/Solar_+X -> Net-(U1-VS2)
- U1 pad 17: Net-(D1-A) -> Net-(Q1-G)
- U1 pad 2: /3.3V Logic/OV2 -> /3.3V Logic/OV1
- U1 pad 3: /3.3V Logic/UV1 -> /3.3V Logic/UV2
- U1 pad 4: /3.3V Logic/OV1 -> /3.3V Logic/OV2
- U14 pad 3: /3.3V and 5V Line/EN_Line_1 -> BATT
- U14 pad 4: GND -> /3.3V and 5V Line/SYNC
- U14 pad 6: /3.3V and 5V Line/EN_Line_2 -> BATT
- U14 pad 7: GND -> GNDS
- U15 pad 16: /MPPT IC/MPPT_SYNC_1.5MHz -> /3.3V and 5V Line/SYNC
- U15 pad 19: BATT -> /MPPT IC/+X_OUT
- U15 pad 20: BATT -> /MPPT IC/+X_OUT
- U15 pad 5: /MPPT IC/+X_MPPT/VOUT_+X -> Net-(Q8-D)
- U16 pad 16: /MPPT IC/MPPT_SYNC_1.5MHz -> /3.3V and 5V Line/SYNC
- U16 pad 19: BATT -> /MPPT IC/+Y_OUT
- U16 pad 20: BATT -> /MPPT IC/+Y_OUT
- U16 pad 5: /MPPT IC/+Y_MPPT/VOUT_+X -> Net-(Q10-D)
- U17 pad 16: /MPPT IC/MPPT_SYNC_1.5MHz -> /3.3V and 5V Line/SYNC
- U17 pad 19: BATT -> /MPPT IC/-X_OUT
- U17 pad 20: BATT -> /MPPT IC/-X_OUT
- U17 pad 5: /MPPT IC/-X_MPPT/VOUT_+X -> Net-(Q12-D)
- U18 pad 16: /MPPT IC/MPPT_SYNC_1.5MHz -> /3.3V and 5V Line/SYNC
- U18 pad 19: BATT -> /MPPT IC/-Y_OUT
- U18 pad 20: BATT -> /MPPT IC/-Y_OUT
- U18 pad 5: /MPPT IC/-Y_MPPT/VOUT_+X -> Net-(Q14-D)
- U6 pad 21: /MPPT IC/MPPT_SYNC_1.5MHz -> /3.3V and 5V Line/SYNC
- U6 pad 26: /3.3V and 5V Line/EN_Line_2 -> /EN1
- U6 pad 27: /3.3V and 5V Line/EN_Line_1 -> /EN2
- U6 pad 30: unconnected-(U6-PB11-Pad30) -> /EN4
- U6 pad 37: unconnected-(U6-PC6-Pad37) -> /OR1
- U6 pad 38: unconnected-(U6-PC7-Pad38) -> /OR2
- U6 pad 42: unconnected-(U6-PA9-Pad42) -> /OR3
- U6 pad 43: unconnected-(U6-PA10-Pad43) -> /OR4
- U6 pad 59: unconnected-(U6-PB7-Pad59) -> /EN3
Routing:
- added copper zone on In1.Cu, net GND
- added copper zone on In4.Cu, net GND
Other:
- board size 90 x 96 mm -> 90.2 x 95.9 mm
