File: EPS_mppt_board.kicad_pcb (KiCad board)
At the start: 6 copper layers, 90.2 x 95.9 mm, 284 parts, among them J1 Conn_01x04_Pin, J2 M80-5400642, J3 M80-5400642, J5 M80-5400642, J6 M80-5400642, J7 ESQ-126-39-G-D, J8 ESQ-126-39-G-D, Q1 SIR5607DP-T1-RE3, Q10 NMOS, Q11 NMOS, Q12 NMOS, Q13 NMOS, Q14 NMOS, Q15 NMOS, Q2 SIR5607DP-T1-RE3, Q3 SIR5607DP-T1-RE3, Q4 SIR5607DP-T1-RE3, Q5 NMOS, Q6 NMOS, Q7 NMOS, Q8 NMOS, Q9 NMOS, U1 LTC4417HUF, U10 TPS259470ARPWR, U11 TPS259470ARPWR, U12 INA3221, U13 TPS259470ARPWR, U14 LTC3633AIUFDPBF, U15 LTC4162IUFD-LADM_PBF, U16 LTC4162IUFD-LADM_PBF, U17 LTC4162IUFD-LADM_PBF, U18 LTC4162IUFD-LADM_PBF, U19 LTC4353IDE-PBF, U2 TPS259470ARPWR, U20 LTC4353IDE-PBF, U3 TPS62177DQCR, U4 TPS3823A-33DBVR, U5 MR20H40, U6 STM32L496RGTx, U7 TCAN334GDCNT, U8 TCAN334GDCNT, U9 TCA9548AMRGER, Y1 8 MHZ Oscillator

Commit message: LTC4162 layout almost done
Parts:
- removed the C63 at (-71.5, 80.3)
- removed the C66 at (-92.6, 110.1)
- removed R110, R111, R112, R113: 100k, Resistor_SMD:R_0603_1608Metric
- removed U19, U20: LTC4353IDE-PBF, zLibrary:DFN-16_DE_LIT-M
- removed U21, U22, U23, U24: ~, Package_TO_SOT_SMD:LFPAK33
- added C100: 10 uF, Capacitor_SMD:C_1206_3216Metric, F.Cu at (159.7, 120.7)
- added C59: 47 uF, Capacitor_Tantalum_SMD:CP_EIA-7343-43_Kemet-X, F.Cu at (115.5, 86.1)
- added C64: 100n, Resistor_SMD:R_0402_1005Metric, F.Cu at (128.8, 78.1)
- C17, C18, C19, C20, C21, C22, C23, C24, C25, C26, C27, C28, C29, C30, C31, C32, C33, C34, C35, C36, C37, C38, C39, C40, C41, C42, C43, C44, C45, C46, C47, C48, C49, D3, D4, D5, FB1, J1, JP2, JP3, JP4, R20, R21, R22, R23, R24, R25, R26, R27, R28, R29, R30, R31, R32, R33, R34, R35, R36, R37, R38, R39, R40, R41, R42, R43, R44, R45, R46, R47, R48, R49, R50, R51, R52, R53, R54, R55, R56, R57, R58, R59, R60, R61, R62, R63, R64, R65, R66, R67, R68, R69, R70, U10, U11, U12, U13, U5, U6, U7, U8, U9, Y1: moved to B.Cu
- C57: value 100uF -> 47 uF; footprint Capacitor_Tantalum_SMD:CP_EIA-7361-38_AVX-V -> Capacitor_Tantalum_SMD:CP_EIA-7343-43_Kemet-X
- C58: value 22 uF -> 47 uF; footprint zLibrary:CAP_C2220C_2S_KEM-M -> Capacitor_Tantalum_SMD:CP_EIA-7343-43_Kemet-X
- C60: renamed from C59; footprint Capacitor_SMD:C_0603_1608Metric -> Capacitor_SMD:C_0402_1005Metric
- C61: renamed from C60; footprint Capacitor_SMD:C_0603_1608Metric -> Capacitor_SMD:C_0402_1005Metric
- C62: renamed from C61; footprint Capacitor_SMD:C_0603_1608Metric -> Capacitor_SMD:C_0402_1005Metric
- C65: footprint zLibrary:CAP_C1210C_X7R_2S_FW_KEM-M -> Capacitor_SMD:C_1206_3216Metric
- C67, C76: value 22 uF -> 10 uF; footprint zLibrary:CAP_C2220C_2S_KEM-M -> Capacitor_SMD:C_1206_3216Metric
- C68, C70, C79: value 100n -> 47 uF; footprint Capacitor_SMD:C_0603_1608Metric -> Capacitor_Tantalum_SMD:CP_EIA-7343-43_Kemet-X
- C69: value 22nF -> 47 uF; footprint Capacitor_SMD:C_0603_1608Metric -> Capacitor_Tantalum_SMD:CP_EIA-7343-43_Kemet-X
- C71: value 4.7 uF -> 100n; footprint Capacitor_SMD:C_0603_1608Metric -> Capacitor_SMD:C_0402_1005Metric
- C72, C83: value 10 uF -> 22nF; footprint zLibrary:CAP_C1210C_X7R_2S_FW_KEM-M -> Capacitor_SMD:C_0402_1005Metric
- C73, C82: value 1 uF -> 100n; footprint Capacitor_SMD:C_0603_1608Metric -> Capacitor_SMD:C_0402_1005Metric
- C74: value 10 uF -> 4.7 uF; footprint zLibrary:CAP_C1210C_X7R_2S_FW_KEM-M -> Capacitor_SMD:C_0603_1608Metric
- C75: value 100uF -> 100n; footprint Capacitor_Tantalum_SMD:CP_EIA-7361-38_AVX-V -> Resistor_SMD:R_0402_1005Metric
- C77, C88, C99: value 100n -> 1 uF
- C78, C87: value 22nF -> 10 uF; footprint Capacitor_SMD:C_0603_1608Metric -> Capacitor_SMD:C_1206_3216Metric
- C80: value 4.7 uF -> 47 uF; footprint Capacitor_SMD:C_0603_1608Metric -> Capacitor_Tantalum_SMD:CP_EIA-7343-43_Kemet-X
- C81, C90, C92: value 10 uF -> 47 uF; footprint zLibrary:CAP_C1210C_X7R_2S_FW_KEM-M -> Capacitor_Tantalum_SMD:CP_EIA-7343-43_Kemet-X
- C84: value 100uF -> 100n; footprint Capacitor_Tantalum_SMD:CP_EIA-7361-38_AVX-V -> Capacitor_SMD:C_0402_1005Metric
- C85: value 22 uF -> 4.7 uF; footprint zLibrary:CAP_C2220C_2S_KEM-M -> Capacitor_SMD:C_0603_1608Metric
- C86: footprint Capacitor_SMD:C_0603_1608Metric -> Resistor_SMD:R_0402_1005Metric
- C89: value 4.7 uF -> 10 uF; footprint Capacitor_SMD:C_0603_1608Metric -> Capacitor_SMD:C_1206_3216Metric
- C91: value 1 uF -> 47 uF; footprint Capacitor_SMD:C_0603_1608Metric -> Capacitor_Tantalum_SMD:CP_EIA-7343-43_Kemet-X
- C93: value 56n -> 100n; footprint Capacitor_SMD:C_0603_1608Metric -> Capacitor_SMD:C_0402_1005Metric
- C94: value 56n -> 22nF; footprint Capacitor_SMD:C_0603_1608Metric -> Capacitor_SMD:C_0402_1005Metric
- C95: footprint Capacitor_SMD:C_0603_1608Metric -> Capacitor_SMD:C_0402_1005Metric
- C96: value 100 uF -> 4.7 uF; footprint Capacitor_Tantalum_SMD:CP_EIA-7361-38_AVX-V -> Capacitor_SMD:C_0603_1608Metric
- C97: value 56n -> 100n; footprint Capacitor_SMD:C_0603_1608Metric -> Resistor_SMD:R_0402_1005Metric
- C98: value 56n -> 10 uF; footprint Capacitor_SMD:C_0603_1608Metric -> Capacitor_SMD:C_1206_3216Metric
- L4, L5, L6, L7: footprint zLibrary:IND_SRP7028A-4R7M_BRN-M -> zLibrary:XAL6060472MEC
- Q10, Q11, Q12, Q13, Q14, Q15, Q5, Q6, Q7, Q8, Q9: value NMOS -> Q_NMOS; footprint Package_TO_SOT_SMD:TSOT-23 -> zLibrary:IFX-PG-TSDSON-8-44-V
- R100, R108, R84, R92: value 25m -> 10m; footprint Resistor_SMD:R_0815_2038Metric -> Resistor_SMD:R_0612_1632Metric
- R102, R78, R86, R94: footprint Resistor_SMD:R_0805_2012Metric -> Resistor_SMD:R_1206_3216Metric
- R105, R81, R89, R97: footprint Resistor_SMD:R_0805_2012Metric -> Resistor_SMD:R_0603_1608Metric
- R106, R82, R90, R98: footprint Resistor_SMD:R_0815_2038Metric -> Resistor_SMD:R_0612_1632Metric
- R107, R83, R91, R99: value 44.2k -> 63.4k
- moved C95 364.7 mm to (163.3, 116.7)
- moved C94 364.4 mm to (163.4, 119.1)
- moved C93 364.4 mm to (163.3, 114.8)
- moved C99 352.6 mm to (162.8, 111.6), turned to 90 degrees
- moved C97 345.1 mm to (156.1, 116.5), turned to 180 degrees
- moved C98 342.4 mm to (153.6, 120.7), turned to 180 degrees
- moved J1 300.4 mm to (182.2, 90.2), turned to -90 degrees
- moved C70 285.3 mm to (177.0, 66.2), turned to 90 degrees
- moved C68 280.7 mm to (172.1, 66.2), turned to 90 degrees
- moved D9 276.6 mm to (178.1, 122.8), turned to -90 degrees
- moved C69 276.3 mm to (167.3, 66.2), turned to 90 degrees
- moved C96 275.0 mm to (164.1, 117.9)
- moved Q10 273.0 mm to (170.8, 80.8), turned to -90 degrees
- moved C71 271.1 mm to (163.4, 70.8)
- moved C77 270.8 mm to (162.9, 67.5), turned to 90 degrees
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- renumbered C62 to C63, C64 to C66, H3 to H2, H2 to H3, J6 to J3, J5 to J4, J3 to J5, J7 to J6, J8 to J7
Connections:
- C65 pad 1: /MPPT IC/+X_MPPT/VOUT_+X -> GND
- C65 pad 2: GND -> BATT
- C67 pad 1: Net-(C66-Pad1) -> /MPPT IC/+X_MPPT/VOUT_+X
- C68 pad 1: /MPPT IC/SOLAR_+Y -> Net-(C68-Pad1)
- C69 pad 1: Net-(U16-BOOST) -> Net-(C68-Pad1)
- C69 pad 2: Net-(U16-SW) -> GND
- C70 pad 1: /MPPT IC/+Y_MPPT/VOUT_+X -> Net-(C68-Pad1)
- C71 pad 1: /MPPT IC/+Y_MPPT/IntVCC_+X -> /MPPT IC/SOLAR_+Y
- C72 pad 1: GND -> Net-(U16-BOOST)
- C72 pad 2: /MPPT IC/+Y_OUT -> Net-(U16-SW)
- C73 pad 1: /MPPT IC/+Y_MPPT/VCC2P5_+X -> /MPPT IC/+Y_MPPT/VOUT_+X
- C74 pad 1: /MPPT IC/+Y_MPPT/VOUT_+X -> /MPPT IC/+Y_MPPT/IntVCC_+X
- C75 pad 1: Net-(C75-Pad1) -> /MPPT IC/+Y_MPPT/BATSENS
- C76 pad 1: Net-(C75-Pad1) -> GND
- C76 pad 2: GND -> BATT
- C77 pad 1: /MPPT IC/SOLAR_-X -> /MPPT IC/+Y_MPPT/VCC2P5_+X
- C78 pad 1: Net-(U17-BOOST) -> /MPPT IC/+Y_MPPT/VOUT_+X
- C78 pad 2: Net-(U17-SW) -> GND
- C79 pad 1: /MPPT IC/-X_MPPT/VOUT_+X -> Net-(C79-Pad1)
- C80 pad 1: /MPPT IC/-X_MPPT/IntVCC_+X -> Net-(C79-Pad1)
- C81 pad 1: GND -> Net-(C79-Pad1)
- C81 pad 2: /MPPT IC/-X_OUT -> GND
- C82 pad 1: /MPPT IC/-X_MPPT/VCC2P5_+X -> /MPPT IC/SOLAR_-X
- C83 pad 1: /MPPT IC/-X_MPPT/VOUT_+X -> Net-(U17-BOOST)
- C83 pad 2: GND -> Net-(U17-SW)
- C84 pad 1: Net-(C84-Pad1) -> /MPPT IC/-X_MPPT/VOUT_+X
- C85 pad 1: Net-(C84-Pad1) -> /MPPT IC/-X_MPPT/IntVCC_+X
- C86 pad 1: /MPPT IC/SOLAR_-Y -> /MPPT IC/-X_MPPT/BATSENS
- C87 pad 1: Net-(U18-BOOST) -> GND
- C87 pad 2: Net-(U18-SW) -> BATT
- C88 pad 1: /MPPT IC/-Y_MPPT/VOUT_+X -> /MPPT IC/-X_MPPT/VCC2P5_+X
- C89 pad 1: /MPPT IC/-Y_MPPT/IntVCC_+X -> /MPPT IC/-X_MPPT/VOUT_+X
- C90 pad 1: GND -> Net-(C90-Pad1)
- C90 pad 2: /MPPT IC/-Y_OUT -> GND
- C91 pad 1: /MPPT IC/-Y_MPPT/VCC2P5_+X -> Net-(C90-Pad1)
- C92 pad 1: /MPPT IC/-Y_MPPT/VOUT_+X -> Net-(C90-Pad1)
- C93 pad 1: Net-(U19-CPO2) -> /MPPT IC/SOLAR_-Y
- C93 pad 2: /MPPT IC/-Y_OUT -> GND
- C94 pad 1: Net-(U19-CPO1) -> Net-(U18-BOOST)
- C94 pad 2: /MPPT IC/+Y_OUT -> Net-(U18-SW)
- C95 pad 1: Net-(U19-VCC) -> /MPPT IC/-Y_MPPT/VOUT_+X
- C96 pad 1: BATT -> /MPPT IC/-Y_MPPT/IntVCC_+X
- C97 pad 1: Net-(U20-CPO2) -> /MPPT IC/-Y_MPPT/BATSENS
- C97 pad 2: /MPPT IC/-X_OUT -> GND
- C98 pad 1: Net-(U20-CPO1) -> GND
- C98 pad 2: /MPPT IC/+X_OUT -> BATT
- C99 pad 1: Net-(U20-VCC) -> /MPPT IC/-Y_MPPT/VCC2P5_+X
- J2 pad 3: unconnected-(J2-Pad3) -> /3.3V Logic/Solar_+X
- J2 pad 4: /3.3V Logic/Solar_+X -> unconnected-(J2-Pad4)
- J3 pad 3: unconnected-(J6-Pad3) -> /MPPT IC/SOLAR_+Y
- J3 pad 4: /MPPT IC/SOLAR_-Y -> unconnected-(J3-Pad4)
- J4 pad 1: GND -> /MPPT IC/SOLAR_-X
- J4 pad 4: /MPPT IC/SOLAR_-X -> GND
- J5 pad 3: unconnected-(J3-Pad3) -> /MPPT IC/SOLAR_-Y
- J5 pad 4: /MPPT IC/SOLAR_+Y -> unconnected-(J5-Pad4)
- L4 pad 2: Net-(Q9-S) -> Net-(U15-CSP)
- L5 pad 2: Net-(Q11-S) -> Net-(U16-CSP)
- L6 pad 2: Net-(Q13-S) -> Net-(U17-CSP)
- L7 pad 2: Net-(Q15-S) -> Net-(U18-CSP)
- Q10 pad 1: Net-(Q10-D) -> /MPPT IC/SOLAR_+Y
- Q10 pad 2: Net-(Q10-G) -> /MPPT IC/SOLAR_+Y
- Q11 pad 1: /MPPT IC/+Y_MPPT/VOUT_+X -> Net-(U16-CSP)
- Q11 pad 2: Net-(Q11-G) -> Net-(U16-CSP)
- Q11 pad 3: Net-(Q11-S) -> Net-(U16-CSP)
- Q12 pad 1: Net-(Q12-D) -> /MPPT IC/SOLAR_-X
- Q12 pad 2: Net-(Q12-G) -> /MPPT IC/SOLAR_-X
- Q13 pad 1: /MPPT IC/-X_MPPT/VOUT_+X -> Net-(U17-CSP)
- Q13 pad 2: Net-(Q13-G) -> Net-(U17-CSP)
- Q13 pad 3: Net-(Q13-S) -> Net-(U17-CSP)
- Q14 pad 1: Net-(Q14-D) -> /MPPT IC/SOLAR_-Y
- Q14 pad 2: Net-(Q14-G) -> /MPPT IC/SOLAR_-Y
- Q15 pad 1: /MPPT IC/-Y_MPPT/VOUT_+X -> Net-(U18-CSP)
- Q15 pad 2: Net-(Q15-G) -> Net-(U18-CSP)
- Q15 pad 3: Net-(Q15-S) -> Net-(U18-CSP)
- Q5 pad 1: Net-(Q5-D) -> GND
- Q5 pad 2: /Current Sensing and Fault Detection/OBC_3V3_ShutDown -> GND
- Q6 pad 1: Net-(Q6-D) -> GND
- Q6 pad 2: /Current Sensing and Fault Detection/ADCS_3V3_ShutDown -> GND
- Q7 pad 1: Net-(Q7-D) -> GND
- Q7 pad 2: /Current Sensing and Fault Detection/ADCS_5V_ShutDown -> GND
- Q8 pad 1: Net-(Q8-D) -> /3.3V Logic/Solar_+X
- Q8 pad 2: Net-(Q8-G) -> /3.3V Logic/Solar_+X
- Q9 pad 1: /MPPT IC/+X_MPPT/VOUT_+X -> Net-(U15-CSP)
- Q9 pad 2: Net-(Q9-G) -> Net-(U15-CSP)
- Q9 pad 3: Net-(Q9-S) -> Net-(U15-CSP)
- R100 pad 1: Net-(Q13-S) -> Net-(U17-CSP)
- R100 pad 2: /MPPT IC/-X_OUT -> BATT
- R102 pad 2: Net-(C84-Pad1) -> Net-(C90-Pad1)
- R106 pad 1: Net-(Q14-D) -> Net-(U18-CLP)
- R108 pad 1: Net-(Q15-S) -> Net-(U18-CSP)
- R108 pad 2: /MPPT IC/-Y_OUT -> BATT
- R40 pad 2: Net-(Q5-D) -> Net-(U10-EN_UVLO)
- R41 pad 1: Net-(Q5-D) -> Net-(U10-EN_UVLO)
- R51 pad 2: Net-(Q6-D) -> Net-(U11-EN_UVLO)
- R52 pad 1: Net-(Q6-D) -> Net-(U11-EN_UVLO)
- R66 pad 2: Net-(Q7-D) -> Net-(U13-EN_UVLO)
- R67 pad 1: Net-(Q7-D) -> Net-(U13-EN_UVLO)
- R82 pad 1: Net-(Q8-D) -> Net-(U15-CLP)
- R84 pad 1: Net-(Q9-S) -> Net-(U15-CSP)
- R84 pad 2: /MPPT IC/+X_OUT -> BATT
- R86 pad 2: Net-(C66-Pad1) -> Net-(C68-Pad1)
- R90 pad 1: Net-(Q10-D) -> Net-(U16-CLP)
- R92 pad 1: Net-(Q11-S) -> Net-(U16-CSP)
- R92 pad 2: /MPPT IC/+Y_OUT -> BATT
- R94 pad 2: Net-(C75-Pad1) -> Net-(C79-Pad1)
- R98 pad 1: Net-(Q12-D) -> Net-(U17-CLP)
- U10 pad 1: Net-(Q5-D) -> Net-(U10-EN_UVLO)
- U11 pad 1: Net-(Q6-D) -> Net-(U11-EN_UVLO)
- U13 pad 1: Net-(Q7-D) -> Net-(U13-EN_UVLO)
- U15 pad 19: /MPPT IC/+X_OUT -> /MPPT IC/+X_MPPT/BATSENS
- U15 pad 20: /MPPT IC/+X_OUT -> BATT
- U15 pad 21: Net-(Q9-S) -> Net-(U15-CSP)
- U15 pad 5: Net-(Q8-D) -> Net-(U15-CLP)
- U16 pad 19: /MPPT IC/+Y_OUT -> /MPPT IC/+Y_MPPT/BATSENS
- U16 pad 20: /MPPT IC/+Y_OUT -> BATT
- U16 pad 21: Net-(Q11-S) -> Net-(U16-CSP)
- U16 pad 5: Net-(Q10-D) -> Net-(U16-CLP)
- U17 pad 19: /MPPT IC/-X_OUT -> /MPPT IC/-X_MPPT/BATSENS
- U17 pad 20: /MPPT IC/-X_OUT -> BATT
- U17 pad 21: Net-(Q13-S) -> Net-(U17-CSP)
- U17 pad 5: Net-(Q12-D) -> Net-(U17-CLP)
- U18 pad 19: /MPPT IC/-Y_OUT -> /MPPT IC/-Y_MPPT/BATSENS
- U18 pad 20: /MPPT IC/-Y_OUT -> BATT
- U18 pad 21: Net-(Q15-S) -> Net-(U18-CSP)
- U18 pad 5: Net-(Q14-D) -> Net-(U18-CLP)
- U6 pad 26: /EN1 -> unconnected-(U6-PB0-Pad26)
- U6 pad 27: /EN2 -> unconnected-(U6-PB1-Pad27)
- U6 pad 30: /EN4 -> unconnected-(U6-PB11-Pad30)
- U6 pad 37: /OR1 -> unconnected-(U6-PC6-Pad37)
- U6 pad 38: /OR2 -> unconnected-(U6-PC7-Pad38)
- U6 pad 42: /OR3 -> unconnected-(U6-PA9-Pad42)
- U6 pad 43: /OR4 -> unconnected-(U6-PA10-Pad43)
- U6 pad 59: /EN3 -> unconnected-(U6-PB7-Pad59)
Routing:
- net BATT: track 0.00 -> 72.1 mm, vias 0 -> 32
- net +3.3V: track 0.00 -> 37.8 mm, vias 0 -> 12
- net Net-(Q13-G): track 0.00 -> 26.8 mm, vias 0 -> 2
- net Net-(Q15-G): track 0.00 -> 26.8 mm, vias 0 -> 2
- net Net-(Q9-G): track 0.00 -> 26.8 mm, vias 0 -> 2
- net Net-(Q11-G): track 0.00 -> 26.8 mm, vias 0 -> 2
- net /MPPT IC/+Y_MPPT/IntVCC_+X: track 0.00 -> 26.5 mm, vias 0 -> 2
- net /MPPT IC/-X_MPPT/IntVCC_+X: track 0.00 -> 26.5 mm, vias 0 -> 2
- net /MPPT IC/+X_MPPT/IntVCC_+X: track 0.00 -> 26.5 mm, vias 0 -> 2
- net /MPPT IC/-Y_MPPT/IntVCC_+X: track 0.00 -> 26.5 mm, vias 0 -> 2
- net /MPPT IC/+Y_MPPT/VCC2P5_+X: track 0.00 -> 21.7 mm, vias 0 -> 2
- net /MPPT IC/-Y_MPPT/VCC2P5_+X: track 0.00 -> 20.6 mm, vias 0 -> 2
- net /MPPT IC/-X_MPPT/VCC2P5_+X: track 0.00 -> 19.0 mm, vias 0 -> 2
- net /MPPT IC/+X_MPPT/VCC2P5_+X: track 0.00 -> 19.0 mm, vias 0 -> 2
- net GND: track 0.00 -> 18.0 mm, vias 0 -> 88
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- added copper zone on F.Cu, net +3.3V
- added copper zone on F.Cu, net /3.3V Logic/Solar_+X
- added copper zone on F.Cu, net /MPPT IC/+X_MPPT/VOUT_+X
- added copper zone on F.Cu, net /MPPT IC/+Y_MPPT/VOUT_+X
- added copper zone on F.Cu, net /MPPT IC/-X_MPPT/VOUT_+X
- added copper zone on F.Cu, net /MPPT IC/-Y_MPPT/VOUT_+X
- added copper zone on F.Cu, net /MPPT IC/SOLAR_+Y
- added copper zone on F.Cu, net /MPPT IC/SOLAR_-X
- added copper zone on F.Cu, net /MPPT IC/SOLAR_-Y
- added copper zone on F.Cu, net BATT
- added copper zone on In2.Cu, net BATT
- added copper zone on F.Cu, net GND
- added copper zone on F.Cu, net Net-(C57-Pad1)
- added copper zone on F.Cu, net Net-(C68-Pad1)
- added copper zone on F.Cu, net Net-(C79-Pad1)
- added copper zone on F.Cu, net Net-(C90-Pad1)
- added copper zone on F.Cu, net Net-(U15-CLP)
- added copper zone on F.Cu, net Net-(U15-CSP)
- added copper zone on F.Cu, net Net-(U15-SW)
- added copper zone on F.Cu, net Net-(U16-CLP)
- added copper zone on F.Cu, net Net-(U16-CSP)
- added copper zone on F.Cu, net Net-(U16-SW)
- added copper zone on F.Cu, net Net-(U17-CLP)
- added copper zone on F.Cu, net Net-(U17-CSP)
- added copper zone on F.Cu, net Net-(U17-SW)
- added copper zone on F.Cu, net Net-(U18-CLP)
- added copper zone on F.Cu, net Net-(U18-CSP)
- added copper zone on F.Cu, net Net-(U18-SW)
