File: EPS_mppt_board.kicad_pcb (KiCad board)
At the start: 6 copper layers, 90.2 x 95.9 mm, 284 parts, among them J1 Conn_01x04_Pin, J2 M80-5400642, J3 M80-5400642, J4 M80-5400642, J5 M80-5400642, J6 ESQ-126-39-G-D, J7 ESQ-126-39-G-D, Q1 SIR5607DP-T1-RE3, Q10 Q_NMOS, Q11 Q_NMOS, Q12 Q_NMOS, Q13 Q_NMOS, Q14 Q_NMOS, Q15 Q_NMOS, Q2 SIR5607DP-T1-RE3, Q3 SIR5607DP-T1-RE3, Q4 SIR5607DP-T1-RE3, Q5 Q_NMOS, Q6 Q_NMOS, Q7 Q_NMOS, Q8 Q_NMOS, Q9 Q_NMOS, U1 LTC4417HUF, U10 TPS259470ARPWR, U11 TPS259470ARPWR, U12 INA3221, U13 TPS259470ARPWR, U14 LTC3633AIUFDPBF, U15 LTC4162IUFD-LADM_PBF, U16 LTC4162IUFD-LADM_PBF, U17 LTC4162IUFD-LADM_PBF, U18 LTC4162IUFD-LADM_PBF, U2 TPS259470ARPWR, U3 TPS62177DQCR, U4 TPS3823A-33DBVR, U5 MR20H40, U6 STM32L496RGTx, U7 TCAN334GDCNT, U8 TCAN334GDCNT, U9 TCA9548AMRGER, Y1 8 MHZ Oscillator

Commit message: Efuses for this board and Battery board
Parts:
- removed the C30 at (-14.4, 69.9)
- removed JP3, JP4: S_Jumper, Jumper:SolderJumper-2_P1.3mm_Open_TrianglePad1.0x1.5mm
- removed the L1 at (-133.0, 52.5)
- removed the R29 at (-5.51, 33.7)
- removed the R30 at (-49.4, 68.6)
- removed the R31 at (-4.42, 73.6)
- removed the R32 at (-4.42, 76.1)
- removed the R33 at (-4.42, 78.6)
- removed the R34 at (-8.43, 68.6)
- removed the R35 at (-8.43, 71.1)
- removed the R36 at (-8.43, 73.6)
- removed the R37 at (-8.43, 76.1)
- removed the R38 at (-8.43, 78.6)
- added C108: 100n, Capacitor_SMD:C_0603_1608Metric, B.Cu at (159.5, 107.8)
- added C109: 100n, Capacitor_SMD:C_0603_1608Metric, B.Cu at (159.2, 110.8)
- added C110: 100n, Capacitor_SMD:C_0603_1608Metric, B.Cu at (171.2, 109.0)
- added C36: 10 uF, Capacitor_SMD:C_0603_1608Metric, B.Cu at (162.9, 139.7)
- added C58: 22uF, Capacitor_SMD:C_1210_3225Metric, F.Cu at (134.4, 96.6)
- added C60: 22uF, Capacitor_SMD:C_1210_3225Metric, F.Cu at (134.4, 103.4)
- added J8: ESQ-106-39-G-D, zLibrary:SAMTEC_ESQ-106-39-G-D, F.Cu at (150.1, 135.8)
- added R105: 33, Resistor_SMD:R_0402_1005Metric, B.Cu at (170.4, 107.7)
- added R106: 33, Resistor_SMD:R_0402_1005Metric, B.Cu at (161.3, 104.8)
- added R107: 33, Resistor_SMD:R_0402_1005Metric, B.Cu at (160.1, 109.0)
- added R108: 33, Resistor_SMD:R_0402_1005Metric, B.Cu at (159.8, 105.2)
- added R109: 33, Resistor_SMD:R_0402_1005Metric, B.Cu at (169.9, 111.1)
- added R19: 100k, Resistor_SMD:R_0603_1608Metric, F.Cu at (158.8, 96.7)
- added R20: 100k, Resistor_SMD:R_0603_1608Metric, F.Cu at (158.5, 102.0)
- added R21: 100k, Resistor_SMD:R_0603_1608Metric, F.Cu at (158.8, 95.2)
- added R22: 10k, Resistor_SMD:R_0805_2012Metric, F.Cu at (162.0, 95.8)
- added R23: 10k, Resistor_SMD:R_0805_2012Metric, F.Cu at (157.1, 90.6)
- added U19: LMK1C1106PWR, zLibrary:PW0014A-IPC_B, B.Cu at (165.4, 108.4)
- C10: value 100pF -> 2.2nF
- C11: value 1uF -> 2.2nF
- C12: value 22uF -> 100pF; footprint zLibrary:CAP_C2220C_2S_KEM-M -> Capacitor_SMD:C_0603_1608Metric
- C13: value 100nF -> 100pF
- C14, C15: value 22uF -> 10uF; footprint zLibrary:CAP_C2220C_2S_KEM-M -> Capacitor_SMD:C_1206_3216Metric
- C16, D2, JP1, Q5, Q6, Q7, U4: moved to B.Cu
- C41: renamed from C36; footprint zLibrary:CAP_C1210C_X7R_2S_FW_KEM-M -> Capacitor_SMD:C_1206_3216Metric
- C50: renamed from C45; footprint zLibrary:CAP_C1210C_X7R_2S_FW_KEM-M -> Capacitor_SMD:C_1206_3216Metric
- C54: renamed from C49; footprint zLibrary:CAP_C1210C_X7R_2S_FW_KEM-M -> Capacitor_SMD:C_1206_3216Metric
- C55: renamed from C50; footprint zLibrary:CAP_C2220C_2S_KEM-M -> Capacitor_SMD:C_1210_3225Metric
- C62: renamed from C55; footprint Capacitor_SMD:C_0603_1608Metric -> Capacitor_SMD:C_0402_1005Metric
- C63: renamed from C56; footprint zLibrary:CAP_C2220C_2S_KEM-M -> Capacitor_SMD:C_1210_3225Metric
- C7, J1: moved to F.Cu
- C9: value 2.2nF -> 100nF
- R14: value 350k -> 182k
- R15, R18: value 100k -> 20k
- R16: value 5k -> 100k
- R17: value 100k -> 182k
- R24: renamed from R19; moved to B.Cu
- U3: value TPS62177DQCR -> TPS259470ARPWR; footprint zLibrary:DQC0010A -> zLibrary:RPW0010A-MFG
- moved C14 300.8 mm to (161.8, 99.0), turned to 90 degrees
- moved C12 298.9 mm to (158.1, 98.4)
- moved C15 298.0 mm to (161.8, 92.1), turned to 90 degrees
- moved C13 282.9 mm to (159.1, 92.3)
- moved U3 280.6 mm to (155.6, 94.2), turned to 90 degrees
- moved C11 278.9 mm to (154.7, 91.1), turned to 90 degrees
- moved R15 277.7 mm to (154.0, 104.2)
- moved R16 277.5 mm to (157.0, 104.2)
- moved U2 277.5 mm to (155.6, 100.8), turned to 90 degrees
- moved C9 275.5 mm to (153.1, 93.0), turned to 90 degrees
- moved R18 275.0 mm to (155.7, 96.8)
- moved R17 274.0 mm to (153.1, 96.0), turned to -90 degrees
- moved R14 273.3 mm to (151.8, 103.5), turned to -90 degrees
- moved C16 272.4 mm to (183.2, 85.5)
- moved R24 268.6 mm to (179.4, 82.6), turned to 180 degrees
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- renumbered C93 to C100, C94 to C101, C95 to C102, C96 to C103, C97 to C104, C98 to C105, C99 to C106, C100 to C107, C104 to C17, C101 to C18, C102 to C19, C103 to C20, C105 to C21, C17 to C22, C18 to C23, C19 to C24, C20 to C25, C21 to C26, C22 to C27, C23 to C28, C24 to C29, C25 to C30, C26 to C32, C27 to C33, C28 to C34, C29 to C35, C32 to C37, C33 to C38, C34 to C39, C35 to C40, C37 to C42, C38 to C43, C39 to C44, C40 to C45, C41 to C46, C42 to C47, C43 to C48, C44 to C49, C46 to C51, C47 to C52, C48 to C53, C51 to C56, C52 to C57, C53 to C59, C54 to C61, C57 to C64, C58 to C65, C59 to C66, C60 to C67, C61 to C68, C62 to C69, C63 to C70, C64 to C71, C65 to C72, C66 to C73, C67 to C74, C68 to C75, C69 to C76, C70 to C77, C71 to C78, C72 to C79, C73 to C80, C74 to C81, C75 to C82, C76 to C83, C77 to C84, C78 to C85, C79 to C86, C80 to C87, C81 to C88, C82 to C89, C83 to C90, C84 to C91, C85 to C92, C86 to C93, C87 to C94, C88 to C95, C89 to C96, C90 to C97, C91 to C98, C92 to C99, D6 to D10, D7 to D11, D8 to D12, D9 to D13, D10 to D3, D11 to D4, D12 to D5, D13 to D6, D3 to D7, D4 to D8, D5 to D9, J5 to J3, J3 to J5, L2 to L1, L3 to L2, L4 to L3, L5 to L4, L6 to L5, L7 to L6, R105 to R100, R106 to R101, R107 to R102, R108 to R103, R109 to R104, R20 to R25, R21 to R26, R22 to R27, R23 to R28, R24 to R29, R25 to R30, R26 to R31, R27 to R32, R28 to R33, R39 to R34, R40 to R35, R41 to R36, R42 to R37, R43 to R38, R44 to R39, R45 to R40, R46 to R41, R47 to R42, R48 to R43, R49 to R44, R50 to R45, R51 to R46, R52 to R47, R53 to R48, R54 to R49, R55 to R50, R56 to R51, R57 to R52, R58 to R53, R59 to R54, R60 to R55, R61 to R56, R62 to R57, R63 to R58, R64 to R59, R65 to R60, R66 to R61, R67 to R62, R68 to R63, R69 to R64, R70 to R65, R71 to R66, R72 to R67, R73 to R68, R74 to R69, R75 to R70, R76 to R71, R77 to R72, R78 to R73, R79 to R74, R80 to R75, R81 to R76, R82 to R77, R83 to R78, R84 to R79, R85 to R80, R86 to R81, R87 to R82, R88 to R83, R89 to R84, R90 to R85, R91 to R86, R92 to R87, R93 to R88, R94 to R89, R95 to R90, R96 to R91, R97 to R92, R98 to R93, R99 to R94, R100 to R95, R101 to R96, R102 to R97, R103 to R98, R104 to R99
Connections:
- C10 pad 1: Net-(U2-dVdt) -> Net-(U2-ITIMER)
- C105 pad 2: BATT -> BATT_2
- C11 pad 1: Net-(U2-OUT) -> Net-(U3-ITIMER)
- C12 pad 1: Net-(U2-OUT) -> Net-(U2-dVdt)
- C13 pad 1: Net-(U2-OUT) -> Net-(U3-dVdt)
- C14 pad 1: +3.3V -> /3.3V Logic/3V3_Out_Batt
- C17 pad 1: BATT -> BATT_2
- C18 pad 1: BATT -> BATT_1
- C19 pad 1: BATT -> BATT_2
- C20 pad 1: BATT -> BATT_1
- C31 pad 1: +3.3V -> GND
- C31 pad 2: GND -> Net-(U6-NRST)
- C55 pad 1: /3.3V and 5V Line/3.3V_Line -> /3.3V Logic/3V3_In
- C56 pad 2: GNDS -> GND
- C6 pad 1: Net-(Q1-D) -> /3.3V Logic/VIN_Out
- C7 pad 1: Net-(Q1-D) -> /3.3V Logic/VIN_Out
- C72 pad 2: BATT -> BATT_1
- C8 pad 1: Net-(Q1-D) -> /3.3V Logic/3V3_In
- C83 pad 2: BATT -> BATT_1
- C9 pad 1: Net-(U2-ITIMER) -> /3.3V Logic/3V3_In
- C94 pad 2: BATT -> BATT_2
- L1 pad 1: /3.3V and 5V Line/3.3V_Line -> /3.3V Logic/3V3_In
- Q1 pad 5: Net-(Q1-D) -> /3.3V Logic/VIN_Out
- Q4 pad 5: Net-(Q1-D) -> /3.3V Logic/VIN_Out
- R103 pad 2: BATT -> BATT_2
- R14 pad 1: Net-(Q1-D) -> /3.3V Logic/3V3_In
- R15 pad 1: +3.3V -> Net-(U2-EN_UVLO)
- R15 pad 2: Net-(U2-!FLT) -> Net-(U2-OVLO)
- R16 pad 1: Net-(U2-ILM) -> Net-(U2-OVLO)
- R17 pad 1: +3.3V -> /3.3V Logic/3V3_In
- R17 pad 2: Net-(U2-AUXOFF) -> Net-(U3-EN_UVLO)
- R18 pad 1: +3.3V -> Net-(U3-EN_UVLO)
- R18 pad 2: Net-(U3-PG) -> Net-(U3-OVLO)
- R40 pad 1: /3.3V and 5V Line/3.3V_Line -> /3.3V Logic/3V3_In
- R41 pad 1: /3.3V and 5V Line/3.3V_Line -> /3.3V Logic/3V3_In
- R45 pad 1: /3.3V and 5V Line/3.3V_Line -> /3.3V Logic/3V3_In
- R49 pad 1: /3.3V and 5V Line/3.3V_Line -> /3.3V Logic/3V3_In
- R66 pad 1: /3.3V and 5V Line/3.3V_Line -> /3.3V Logic/3V3_In
- R67 pad 2: GNDS -> GND
- R68 pad 2: GNDS -> GND
- R72 pad 2: GNDS -> GND
- R79 pad 2: BATT -> BATT_1
- R87 pad 2: BATT -> BATT_1
- R95 pad 2: BATT -> BATT_2
- U1 pad 12: Net-(Q1-D) -> /3.3V Logic/VIN_Out
- U14 pad 12: /3.3V and 5V Line/3.3V_Line -> /3.3V Logic/3V3_In
- U14 pad 15: BATT -> /3.3V Logic/VIN_Out
- U14 pad 16: BATT -> /3.3V Logic/VIN_Out
- U14 pad 21: BATT -> /3.3V Logic/VIN_Out
- U14 pad 22: BATT -> /3.3V Logic/VIN_Out
- U14 pad 3: BATT -> /3.3V Logic/VIN_Out
- U14 pad 6: BATT -> /3.3V Logic/VIN_Out
- U14 pad 7: GNDS -> GND
- U15 pad 16: /3.3V and 5V Line/SYNC -> /MPPT IC/MPPT_SYNC_1.5MHz_1
- U15 pad 20: BATT -> BATT_1
- U16 pad 16: /3.3V and 5V Line/SYNC -> /MPPT IC/MPPT_SYNC_1.5MHz_3
- U16 pad 20: BATT -> BATT_1
- U17 pad 16: /3.3V and 5V Line/SYNC -> /MPPT IC/MPPT_SYNC_1.5MHz_2
- U17 pad 20: BATT -> BATT_2
- U18 pad 16: /3.3V and 5V Line/SYNC -> /MPPT IC/MPPT_SYNC_1.5MHz_4
- U18 pad 20: BATT -> BATT_2
- U2 pad 2: GND -> Net-(U2-OVLO)
- U2 pad 3: Net-(U2-AUXOFF) -> GND
- U2 pad 5: Net-(Q1-D) -> /3.3V Logic/3V3_In
- U2 pad 6: Net-(U2-OUT) -> /3.3V Logic/3V3_Out_Batt
- U3 pad 1: GND -> Net-(U3-EN_UVLO)
- U3 pad 10: +3.3V -> Net-(U3-ITIMER)
- U3 pad 2: Net-(U2-OUT) -> Net-(U3-OVLO)
- U3 pad 3: Net-(U2-OUT) -> GND
- U3 pad 4: GND -> Net-(U3-!FLT)
- U3 pad 5: GND -> /3.3V Logic/3V3_In
- U3 pad 6: GND -> +3.3V
- U3 pad 7: Net-(U3-PG) -> Net-(U3-dVdt)
- U3 pad 8: +3.3V -> GND
- U6 pad 21: /3.3V and 5V Line/SYNC -> unconnected-(U6-PA5-Pad21)
- U6 pad 37: unconnected-(U6-PC6-Pad37) -> /STM32L4/MPPT_SYNC
Routing:
- net /MPPT IC/MPPT_SYNC_1.5MHz_2: track 0.00 -> 85.4 mm, vias 0 -> 1
- net GND: track 18.0 -> 96.3 mm, vias 108 -> 199
- net BATT: track 72.1 -> 0.00 mm, vias 58 -> 0
- net /Current Sensing and Fault Detection/OBC_3V3_ShutDown: track 0.00 -> 69.3 mm, vias 0 -> 2
- net /MPPT IC/!SMB_ALERT_-X: track 9.01 -> 73.2 mm, vias 0 -> 5
- net /3.3V Logic/!VAL1: track 0.00 -> 60.7 mm, vias 0 -> 2
- net /3.3V Logic/!VAL2: track 0.00 -> 52.8 mm, vias 0 -> 4
- net /Current Sensing and Fault Detection/PV_INA3221: track 0.00 -> 52.6 mm, vias 0 -> 5
- net /3.3V and 5V Line/PGOOD2: track 0.00 -> 47.4 mm, vias 0 -> 3
- net /3.3V Logic/VIN_Out: track 0.00 -> 44.5 mm, vias 0 -> 11
- net /STM32L4/C_SHDN2: track 0.00 -> 44.3 mm, vias 0 -> 4
- net /I2C Mux/SCL_-Y: track 7.46 -> 51.1 mm, vias 1 -> 4
- net /3.3V and 5V Line/PGOOD1: track 0.00 -> 43.2 mm, vias 0 -> 3
- net /MPPT IC/!SMB_ALERT_+Y: track 9.01 -> 51.4 mm, vias 0 -> 2
- net /3.3V and 5V Line/SYNC: track 0.00 -> 38.1 mm, vias 0 -> 2
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- added copper zone on B.Cu, net +3.3V
- added copper zone on In3.Cu, net +3.3V
- added copper zone on B.Cu, net /3.3V Logic/3V3_In
- added copper zone on F.Cu, net /3.3V Logic/3V3_In
- added copper zone on In2.Cu, net /3.3V Logic/3V3_In
- added copper zone on F.Cu, net /3.3V Logic/3V3_Out_Batt
- added copper zone on B.Cu, net /3.3V Logic/VIN_Out
- added copper zone on F.Cu, net /3.3V Logic/VIN_Out
- added copper zone on F.Cu, net /3.3V and 5V Line/5V_Line
- added copper zone on F.Cu, net /3.3V and 5V Line/INTVCC
- added copper zone on F.Cu, net /3.3V and 5V Line/SW2
- added copper zone on B.Cu, net /Current Sensing and Fault Detection/ADCS_5V
- added copper zone on B.Cu, net /Current Sensing and Fault Detection/OBC_3V3
- added copper zone on F.Cu, net BATT_1
- added copper zone on In2.Cu, net BATT_1
- added copper zone on F.Cu, net BATT_2
- added copper zone on In2.Cu, net BATT_2
- added copper zone on B.Cu, net GND
- added copper zone on B.Cu, net Net-(U1-VS1)
- added copper zone on B.Cu, net Net-(U10-EN_UVLO)
- added copper zone on In3.Cu, net Net-(U10-EN_UVLO)
- added copper zone on F.Cu, net Net-(U14-BOOST1)
- added copper zone on F.Cu, net Net-(U14-BOOST2)
- added copper zone on F.Cu, net Net-(U14-SW1)
- removed copper zone on F.Cu, net BATT
- removed copper zone on In2.Cu, net BATT
Other:
- board text added: "C38"
- board text added: "C39"
- board text added: "C40"
- board text added: "C43"
- board text added: "C44"
- board text added: "R45"
- board text added: "R46"
- board text added: "R47"
- board text added: "R48"
- board text added: "R50"
- board text added: "R54"
- board text added: "R55"
- board text added: "R56"
- board text added: "R57"
- board text added: "U12"

Commit message: Mostly done routing, still yet to start DRC
Parts:
- added R110: 10k, Resistor_SMD:R_0603_1608Metric, B.Cu at (174.6, 106.7)
- moved C34 56.4 mm to (123.7, 67.5)
- moved R30 56.4 mm to (119.4, 62.5)
- moved U7 56.4 mm to (120.8, 66.1)
- moved U8 56.4 mm to (113.8, 66.0)
- moved C35 56.4 mm to (116.7, 67.4)
- moved R31 56.0 mm to (113.6, 62.3)
- moved C36 30.3 mm to (135.9, 125.9)
- moved U9 27.8 mm to (142.6, 123.2)
- moved C37 27.4 mm to (138.9, 122.9), turned to 90 degrees
- moved C24 7.08 mm to (169.0, 77.8), turned to -90 degrees
- moved R65 6.14 mm to (149.0, 76.3), turned to 180 degrees
- moved R81 4.72 mm to (177.2, 72.8)
- moved R1 3.45 mm to (108.5, 98.1)
- moved D1 3.21 mm to (121.1, 108.4)
- moved C23 2.24 mm to (173.1, 98.6)
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Connections:
- J6 pad 01: unconnected-(J6-Pad01) -> /PC104/CAN2-
- J6 pad 02: unconnected-(J6-Pad02) -> /PC104/CAN-
- J6 pad 03: unconnected-(J6-Pad03) -> /PC104/CAN2+
- J6 pad 04: unconnected-(J6-Pad04) -> /PC104/CAN+
- J6 pad 25: unconnected-(J6-Pad25) -> GND
- J6 pad 26: unconnected-(J6-Pad26) -> GND
- J6 pad 27: unconnected-(J6-Pad27) -> /Current Sensing and Fault Detection/OBC_3V3_Line_Out
- J6 pad 28: unconnected-(J6-Pad28) -> /Current Sensing and Fault Detection/OBC_3V3_Line_Out
- J6 pad 29: unconnected-(J6-Pad29) -> GND
- J6 pad 30: unconnected-(J6-Pad30) -> GND
- J6 pad 31: unconnected-(J6-Pad31) -> /Current Sensing and Fault Detection/ADCS_3V3_Line_Out
- J6 pad 32: unconnected-(J6-Pad32) -> /Current Sensing and Fault Detection/ADCS_3V3_Line_Out
- J6 pad 33: unconnected-(J6-Pad33) -> GND
- J6 pad 34: unconnected-(J6-Pad34) -> GND
- J6 pad 35: unconnected-(J6-Pad35) -> /Current Sensing and Fault Detection/ADCS_5V_Line_Out
- J6 pad 36: unconnected-(J6-Pad36) -> /Current Sensing and Fault Detection/ADCS_5V_Line_Out
- J6 pad 37: unconnected-(J6-Pad37) -> GND
- J6 pad 38: unconnected-(J6-Pad38) -> GND
- J6 pad 41: unconnected-(J6-Pad41) -> GND
- J6 pad 45: unconnected-(J6-Pad45) -> GND
- J6 pad 46: unconnected-(J6-Pad46) -> GND
- J6 pad 47: unconnected-(J6-Pad47) -> /3.3V Logic/3V3_Out_Batt
- J6 pad 48: unconnected-(J6-Pad48) -> /3.3V Logic/3V3_Out_Batt
- J6 pad 49: unconnected-(J6-Pad49) -> GND
- J6 pad 50: unconnected-(J6-Pad50) -> GND
- J6 pad 51: unconnected-(J6-Pad51) -> GND
- J6 pad 52: unconnected-(J6-Pad52) -> GND
- J7 pad 33: unconnected-(J7-Pad33) -> BATT
- J7 pad 34: unconnected-(J7-Pad34) -> BATT
- U19 pad 2: +3.3V -> Net-(U19-1G)
- U7 pad 7: /PC104/CAN2+ -> /PC104/CAN+
- U8 pad 7: /PC104/CAN+ -> /PC104/CAN2+
- U9 pad 16: unconnected-(U9-SD7-Pad16) -> /I2C Mux/SDA_-X
- U9 pad 17: unconnected-(U9-SC7-Pad17) -> /I2C Mux/SCL_-X
- U9 pad 3: /I2C Mux/SDA_-X -> unconnected-(U9-SD1-Pad3)
- U9 pad 4: /I2C Mux/SCL_-X -> unconnected-(U9-SC1-Pad4)
Routing:
- net /I2C Mux/I2C_Reset: track 0.00 -> 136.7 mm, vias 0 -> 8
- net /Current Sensing and Fault Detection/SDA_INA3221: track 8.03 -> 132.1 mm, vias 2 -> 5
- net /I2C Mux/SCL_+Y: track 7.46 -> 131.1 mm, vias 1 -> 7
- net /STM32L4/C_SHDN: track 5.15 -> 115.8 mm, vias 1 -> 4
- net /I2C Mux/SCL_+X: track 7.46 -> 104.5 mm, vias 1 -> 3
- net /STM32L4/C_SHDN2: track 44.3 -> 135.3 mm, vias 4 -> 2
- net /Current Sensing and Fault Detection/ADCS_3V3_ShutDown: track 1.55 -> 89.2 mm, vias 1 -> 4
- net /STM32L4/CANTX2: track 0.00 -> 82.9 mm, vias 0 -> 2
- net /STM32L4/CANRX2: track 0.00 -> 80.4 mm, vias 0 -> 2
- net /Current Sensing and Fault Detection/SCL_INA3221: track 9.37 -> 87.4 mm, vias 2 -> 6
- net /I2C Mux/SDA_+X: track 5.88 -> 81.6 mm, vias 1 -> 3
- net /STM32L4/CANRX: track 0.00 -> 72.7 mm, vias 0 -> 2
- net /STM32L4/CANTX: track 0.00 -> 72.7 mm, vias 0 -> 2
- net GND: track 96.3 -> 168.1 mm, vias 199 -> 251
- net /I2C Mux/SDA_+Y: track 5.88 -> 77.2 mm, vias 1 -> 4
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- added copper zone on In2.Cu, net +3.3V
- added copper zone on In2.Cu, net /3.3V Logic/3V3_Out_Batt
- added copper zone on B.Cu, net /3.3V and 5V Line/5V_Line
- added copper zone on In2.Cu, net /3.3V and 5V Line/5V_Line
- added copper zone on B.Cu, net /Current Sensing and Fault Detection/ADCS_3V3
- added copper zone on B.Cu, net /Current Sensing and Fault Detection/ADCS_3V3_Line_Out
- added copper zone on In2.Cu, net /Current Sensing and Fault Detection/ADCS_3V3_Line_Out
- added copper zone on B.Cu, net /Current Sensing and Fault Detection/ADCS_5V_Line_Out
- added copper zone on B.Cu, net /Current Sensing and Fault Detection/OBC_3V3_Line_Out
- added copper zone on In2.Cu, net /Current Sensing and Fault Detection/OBC_3V3_Line_Out
- added copper zone on B.Cu, net BATT
- added copper zone on B.Cu, net Net-(U1-VS2)
- added copper zone on B.Cu, net Net-(U13-EN_UVLO)
Other:
- outline, holes or cut-outs redrawn
- board text added: "(If It Works)"
- board text added: "3V3"
- board text added: "Designed By: Jaron Cyna"
- board text added: "GND"
- board text added: "SWCLK"
- board text added: "SWDIO"
- board text added: "Stegosaurus"
