File: EPS_mppt_board.kicad_pcb (KiCad board)
At the start: 6 copper layers, 90.2 x 95.9 mm, 287 parts, among them J1 Conn_01x04_Pin, J2 M80-5400642, J3 M80-5400642, J4 M80-5400642, J5 M80-5400642, J6 ESQ-126-39-G-D, J7 ESQ-126-39-G-D, J8 ESQ-106-39-G-D, Q1 SIR5607DP-T1-RE3, Q10 Q_NMOS, Q11 Q_NMOS, Q12 Q_NMOS, Q13 Q_NMOS, Q14 Q_NMOS, Q15 Q_NMOS, Q2 SIR5607DP-T1-RE3, Q3 SIR5607DP-T1-RE3, Q4 SIR5607DP-T1-RE3, Q5 Q_NMOS, Q6 Q_NMOS, Q7 Q_NMOS, Q8 Q_NMOS, Q9 Q_NMOS, U1 LTC4417HUF, U10 TPS259470ARPWR, U11 TPS259470ARPWR, U12 INA3221, U13 TPS259470ARPWR, U14 LTC3633AIUFDPBF, U15 LTC4162IUFD-LADM_PBF, U16 LTC4162IUFD-LADM_PBF, U17 LTC4162IUFD-LADM_PBF, U18 LTC4162IUFD-LADM_PBF, U19 LMK1C1106PWR, U2 TPS259470ARPWR, U20 TCAN337G, U21 TCAN337G, U3 TPS259470ARPWR, U4 TPS3823A-33DBVR, U5 MR20H40, U6 STM32L496RGTx, U9 TCA9548AMRGER, Y1 8 MHZ Oscillator

Commit message: Added Batt 1 and Batt 2 charging
Parts:
- moved R83 0.29 mm to (156.5, 63.3)
- moved R82 0.29 mm to (156.2, 64.8)
- moved R84 0.29 mm to (156.9, 61.8)
Connections:
- net /3.3V Logic/!VAL1 renamed /EPS Logic/!VAL1
- net /3.3V Logic/!VAL2 renamed /EPS Logic/!VAL2
- net /3.3V Logic/!VAL3 renamed /EPS Logic/!VAL3
- net /3.3V Logic/3V3_In renamed /3.3V and 5V Line/3.3V_Line
- net /3.3V Logic/3V3_Out_Batt renamed /EPS Logic/3V3_Out_Batt
- net /3.3V Logic/OR'd_VOUT renamed /EPS Logic/OR'd_VOUT
- net /3.3V Logic/OV1 renamed /EPS Logic/OV1
- net /3.3V Logic/OV2 renamed /EPS Logic/OV2
- net /3.3V Logic/OV3 renamed /EPS Logic/OV3
- net /3.3V Logic/UV1 renamed /EPS Logic/UV1
- net /3.3V Logic/UV2 renamed /EPS Logic/UV2
- net /3.3V Logic/UV3 renamed /EPS Logic/UV3
- net /3.3V Logic/VIN_Out renamed /3.3V and 5V Line/Battery_V_in1
- J6 pad 39: unconnected-(J6-Pad39) -> BATT_1
- J6 pad 40: unconnected-(J6-Pad40) -> BATT_1
- J7 pad 37: unconnected-(J7-Pad37) -> BATT_2
- J7 pad 38: unconnected-(J7-Pad38) -> BATT_2
Routing:
- net Net-(Q15-G): track 26.8 -> 23.4 mm
- net /STM32L4/C_S1: track 73.0 -> 74.2 mm
- net Net-(U17-SW): track 6.53 -> 5.71 mm
- net /I2C Mux/I2C_Reset: track 131.1 -> 130.5 mm
- net +3.3V: track 135.8 -> 135.9 mm, vias 61 -> 65
- net BATT_2: vias 15 -> 25
- added copper zone on In3.Cu, net BATT_1
- added copper zone on B.Cu, net BATT_2
- removed copper zone on In2.Cu, net BATT_1
