File: External Watchdog IC.kicad_sch (KiCad schematic)
At the start: 5 parts, among them U4 TPS3823A-33DBVR

Commit message: Started PCB layout
Parts:
- renumbered C15 to C16, D10 to D2
Changed lines of the file:
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@@
 		(dnp no)
 		(fields_autoplaced yes)
-		(property "Reference" "#PWR030"
+		(property "Reference" "#PWR031"
 			(at 54.61 74.93 0)
 			(effects
@@
 			(project ""
 				(path "/8f246f89-1ec7-4136-9977-839b50e116ed/61eb8b07-a516-4600-8bd8-c85438ae98cc"
-					(reference "#PWR030")
+					(reference "#PWR031")
 					(unit 1)
 				)
@@
 		(on_board yes)
 		(dnp no)
-		(property "Reference" "C15"
+		(property "Reference" "C16"
 			(at 47.498 64.77 0)
 			(effects
@@
 			(project ""
 				(path "/8f246f89-1ec7-4136-9977-839b50e116ed/61eb8b07-a516-4600-8bd8-c85438ae98cc"
-					(reference "C15")
+					(reference "C16")
 					(unit 1)
 				)
@@
 		(dnp no)
 		(fields_autoplaced yes)
-		(property "Reference" "#PWR032"
+		(property "Reference" "#PWR033"
 			(at 68.58 62.23 0)
 			(effects
@@
 			(project ""
 				(path "/8f246f89-1ec7-4136-9977-839b50e116ed/61eb8b07-a516-4600-8bd8-c85438ae98cc"
-					(reference "#PWR032")
+					(reference "#PWR033")
 					(unit 1)
 				)
@@
 		(dnp no)
 		(fields_autoplaced yes)
-		(property "Reference" "#PWR031"
+		(property "Reference" "#PWR032"
 			(at 64.77 77.47 0)
 			(effects
@@
 			(project "EPS_mppt_board"
 				(path "/8f246f89-1ec7-4136-9977-839b50e116ed/61eb8b07-a516-4600-8bd8-c85438ae98cc"
-					(reference "#PWR031")
+					(reference "#PWR032")
 					(unit 1)
 				)
@@
 		(dnp no)
 		(fields_autoplaced yes)
-		(property "Reference" "D10"
+		(property "Reference" "D2"
 			(at 155.8925 54.61 0)
 			(effects
@@
 			(project ""
 				(path "/8f246f89-1ec7-4136-9977-839b50e116ed/61eb8b07-a516-4600-8bd8-c85438ae98cc"
-					(reference "D10")
+					(reference "D2")
 					(unit 1)
 				)
@@
 		(dnp no)
 		(fields_autoplaced yes)
-		(property "Reference" "#PWR034"
+		(property "Reference" "#PWR035"
 			(at 140.97 63.5 0)
 			(effects
@@
 			(project "EPS_mppt_board"
 				(path "/8f246f89-1ec7-4136-9977-839b50e116ed/61eb8b07-a516-4600-8bd8-c85438ae98cc"
-					(reference "#PWR034")
+					(reference "#PWR035")
 					(unit 1)
 				)
@@
 		(on_board yes)
 		(dnp no)
-		(property "Reference" "#PWR033"
+		(property "Reference" "#PWR034"
 			(at 71.12 92.71 0)
 			(effects
@@
 			(project "EPS_mppt_board"
 				(path "/8f246f89-1ec7-4136-9977-839b50e116ed/61eb8b07-a516-4600-8bd8-c85438ae98cc"
-					(reference "#PWR033")
-					(unit 1)
-				)
+					(reference "#PWR034")
+					(unit 1)
+				)
