File: External Watchdog IC.kicad_sch (KiCad schematic)
At the start: 5 parts, among them U4 TPS3823A-33DBVR

Commit message: Efuses for this board and Battery board
Parts:
- renumbered R19 to R24
Changed lines of the file:
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@@
 		(dnp no)
 		(fields_autoplaced yes)
-		(property "Reference" "#PWR031"
+		(property "Reference" "#PWR036"
 			(at 54.61 74.93 0)
 			(effects
@@
 			(project ""
 				(path "/8f246f89-1ec7-4136-9977-839b50e116ed/61eb8b07-a516-4600-8bd8-c85438ae98cc"
-					(reference "#PWR031")
+					(reference "#PWR036")
 					(unit 1)
 				)
@@
 		(dnp no)
 		(fields_autoplaced yes)
-		(property "Reference" "R19"
+		(property "Reference" "R24"
 			(at 66.04 71.12 90)
 			(effects
@@
 			(project "EPS_mppt_board"
 				(path "/8f246f89-1ec7-4136-9977-839b50e116ed/61eb8b07-a516-4600-8bd8-c85438ae98cc"
-					(reference "R19")
+					(reference "R24")
 					(unit 1)
 				)
@@
 		(dnp no)
 		(fields_autoplaced yes)
-		(property "Reference" "#PWR033"
+		(property "Reference" "#PWR038"
 			(at 68.58 62.23 0)
 			(effects
@@
 			(project ""
 				(path "/8f246f89-1ec7-4136-9977-839b50e116ed/61eb8b07-a516-4600-8bd8-c85438ae98cc"
-					(reference "#PWR033")
+					(reference "#PWR038")
 					(unit 1)
 				)
@@
 		(dnp no)
 		(fields_autoplaced yes)
-		(property "Reference" "#PWR032"
+		(property "Reference" "#PWR037"
 			(at 64.77 77.47 0)
 			(effects
@@
 			(project "EPS_mppt_board"
 				(path "/8f246f89-1ec7-4136-9977-839b50e116ed/61eb8b07-a516-4600-8bd8-c85438ae98cc"
-					(reference "#PWR032")
+					(reference "#PWR037")
 					(unit 1)
 				)
@@
 		(dnp no)
 		(fields_autoplaced yes)
-		(property "Reference" "#PWR035"
+		(property "Reference" "#PWR040"
 			(at 140.97 63.5 0)
 			(effects
@@
 			(project "EPS_mppt_board"
 				(path "/8f246f89-1ec7-4136-9977-839b50e116ed/61eb8b07-a516-4600-8bd8-c85438ae98cc"
-					(reference "#PWR035")
+					(reference "#PWR040")
 					(unit 1)
 				)
@@
 		(on_board yes)
 		(dnp no)
-		(property "Reference" "#PWR034"
+		(property "Reference" "#PWR039"
 			(at 71.12 92.71 0)
 			(effects
@@
 			(project "EPS_mppt_board"
 				(path "/8f246f89-1ec7-4136-9977-839b50e116ed/61eb8b07-a516-4600-8bd8-c85438ae98cc"
-					(reference "#PWR034")
-					(unit 1)
-				)
+					(reference "#PWR039")
+					(unit 1)
+				)
