File: MPPT_IC.kicad_sch (KiCad schematic)
At the start: 93 parts, among them Q10 NMOS, Q3 NMOS, Q4 NMOS, Q5 NMOS, Q6 NMOS, Q7 NMOS, Q8 NMOS, Q9 NMOS, U6 LTC4162IUFD-LADM_PBF, U7 LTC4162IUFD-LADM_PBF, U8 LTC4162IUFD-LADM_PBF, U9 LTC4162IUFD-LADM_PBF

Commit message: Added footprints to caps
Parts:
- removed C11, C23, C32, C33, C41, C42, C43: 47 uF, symbol Device:C
- added C30, C39: 100uF, Capacitor_Tantalum_SMD:CP_EIA-7361-38_AVX-V, symbol Device:C
- added C40: 22 uF, Capacitor_SMD:C_1210_3225Metric, symbol Device:C
- C10: renamed from C9; value 0.1 uF -> 100n; footprint (none) -> Capacitor_SMD:C_0603_1608Metric
- C11: renamed from C10; footprint (none) -> Capacitor_SMD:C_0402_1005Metric; MANUFACTURER (none) -> DigiKey; MANUFACTURER_PART_NUMBER (none) -> CL05B223KP5NNNC
- C12, C21: value 47 uF -> 100uF; footprint (none) -> Capacitor_Tantalum_SMD:CP_EIA-7361-38_AVX-V; MANUFACTURER (none) -> DigiKey; MANUFACTURER_PART_NUMBER (none) -> T52M9107M035C0055
- C13, C22, C31: value 47 uF -> 22 uF; footprint (none) -> Capacitor_SMD:C_1210_3225Metric; MANUFACTURER (none) -> DigiKey; MANUFACTURER_PART_NUMBER (none) -> CL32B226KAJNFNE
- C14, C17: footprint (none) -> Capacitor_SMD:C_1206_3216Metric; MANUFACTURER (none) -> DigiKey; MANUFACTURER_PART_NUMBER (none) -> CL31B106KAHNFNE
- C15: footprint (none) -> Capacitor_SMD:C_0603_1608Metric; MANUFACTURER (none) -> DigiKey; MANUFACTURER_PART_NUMBER (none) -> CL10B105KQ8NNNC
- C16: footprint (none) -> Capacitor_SMD:C_0603_1608Metric; MANUFACTURER (none) -> DigiKey; MANUFACTURER_PART_NUMBER (none) -> CL10B475KQ8NQNC
- C18, C19: value 0.1 uF -> 100n; footprint (none) -> Capacitor_SMD:C_0603_1608Metric
- C20: footprint (none) -> Capacitor_SMD:C_0402_1005Metric; MANUFACTURER (none) -> DigiKey; MANUFACTURER_PART_NUMBER (none) -> CL05B223KP5NNNC
- C23: renamed from C24; footprint (none) -> Capacitor_SMD:C_1206_3216Metric; MANUFACTURER (none) -> DigiKey; MANUFACTURER_PART_NUMBER (none) -> CL31B106KAHNFNE
- C24: renamed from C25; footprint (none) -> Capacitor_SMD:C_0603_1608Metric; MANUFACTURER (none) -> DigiKey; MANUFACTURER_PART_NUMBER (none) -> CL10B105KQ8NNNC
- C25: renamed from C26; footprint (none) -> Capacitor_SMD:C_0603_1608Metric; MANUFACTURER (none) -> DigiKey; MANUFACTURER_PART_NUMBER (none) -> CL10B475KQ8NQNC
- C26: renamed from C27; footprint (none) -> Capacitor_SMD:C_1206_3216Metric; MANUFACTURER (none) -> DigiKey; MANUFACTURER_PART_NUMBER (none) -> CL31B106KAHNFNE
- C27: renamed from C28; value 0.1 uF -> 100n; footprint (none) -> Capacitor_SMD:C_0603_1608Metric
- C28: renamed from C29; value 0.1 uF -> 100n; footprint (none) -> Capacitor_SMD:C_0603_1608Metric
- C29: renamed from C30; footprint (none) -> Capacitor_SMD:C_0402_1005Metric; MANUFACTURER (none) -> DigiKey; MANUFACTURER_PART_NUMBER (none) -> CL05B223KP5NNNC
- C32: renamed from C34; footprint (none) -> Capacitor_SMD:C_1206_3216Metric; MANUFACTURER (none) -> DigiKey; MANUFACTURER_PART_NUMBER (none) -> CL31B106KAHNFNE
- C33: renamed from C35; footprint (none) -> Capacitor_SMD:C_0603_1608Metric; MANUFACTURER (none) -> DigiKey; MANUFACTURER_PART_NUMBER (none) -> CL10B105KQ8NNNC
- C34: renamed from C36; footprint (none) -> Capacitor_SMD:C_0603_1608Metric; MANUFACTURER (none) -> DigiKey; MANUFACTURER_PART_NUMBER (none) -> CL10B475KQ8NQNC
- C35: renamed from C37; footprint (none) -> Capacitor_SMD:C_1206_3216Metric; MANUFACTURER (none) -> DigiKey; MANUFACTURER_PART_NUMBER (none) -> CL31B106KAHNFNE
- C36: renamed from C38; value 0.1 uF -> 100n; footprint (none) -> Capacitor_SMD:C_0603_1608Metric
- C37: renamed from C39; value 0.1 uF -> 100n; footprint (none) -> Capacitor_SMD:C_0603_1608Metric
- C38: renamed from C40; footprint (none) -> Capacitor_SMD:C_0402_1005Metric; MANUFACTURER (none) -> DigiKey; MANUFACTURER_PART_NUMBER (none) -> CL05B223KP5NNNC
- C41: renamed from C44; footprint (none) -> Capacitor_SMD:C_1206_3216Metric; MANUFACTURER (none) -> DigiKey; MANUFACTURER_PART_NUMBER (none) -> CL31B106KAHNFNE
- C42: renamed from C45; footprint (none) -> Capacitor_Tantalum_SMD:CP_EIA-7361-38_AVX-V; MANUFACTURER (none) -> DigiKey; MANUFACTURER_PART_NUMBER (none) -> T52M9107M035C0055
- C6: renamed from C5; footprint (none) -> Capacitor_SMD:C_0603_1608Metric; MANUFACTURER (none) -> DigiKey; MANUFACTURER_PART_NUMBER (none) -> CL10B105KQ8NNNC
- C7: renamed from C6; footprint (none) -> Capacitor_SMD:C_0603_1608Metric; MANUFACTURER (none) -> DigiKey; MANUFACTURER_PART_NUMBER (none) -> CL10B475KQ8NQNC
- C8: renamed from C7; footprint (none) -> Capacitor_SMD:C_1206_3216Metric; MANUFACTURER (none) -> DigiKey; MANUFACTURER_PART_NUMBER (none) -> CL31B106KAHNFNE
- C9: renamed from C8; value 0.1 uF -> 100n; footprint (none) -> Capacitor_SMD:C_0603_1608Metric
Connections:
- net GND: now also C30.2, C39.2, C40.2
- net at C31.1, R20.2: now also C30.1
- net at R27.2: now also C39.1, C40.1

Commit message: edited 3V3 Logic to add Efuse and UVLO
Changed lines of the file:
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@@
 		(comment 1 "Switched to IC based MPPT from a discrete one for Power and Reliabillity")
 	)
-	(rectangle
-		(start 12.7 12.7)
-		(end 284.48 100.33)
-		(stroke
-			(width 0.762)
-			(type solid)
-			(color 132 0 0 1)
-		)
-		(fill
-			(type none)
-		)
-	)
-	(rectangle
-		(start 12.7 100.33)
-		(end 284.48 189.23)
-		(stroke
-			(width 0.762)
-			(type solid)
-			(color 132 0 0 1)
-		)
-		(fill
-			(type none)
-		)
-	)
-	(rectangle
-		(start 12.7 189.23)
-		(end 284.48 278.13)
-		(stroke
-			(width 0.762)
-			(type solid)
-			(color 132 0 0 1)
-		)
-		(fill
-			(type none)
-		)
-	)
-	(rectangle
-		(start 110.49 367.03)
-		(end 176.53 407.67)
-		(stroke
-			(width 0.762)
-			(type solid)
-			(color 132 0 0 1)
-		)
-		(fill
-			(type none)
-		)
-	)
-	(rectangle
-		(start 12.7 278.13)
-		(end 284.48 367.03)
-		(stroke
-			(width 0.762)
-			(type solid)
-			(color 132 0 0 1)
-		)
-		(fill
-			(type none)
-		)
-	)
 	(text "-X MPPT"
 		(exclude_from_sim no)
@@
 		)
 	)
+	(polyline
+		(pts
+			(xy 110.49 367.03) (xy 175.26 367.03)
+		)
+		(stroke
+			(width 0.762)
+			(type dash)
+		)
+	)
 	(wire
 		(pts
@@
 		)
 	)
+	(polyline
+		(pts
+			(xy 12.7 99.06) (xy 284.48 99.06)
+		)
+		(stroke
+			(width 0.762)
+			(type dash)
+		)
+	)
 	(wire
 		(pts
@@
 		)
 	)
+	(polyline
+		(pts
+			(xy 12.7 189.23) (xy 284.48 189.23)
+		)
+		(stroke
+			(width 0.762)
+			(type dash)
+		)
+	)
 	(wire
 		(pts
@@
 		)
 	)
+	(polyline
+		(pts
+			(xy 175.26 367.03) (xy 175.26 407.67)
+		)
+		(stroke
+			(width 0.762)
+			(type dash)
+		)
+	)
 	(wire
 		(pts
@@
 		)
 	)
+	(polyline
+		(pts
+			(xy 12.7 278.13) (xy 284.48 278.13)
+		)
+		(stroke
+			(width 0.762)
+			(type dash)
+		)
+	)
 	(wire
 		(pts
@@
 					(size 1.27 1.27)
 				)
+				(hide yes)
 			)
 		)
@@
 					(size 1.27 1.27)
 				)
+				(hide yes)
 			)
 		)
@@
 					(size 1.27 1.27)
 				)
+				(hide yes)
 			)
 		)
@@
 					(size 1.27 1.27)
 				)
+				(hide yes)
 			)
 		)
@@
 					(size 1.27 1.27)
 				)
+				(hide yes)
 			)
 		)
@@
 					(size 1.27 1.27)
 				)
+				(hide yes)
 			)
 		)
@@
 					(size 1.27 1.27)
 				)
+				(hide yes)
 			)
 		)
@@
 					(size 1.27 1.27)
 				)
+				(hide yes)
 			)
 		)
@@
 					(size 1.27 1.27)
 				)
+				(hide yes)
 			)
 		)
@@
 					(size 1.27 1.27)
 				)
+				(hide yes)
 			)
 		)
@@
 					(size 1.27 1.27)
 				)
+				(hide yes)
 			)
 		)
@@
 					(size 1.27 1.27)
 				)
+				(hide yes)
 			)
 		)
@@
 					(size 1.27 1.27)
 				)
+				(hide yes)
 			)
 		)
@@
 					(size 1.27 1.27)
 				)
+				(hide yes)
 			)
 		)
@@
 					(size 1.27 1.27)
 				)
+				(hide yes)
 			)
 		)
@@
 					(size 1.27 1.27)
 				)
+				(hide yes)
 			)
 		)
@@
 					(size 1.27 1.27)
 				)
+				(hide yes)
 			)
 		)
@@
 					(size 1.27 1.27)
 				)
+				(hide yes)
 			)
 		)
@@
 					(size 1.27 1.27)
 				)
+				(hide yes)
 			)
 		)
@@
 					(size 1.27 1.27)
 				)
+				(hide yes)
 			)
 		)
@@
 					(size 1.27 1.27)
 				)
+				(hide yes)
 			)
 		)
@@
 					(size 1.27 1.27)
 				)
+				(hide yes)
 			)
 		)
@@
 					(size 1.27 1.27)
 				)
+				(hide yes)
 			)
 		)
@@
 					(size 1.27 1.27)
 				)
+				(hide yes)
 			)
 		)

Commit message: Added connectors to schematic
Parts:
- removed D3, D4, D5, D6: SMAJ15A, Diode_SMD:D_SMA, symbol Diode:SMAJ15A
- removed TH1, TH2, TH3, TH4: Beta = 3490K (10k), symbol Device:Thermistor_NTC
- added D10, D11, D12, D9: SMAJ22A, Diode_SMD:D_SMA, symbol Diode:SMAJ22A
- C16: renamed from C8; footprint Capacitor_SMD:C_1206_3216Metric -> zLibrary:CAP_C1210C_X7R_2S_FW_KEM-M; MANUFACTURER_PART_NUMBER CL31B106KAHNFNE -> C1210C106M5R2C7186
- C17: renamed from C9; MANUFACTURER (none) -> DigiKey; MANUFACTURER_PART_NUMBER (none) -> 06035C104K4T2A
- C18: renamed from C10; MANUFACTURER (none) -> DigiKey; MANUFACTURER_PART_NUMBER (none) -> 06035C104K4T2A
- C19: renamed from C11; footprint Capacitor_SMD:C_0402_1005Metric -> Capacitor_SMD:C_0603_1608Metric; MANUFACTURER_PART_NUMBER CL05B223KP5NNNC -> CGA3E2X7R1H223K080AA
- C21: renamed from C13; footprint Capacitor_SMD:C_1210_3225Metric -> zLibrary:CAP_C2220C_2S_KEM-M; MANUFACTURER_PART_NUMBER CL32B226KAJNFNE -> C2220C226MMR2L7289
- C22: renamed from C14; footprint Capacitor_SMD:C_1206_3216Metric -> zLibrary:CAP_C1210C_X7R_2S_FW_KEM-M; MANUFACTURER_PART_NUMBER CL31B106KAHNFNE -> C1210C106M5R2C7186
- C25: renamed from C17; footprint Capacitor_SMD:C_1206_3216Metric -> zLibrary:CAP_C1210C_X7R_2S_FW_KEM-M; MANUFACTURER_PART_NUMBER CL31B106KAHNFNE -> C1210C106M5R2C7186
- C26: renamed from C18; MANUFACTURER (none) -> DigiKey; MANUFACTURER_PART_NUMBER (none) -> 06035C104K4T2A
- C27: renamed from C19; MANUFACTURER (none) -> DigiKey; MANUFACTURER_PART_NUMBER (none) -> 06035C104K4T2A
- C28: renamed from C20; footprint Capacitor_SMD:C_0402_1005Metric -> Capacitor_SMD:C_0603_1608Metric; MANUFACTURER_PART_NUMBER CL05B223KP5NNNC -> CGA3E2X7R1H223K080AA
- C30: renamed from C22; footprint Capacitor_SMD:C_1210_3225Metric -> zLibrary:CAP_C2220C_2S_KEM-M; MANUFACTURER_PART_NUMBER CL32B226KAJNFNE -> C2220C226MMR2L7289
- C31: renamed from C23; footprint Capacitor_SMD:C_1206_3216Metric -> zLibrary:CAP_C1210C_X7R_2S_FW_KEM-M; MANUFACTURER_PART_NUMBER CL31B106KAHNFNE -> C1210C106M5R2C7186
- C34: renamed from C26; footprint Capacitor_SMD:C_1206_3216Metric -> zLibrary:CAP_C1210C_X7R_2S_FW_KEM-M; MANUFACTURER_PART_NUMBER CL31B106KAHNFNE -> C1210C106M5R2C7186
- C35: renamed from C27; MANUFACTURER (none) -> DigiKey; MANUFACTURER_PART_NUMBER (none) -> 06035C104K4T2A
- C36: renamed from C28; MANUFACTURER (none) -> DigiKey; MANUFACTURER_PART_NUMBER (none) -> 06035C104K4T2A
- C37: renamed from C29; footprint Capacitor_SMD:C_0402_1005Metric -> Capacitor_SMD:C_0603_1608Metric; MANUFACTURER_PART_NUMBER CL05B223KP5NNNC -> CGA3E2X7R1H223K080AA
- C39: renamed from C31; footprint Capacitor_SMD:C_1210_3225Metric -> zLibrary:CAP_C2220C_2S_KEM-M; MANUFACTURER_PART_NUMBER CL32B226KAJNFNE -> C2220C226MMR2L7289
- C40: renamed from C32; footprint Capacitor_SMD:C_1206_3216Metric -> zLibrary:CAP_C1210C_X7R_2S_FW_KEM-M; MANUFACTURER_PART_NUMBER CL31B106KAHNFNE -> C1210C106M5R2C7186
- C43: renamed from C35; footprint Capacitor_SMD:C_1206_3216Metric -> zLibrary:CAP_C1210C_X7R_2S_FW_KEM-M; MANUFACTURER_PART_NUMBER CL31B106KAHNFNE -> C1210C106M5R2C7186
- C44: renamed from C36; MANUFACTURER (none) -> DigiKey; MANUFACTURER_PART_NUMBER (none) -> 06035C104K4T2A
- C45: renamed from C37; MANUFACTURER (none) -> DigiKey; MANUFACTURER_PART_NUMBER (none) -> 06035C104K4T2A
- C46: renamed from C38; footprint Capacitor_SMD:C_0402_1005Metric -> Capacitor_SMD:C_0603_1608Metric; MANUFACTURER_PART_NUMBER CL05B223KP5NNNC -> CGA3E2X7R1H223K080AA
- C48: renamed from C40; footprint Capacitor_SMD:C_1210_3225Metric -> zLibrary:CAP_C2220C_2S_KEM-M; MANUFACTURER_PART_NUMBER CL32B226KAJNFNE -> C2220C226MMR2L7289
- C49: renamed from C41; footprint Capacitor_SMD:C_1206_3216Metric -> zLibrary:CAP_C1210C_X7R_2S_FW_KEM-M; MANUFACTURER_PART_NUMBER CL31B106KAHNFNE -> C1210C106M5R2C7186
- L2, L3, L4, L5: value 10 uH -> 4.7uH; footprint (none) -> zLibrary:IND_SRP7028A-4R7M_BRN-M; MANUFACTURER (none) -> DigiKey; MANUFACTURER_PART_NUMBER (none) -> SRP7028A-4R7M
- Q10: renamed from Q9; footprint (none) -> Package_TO_SOT_SMD:LFPAK56; MANUFACTURER_PART_NUMBER (none) -> PSMN4R0-40YS,115
- Q11: renamed from Q10; footprint (none) -> Package_TO_SOT_SMD:LFPAK56; MANUFACTURER_PART_NUMBER (none) -> PSMN4R0-40YS,115
- Q4: renamed from Q3; footprint (none) -> Package_TO_SOT_SMD:LFPAK56; MANUFACTURER_PART_NUMBER (none) -> PSMN4R0-40YS,115
- Q5: renamed from Q4; footprint (none) -> Package_TO_SOT_SMD:LFPAK56; MANUFACTURER_PART_NUMBER (none) -> PSMN4R0-40YS,115
- Q6: renamed from Q5; footprint (none) -> Package_TO_SOT_SMD:LFPAK56; MANUFACTURER_PART_NUMBER (none) -> PSMN4R0-40YS,115
- Q7: renamed from Q6; footprint (none) -> Package_TO_SOT_SMD:LFPAK56; MANUFACTURER_PART_NUMBER (none) -> PSMN4R0-40YS,115
- Q8: renamed from Q7; footprint (none) -> Package_TO_SOT_SMD:LFPAK56; MANUFACTURER_PART_NUMBER (none) -> PSMN4R0-40YS,115
- Q9: renamed from Q8; footprint (none) -> Package_TO_SOT_SMD:LFPAK56; MANUFACTURER_PART_NUMBER (none) -> PSMN4R0-40YS,115
- R12: renamed from R6; footprint (none) -> Resistor_SMD:R_0805_2012Metric; MANUFACTURER (none) -> Digikey; MANUFACTURER_PART_NUMBER (none) -> MFCR0805F2R70QHR
- R13: renamed from R7; footprint (none) -> Resistor_SMD:R_0603_1608Metric; MANUFACTURER (none) -> Digikey; MANUFACTURER_PART_NUMBER (none) -> MCT0603MC4701FP500
- R14: renamed from R8; footprint (none) -> Resistor_SMD:R_0603_1608Metric; MANUFACTURER (none) -> Digikey; MANUFACTURER_PART_NUMBER (none) -> MCT0603MC4701FP500
- R15: renamed from R9; footprint (none) -> Resistor_SMD:R_0805_2012Metric; MANUFACTURER (none) -> Digikey; MANUFACTURER_PART_NUMBER (none) -> TNPW080510K0FEEA
- R16: renamed from R10; footprint (none) -> Resistor_SMD:R_0815_2038Metric; MANUFACTURER (none) -> Digikey; MANUFACTURER_PART_NUMBER (none) -> RL3720WT-R025-G
- R17: renamed from R11; footprint (none) -> Resistor_SMD:R_0805_2012Metric; MANUFACTURER (none) -> Digikey; MANUFACTURER_PART_NUMBER (none) -> TNPW080510K0FEEA
- R18: renamed from R12; footprint (none) -> Resistor_SMD:R_0603_1608Metric; MANUFACTURER (none) -> Digikey; MANUFACTURER_PART_NUMBER (none) -> RQ73C1J63K4BTD
- R19: renamed from R13; footprint (none) -> Resistor_SMD:R_0805_2012Metric; MANUFACTURER (none) -> Digikey; MANUFACTURER_PART_NUMBER (none) -> MFCR0805F2R70QHR
- R20: renamed from R14; footprint (none) -> Resistor_SMD:R_0603_1608Metric; MANUFACTURER (none) -> Digikey; MANUFACTURER_PART_NUMBER (none) -> MCT0603MC4701FP500
- R21: renamed from R15; footprint (none) -> Resistor_SMD:R_0603_1608Metric; MANUFACTURER (none) -> Digikey; MANUFACTURER_PART_NUMBER (none) -> MCT0603MC4701FP500
- R22: renamed from R16; footprint (none) -> Resistor_SMD:R_0805_2012Metric; MANUFACTURER (none) -> Digikey; MANUFACTURER_PART_NUMBER (none) -> TNPW080510K0FEEA
- R23: renamed from R17; footprint (none) -> Resistor_SMD:R_0815_2038Metric; MANUFACTURER (none) -> Digikey; MANUFACTURER_PART_NUMBER (none) -> RL3720WT-R025-G
- R24: renamed from R18; footprint (none) -> Resistor_SMD:R_0805_2012Metric; MANUFACTURER (none) -> Digikey; MANUFACTURER_PART_NUMBER (none) -> TNPW080510K0FEEA
- R25: renamed from R19; footprint (none) -> Resistor_SMD:R_0603_1608Metric; MANUFACTURER (none) -> Digikey; MANUFACTURER_PART_NUMBER (none) -> RQ73C1J63K4BTD
- R26: renamed from R20; footprint (none) -> Resistor_SMD:R_0805_2012Metric; MANUFACTURER (none) -> Digikey; MANUFACTURER_PART_NUMBER (none) -> MFCR0805F2R70QHR
- R27: renamed from R21; footprint (none) -> Resistor_SMD:R_0603_1608Metric; MANUFACTURER (none) -> Digikey; MANUFACTURER_PART_NUMBER (none) -> MCT0603MC4701FP500
- R28: renamed from R22; footprint (none) -> Resistor_SMD:R_0603_1608Metric; MANUFACTURER (none) -> Digikey; MANUFACTURER_PART_NUMBER (none) -> MCT0603MC4701FP500
- R29: renamed from R23; footprint (none) -> Resistor_SMD:R_0805_2012Metric; MANUFACTURER (none) -> Digikey; MANUFACTURER_PART_NUMBER (none) -> TNPW080510K0FEEA
- R30: renamed from R24; footprint (none) -> Resistor_SMD:R_0815_2038Metric; MANUFACTURER (none) -> Digikey; MANUFACTURER_PART_NUMBER (none) -> RL3720WT-R025-G
- R31: renamed from R25; footprint (none) -> Resistor_SMD:R_0805_2012Metric; MANUFACTURER (none) -> Digikey; MANUFACTURER_PART_NUMBER (none) -> TNPW080510K0FEEA
- R32: renamed from R26; footprint (none) -> Resistor_SMD:R_0603_1608Metric; MANUFACTURER (none) -> Digikey; MANUFACTURER_PART_NUMBER (none) -> RQ73C1J63K4BTD
- R33: renamed from R27; footprint (none) -> Resistor_SMD:R_0805_2012Metric; MANUFACTURER (none) -> Digikey; MANUFACTURER_PART_NUMBER (none) -> MFCR0805F2R70QHR
- R34: renamed from R28; footprint (none) -> Resistor_SMD:R_0603_1608Metric; MANUFACTURER (none) -> Digikey; MANUFACTURER_PART_NUMBER (none) -> MCT0603MC4701FP500
- R35: renamed from R29; footprint (none) -> Resistor_SMD:R_0603_1608Metric; MANUFACTURER (none) -> Digikey; MANUFACTURER_PART_NUMBER (none) -> MCT0603MC4701FP500
- R36: renamed from R30; footprint (none) -> Resistor_SMD:R_0805_2012Metric; MANUFACTURER (none) -> Digikey; MANUFACTURER_PART_NUMBER (none) -> TNPW080510K0FEEA
- R37: renamed from R31; footprint (none) -> Resistor_SMD:R_0815_2038Metric; MANUFACTURER (none) -> Digikey; MANUFACTURER_PART_NUMBER (none) -> RL3720WT-R025-G
- R38: renamed from R32; footprint (none) -> Resistor_SMD:R_0805_2012Metric; MANUFACTURER (none) -> Digikey; MANUFACTURER_PART_NUMBER (none) -> TNPW080510K0FEEA
- R39: renamed from R33; footprint (none) -> Resistor_SMD:R_0603_1608Metric; MANUFACTURER (none) -> Digikey; MANUFACTURER_PART_NUMBER (none) -> RQ73C1J63K4BTD
- U10: renamed from U9; footprint DBV5 -> Package_DFN_QFN:QFN-28-1EP_4x5mm_P0.5mm_EP2.65x3.65mm_ThermalVias
- U7: renamed from U6; footprint Package_TO_SOT_SMD:TSOT-23-6 -> Package_DFN_QFN:QFN-28-1EP_4x5mm_P0.5mm_EP2.65x3.65mm_ThermalVias
- U8: renamed from U7; footprint Package_TO_SOT_SMD:TSOT-23-6 -> Package_DFN_QFN:QFN-28-1EP_4x5mm_P0.5mm_EP2.65x3.65mm_ThermalVias
- U9: renamed from U8; footprint LTC4162IUFD-LADM_PBF:QFN50P500X400X80-29N -> Package_DFN_QFN:QFN-28-1EP_4x5mm_P0.5mm_EP2.65x3.65mm_ThermalVias
- renumbered C6 to C14, C7 to C15, C12 to C20, C15 to C23, C16 to C24, C21 to C29, C24 to C32, C25 to C33, C30 to C38, C33 to C41, C34 to C42, C39 to C47, C42 to C50
Connections:
- net GND: now also D10.2 (A2), D11.2 (A2), D12.2 (A2), D9.2 (A2)
- net SOLAR_+X: now also D10.1 (A1)
- net SOLAR_+Y: now also D11.1 (A1)
- net SOLAR_-X: now also D9.1 (A1)
- net SOLAR_-Y: now also D12.1 (A1)
- net Thermistor_+Y: now reaches R31.2, U9.10 (NTC)
- net Thermistor_-Y: now reaches R38.2, U10.10 (NTC)
- net Thermistor_+X: now reaches R17.2, U7.10 (NTC)
- net Thermistor_-X: now reaches R24.2, U8.10 (NTC)

Commit message: A bunch of misc schematic changes
Parts:
- removed C14, C23, C32, C41: 1 uF, Capacitor_SMD:C_0603_1608Metric, symbol Device:C
- removed C15, C24, C33, C42: 4.7 uF, Capacitor_SMD:C_0603_1608Metric, symbol Device:C
- removed C16, C22, C25, C31, C34, C40, C43, C49: 10 uF, zLibrary:CAP_C1210C_X7R_2S_FW_KEM-M, symbol Device:C
- removed C17, C18, C26, C27, C35, C36, C44, C45: 100n, Capacitor_SMD:C_0603_1608Metric, symbol Device:C
- removed C19, C28, C37, C46: 22nF, Capacitor_SMD:C_0603_1608Metric, symbol Device:C
- removed C20, C29, C38, C47: 100uF, Capacitor_Tantalum_SMD:CP_EIA-7361-38_AVX-V, symbol Device:C
- removed C21, C30, C39, C48: 22 uF, zLibrary:CAP_C2220C_2S_KEM-M, symbol Device:C
- removed D10, D11, D12, D9: SMAJ22A, Diode_SMD:D_SMA, symbol Diode:SMAJ22A
- removed L2, L3, L4, L5: 4.7uH, zLibrary:IND_SRP7028A-4R7M_BRN-M, symbol Device:L
- removed Q10, Q11, Q4, Q5, Q6, Q7, Q8, Q9: NMOS, Package_TO_SOT_SMD:LFPAK56, symbol Simulation_SPICE:NMOS
- removed R12, R19, R26, R33: 2.5, Resistor_SMD:R_0805_2012Metric, symbol Device:R
- removed R13, R14, R20, R21, R27, R28, R34, R35: 4.7k, Resistor_SMD:R_0603_1608Metric, symbol Device:R
- removed R15, R17, R22, R24, R29, R31, R36, R38: 10k, Resistor_SMD:R_0805_2012Metric, symbol Device:R
- removed R16, R23, R30, R37: 25m, Resistor_SMD:R_0815_2038Metric, symbol Device:R
- removed R18, R25, R32, R39: 63.4k, Resistor_SMD:R_0603_1608Metric, symbol Device:R
- removed U10, U7, U8, U9: LTC4162IUFD-LADM_PBF, Package_DFN_QFN:QFN-28-1EP_4x5mm_P0.5mm_EP2.65x3.65mm_ThermalVias, symbol LTC4162IUFD-LADM_PBF:LTC4162IUFD-LADM_PBF
- renumbered C50 to C14
Connections:
- net Battery: no longer C14.1
- new net MPPT_CAP: C14.1
Other:
- added sheet +X_MPPT (MPPT_indv.kicad_sch)
- added sheet +Y_MPPT (MPPT_indv.kicad_sch)
- added sheet -X_MPPT (MPPT_indv.kicad_sch)
- added sheet -Y_MPPT (MPPT_indv.kicad_sch)
- moved on the sheet: C14
