File: MPPT_IC.kicad_sch (KiCad schematic)
At the start: 9 parts

Commit message: Added Batt 1 and Batt 2 charging
Changed lines of the file:
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@@
 		)
 	)
-	(text_box "Notes:\n-!SMB_ALERT will be tied to a External Interrupt Line (EXTI) on the MCU which will be triggered by a falling edge\n- Think about ferrite Bead Placement on input\n- Assumptions made when calculating inductor val:\n	15V solar input, 8.4V battery, 1.2A max charge limit\n	10uH (max I= 3A) (<30m ohms)"
+	(text_box "Notes:\n-!SMB_ALERT will be tied to a External Interrupt Line (EXTI) on the MCU which will be triggered by a falling edge\n- Assumptions made when calculating inductor val:\n	15V solar input, 8.4V battery, 1.2A max charge limit\n	10uH (max I= 3A) (<30m ohms)"
 		(exclude_from_sim no)
 		(at 13.97 295.91 0)
@@
 	(wire
 		(pts
+			(xy 64.77 114.3) (xy 64.77 264.16)
+		)
+		(stroke
+			(width 0)
+			(type default)
+		)
+	)
+	(wire
+		(pts
 			(xy 222.25 186.69) (xy 218.44 186.69)
 		)
@@
 	(wire
 		(pts
+			(xy 113.03 191.77) (xy 57.15 191.77)
+		)
+		(stroke
+			(width 0)
+			(type default)
+		)
+	)
+	(wire
+		(pts
 			(xy 134.62 313.69) (xy 121.92 313.69)
 		)
@@
 	(wire
 		(pts
+			(xy 57.15 191.77) (xy 57.15 53.34)
+		)
+		(stroke
+			(width 0)
+			(type default)
+		)
+	)
+	(wire
+		(pts
 			(xy 194.31 176.53) (xy 170.18 176.53)
 		)
@@
 	(wire
 		(pts
+			(xy 113.03 114.3) (xy 64.77 114.3)
+		)
+		(stroke
+			(width 0)
+			(type default)
+		)
+	)
+	(wire
+		(pts
 			(xy 91.44 33.02) (xy 113.03 33.02)
 		)
@@
 		(pts
 			(xy 91.44 38.1) (xy 113.03 38.1)
+		)
+		(stroke
+			(width 0)
+			(type default)
+		)
+	)
+	(wire
+		(pts
+			(xy 64.77 264.16) (xy 111.76 264.16)
 		)
 		(stroke
@@
 			(width 0.762)
 			(type dash)
+		)
+	)
+	(wire
+		(pts
+			(xy 57.15 53.34) (xy 113.03 53.34)
+		)
+		(stroke
+			(width 0)
+			(type default)
 		)
 	)
@@
 		)
 	)
-	(hierarchical_label "SDA_+Y"
-		(shape input)
-		(at 92.71 104.14 180)
-		(effects
-			(font
-				(size 1.27 1.27)
-			)
-			(justify right)
-		)
-	)
-	(hierarchical_label "-X_OUT"
-		(shape input)
-		(at 194.31 176.53 0)
-		(effects
-			(font
-				(size 1.27 1.27)
-			)
-			(justify left)
-		)
-	)
-	(hierarchical_label "Thermistor_-X"
-		(shape output)
-		(at 194.31 181.61 0)
-		(effects
-			(font
-				(size 1.27 1.27)
-			)
-			(justify left)
+	(hierarchical_label "SOLAR_-X"
+		(shape input)
+		(at 93.98 99.06 180)
+		(effects
+			(font
+				(size 1.27 1.27)
+			)
+			(justify right)
 		)
 	)
@@
 		)
 	)
-	(hierarchical_label "SCL_+Y"
-		(shape input)
-		(at 92.71 109.22 180)
+	(hierarchical_label "SDA_-X"
+		(shape input)
+		(at 93.98 104.14 180)
+		(effects
+			(font
+				(size 1.27 1.27)
+			)
+			(justify right)
+		)
+	)
+	(hierarchical_label "BattSen1"
+		(shape input)
+		(at 64.77 264.16 180)
+		(effects
+			(font
+				(size 1.27 1.27)
+			)
+			(justify right)
+		)
+	)
+	(hierarchical_label "SCL_-X"
+		(shape input)
+		(at 93.98 109.22 180)
 		(effects
 			(font
@@
 			)
 			(justify left)
-		)
-	)
-	(hierarchical_label "SCL_-X"
-		(shape input)
-		(at 93.98 186.69 180)
-		(effects
-			(font
-				(size 1.27 1.27)
-			)
-			(justify right)
 		)
 	)
@@
 		)
 	)
+	(hierarchical_label "Thermistor_+Y"
+		(shape output)
+		(at 194.31 181.61 0)
+		(effects
+			(font
+				(size 1.27 1.27)
+			)
+			(justify left)
+		)
+	)
+	(hierarchical_label "SCL_+Y"
+		(shape input)
+		(at 95.25 186.69 180)
+		(effects
+			(font
+				(size 1.27 1.27)
+			)
+			(justify right)
+		)
+	)
+	(hierarchical_label "SDA_+Y"
+		(shape input)
+		(at 95.25 181.61 180)
+		(effects
+			(font
+				(size 1.27 1.27)
+			)
+			(justify right)
+		)
+	)
+	(hierarchical_label "!SMB_ALERT_-X"
+		(shape input)
+		(at 93.98 93.98 180)
+		(effects
+			(font
+				(size 1.27 1.27)
+			)
+			(justify right)
+		)
+	)
 	(hierarchical_label "+X_OUT"
 		(shape input)
@@
 	(hierarchical_label "MPPT_SYNC_1.5MHz_3"
 		(shape input)
+		(at 194.31 171.45 0)
+		(effects
+			(font
+				(size 1.27 1.27)
+			)
+			(justify left)
+		)
+	)
+	(hierarchical_label "BattSen2"
+		(shape input)
+		(at 57.15 53.34 180)
+		(effects
+			(font
+				(size 1.27 1.27)
+			)
+			(justify right)
+		)
+	)
+	(hierarchical_label "!SMB_ALERT_+X"
+		(shape input)
+		(at 91.44 33.02 180)
+		(effects
+			(font
+				(size 1.27 1.27)
+			)
+			(justify right)
+		)
+	)
+	(hierarchical_label "MPPT_SYNC_1.5MHz_2"
+		(shape input)
 		(at 194.31 93.98 0)
 		(effects
@@
 		)
 	)
-	(hierarchical_label "!SMB_ALERT_+X"
-		(shape input)
-		(at 91.44 33.02 180)
-		(effects
-			(font
-				(size 1.27 1.27)
-			)
-			(justify right)
-		)
-	)
 	(hierarchical_label "!SMB_ALERT_-Y"
 		(shape input)
@@
 		)
 	)
-	(hierarchical_label "SDA_-X"
-		(shape input)
-		(at 93.98 181.61 180)
-		(effects
-			(font
-				(size 1.27 1.27)
-			)
-			(justify right)
-		)
-	)
-	(hierarchical_label "!SMB_ALERT_-X"
-		(shape input)
-		(at 93.98 171.45 180)
-		(effects
-			(font
-				(size 1.27 1.27)
-			)
-			(justify right)
+	(hierarchical_label "Thermistor_-X"
+		(shape output)
+		(at 194.31 104.14 0)
+		(effects
+			(font
+				(size 1.27 1.27)
+			)
+			(justify left)
+		)
+	)
+	(hierarchical_label "+Y_OUT"
+		(shape input)
+		(at 194.31 176.53 0)
+		(effects
+			(font
+				(size 1.27 1.27)
+			)
+			(justify left)
+		)
+	)
+	(hierarchical_label "SOLAR_+Y"
+		(shape input)
+		(at 95.25 176.53 180)
+		(effects
+			(font
+				(size 1.27 1.27)
+			)
+			(justify right)
+		)
+	)
+	(hierarchical_label "-X_OUT"
+		(shape input)
+		(at 194.31 99.06 0)
+		(effects
+			(font
+				(size 1.27 1.27)
+			)
+			(justify left)
 		)
 	)
@@
 		)
 	)
-	(hierarchical_label "SOLAR_-X"
-		(shape input)
-		(at 93.98 176.53 180)
-		(effects
-			(font
-				(size 1.27 1.27)
-			)
-			(justify right)
-		)
-	)
 	(hierarchical_label "SCL_+X"
 		(shape input)
@@
 		)
 	)
-	(hierarchical_label "MPPT_SYNC_1.5MHz_2"
-		(shape input)
-		(at 194.31 171.45 0)
-		(effects
-			(font
-				(size 1.27 1.27)
-			)
-			(justify left)
-		)
-	)
-	(hierarchical_label "SOLAR_+Y"
-		(shape input)
-		(at 92.71 99.06 180)
-		(effects
-			(font
-				(size 1.27 1.27)
-			)
-			(justify right)
-		)
-	)
-	(hierarchical_label "Thermistor_+Y"
-		(shape output)
-		(at 194.31 104.14 0)
-		(effects
-			(font
-				(size 1.27 1.27)
-			)
-			(justify left)
+	(hierarchical_label "!SMB_ALERT_+Y"
+		(shape input)
+		(at 95.25 171.45 180)
+		(effects
+			(font
+				(size 1.27 1.27)
+			)
+			(justify right)
 		)
 	)
@@
 		(effects
 			(font
-				(size 1.27 1.27)
-			)
-			(justify right)
-		)
-	)
-	(hierarchical_label "+Y_OUT"
-		(shape input)
-		(at 194.31 99.06 0)
-		(effects
-			(font
-				(size 1.27 1.27)
-			)
-			(justify left)
-		)
-	)
-	(hierarchical_label "!SMB_ALERT_+Y"
-		(shape input)
-		(at 92.71 93.98 180)
-		(effects
-			(font
