File: Sensing.kicad_sch (KiCad schematic)
At the start: 0 parts

Commit message: edited 3V3 Logic to add Efuse and UVLO
Parts:
- added U15: INA3221, Package_DFN_QFN:Texas_RGV0016A_VQFN-16-1EP_4x4mm_P0.65mm_EP2.1x2.1mm, symbol Power_Management:INA3221
Changed lines of the file:
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@@
 	(generator_version "9.0")
 	(paper "A4")
+	(symbol
+		(lib_id "Power_Management:INA3221")
+		(at 71.12 60.96 0)
+		(unit 1)
+		(exclude_from_sim no)
+		(in_bom yes)
+		(on_board yes)
+		(dnp no)
+		(fields_autoplaced yes)
+		(property "Reference" "U15"
+			(at 75.8033 40.64 0)
+			(effects
+				(font
+					(size 1.27 1.27)
+				)
+				(justify left)
+			)
+		)
+		(property "Value" "INA3221"
+			(at 75.8033 43.18 0)
+			(effects
+				(font
+					(size 1.27 1.27)
+				)
+				(justify left)
+			)
+		)
+		(property "Footprint" "Package_DFN_QFN:Texas_RGV0016A_VQFN-16-1EP_4x4mm_P0.65mm_EP2.1x2.1mm"
+			(at 71.12 33.02 0)
+			(effects
+				(font
+					(size 1.27 1.27)
+				)
+				(hide yes)
+			)
+		)
+		(property "Datasheet" "http://www.ti.com/lit/ds/symlink/ina3221.pdf"
+			(at 71.12 43.18 0)
+			(effects
+				(font
+					(size 1.27 1.27)
+				)
+				(hide yes)
+			)
+		)
+		(property "Description" "Triple-Channel High-Side Shunt and Bus Voltage Monitor with I2C and SMBUS Compatible Interface, QFN-16"
+			(at 71.12 60.96 0)
+			(effects
+				(font
+					(size 1.27 1.27)
+				)
+				(hide yes)
+			)
+		)
+		(pin "1"
+		)
+		(pin "6"
+		)
+		(pin "14"
+		)
+		(pin "7"
+		)
+		(pin "11"
+		)
+		(pin "15"
+		)
+		(pin "10"
+		)
+		(pin "4"
+		)
+		(pin "13"
+		)
+		(pin "5"
+		)
+		(pin "12"
+		)
+		(pin "2"
+		)
+		(pin "17"
+		)
+		(pin "8"
+		)
+		(pin "3"
+		)
+		(pin "9"
+		)
+		(pin "16"
+		)
+		(instances
+			(project ""
+				(path "/8f246f89-1ec7-4136-9977-839b50e116ed/5683cac5-9988-4b0a-8935-fabef808a774"
+					(reference "U15")
+					(unit 1)
+				)
+			)
+		)
+	)
 )

Commit message: added current sensing and e-fuses
Parts:
- added C73, C77: 100nF, symbol Device:C
- added C74, C75, C76: 1uF, symbol Device:C
- added C78, C82, C86: 100nF, Capacitor_SMD:C_1210_3225Metric, symbol Device:C
- added C79, C83, C87: 2.2nF, Capacitor_SMD:C_1210_3225Metric, symbol Device:C
- added C80, C84, C88: 100pF, Capacitor_SMD:C_1210_3225Metric, symbol Device:C
- added C81, C85, C89: 10uF, Capacitor_SMD:C_1210_3225Metric, symbol Device:C
- added Q12, Q13, Q14: NMOS, symbol Simulation_SPICE:NMOS
- added R61, R65, R66: 4m, symbol Device:R
- added R67, R68, R76, R77, R78, R81, R88, R94, R95, R96: 10k, symbol Device:R
- added R69, R70, R71, R72, R73, R74: 10, symbol Device:R
- added R79, R84: 182k, symbol Device:R
- added R80, R83, R86, R87, R91, R92: 100k, symbol Device:R
- added R82, R85: 20k, symbol Device:R
- added R89: 348k, symbol Device:R
- added R90: 31.6k, symbol Device:R
- added R93: 5kk, symbol Device:R
- added U17, U18, U19: TPS259470ARPWR, RPW0010A-MFG, symbol TPS259470:TPS259470ARPWR
Connections:
- net at U15.1 (IN-3): now also C76.2, R74.2
- net PV_INA3221: now reaches U15.10 (PV)
- net PV_INA3221: now also R78.2
- net at U15.11 (IN-1): now also C74.2, R70.2
- net at U15.12 (IN+1): now also C74.1, R69.2
- net at U15.14 (IN-2): now also C75.2, R72.2
- net at U15.15 (IN+2): now also C75.1, R71.2
- net +3.3V: now reaches U15.16 (VPU)
- net +3.3V: now also U15.4 (VS), C73.1, C77.1, R67.1, R68.1, R76.1, R77.1, R78.1, R80.1, R87.1, R92.1
- net GND: now reaches U15.17 (EP)
- net GND: now also U15.3 (GND), U15.5 (A0), C73.2, C77.2, C78.2, C79.2, C80.2, C81.2, C82.2, C83.2, C84.2, C85.2, C86.2, C87.2, C88.2, C89.2, Q12.3 (S), Q13.3 (S), Q14.3 (S), R81.2, R83.2, R86.2, R88.2, R91.2, R93.2, R94.2, R95.2, R96.2, U17.3 (AUXOFF), U17.8 (GND), U18.3 (AUXOFF), U18.8 (GND), U19.3 (AUXOFF), U19.8 (GND)
- net at U15.2 (IN+3): now also C76.1, R73.2
- net SCL_INA3221: now reaches U15.6 (SCL)
- net SCL_INA3221: now also R68.2
- net SDA_INA3221: now reaches U15.7 (SDA)
- net SDA_INA3221: now also R67.2
- net WAR_INA3221: now reaches U15.8 (WARNING)
- net WAR_INA3221: now also R76.2
- net CRIT_INA3221: now reaches U15.9 (CRITICAL)
- net CRIT_INA3221: now also R77.2
- new net: R90.2, R91.1, U19.2 (OVLO)
- new net: R88.1, U18.9 (ILM)
- new net: C84.1, U18.7 (dVdt)
- new net: Q14.1 (D), R89.2, R90.1, U19.1 (EN_UVLO)
- new net: C89.1, U19.6 (OUT)
- new net: R87.2, U18.4 (!FLT)
- new net: C81.1, U17.6 (OUT)
- new net: R93.1, U19.9 (ILM)
- new net: Q13.1 (D), R84.2, R85.1, U18.1 (EN_UVLO)
- new net: R85.2, R86.1, U18.2 (OVLO)
- new net: C87.1, U19.10 (ITIMER)
- new net: Q12.1 (D), R79.2, R82.1, U17.1 (EN_UVLO)
- new net: C85.1, U18.6 (OUT)
- new net: R92.2, U19.4 (!FLT)
- new net: C83.1, U18.10 (ITIMER)
- new net: C79.1, U17.10 (ITIMER)
- new net: R82.2, R83.1, U17.2 (OVLO)
- new net: R80.2, U17.4 (!FLT)
- new net: C80.1, U17.7 (dVdt)
- new net: R81.1, U17.9 (ILM)
- new net: C88.1, U19.7 (dVdt)
- new net 3V3_Line: R61.1, R65.1, R69.1, R71.1
- new net 5V_Line: R66.1, R73.1
- new net ADCS_3V3: C82.1, R65.2, R72.1, R84.1, U18.5 (IN)
- new net ADCS_3V3_ShutDown: Q13.2 (G), R95.1
- new net ADCS_5V: C86.1, R66.2, R74.1, R89.1, U19.5 (IN)
- new net ADCS_5V_ShutDown: Q14.2 (G), R96.1
- new net OBC3V3: C78.1, R79.1, U17.5 (IN)
- new net OBC_3V3: R61.2, R70.1
- new net OBC_3V3_ShutDown: Q12.2 (G), R94.1
- no-connect marks 0 -> 1
Other:
- note added: "ADCS 3.3V E-Fuse"
- note added: "ADCS 5V E-Fuse"
- note added: "Current Sensing"
- note added: "OBC 3.3V E-Fuse"
- company: (none) -> QSET (Jaron Cyna)
- title: (none) -> Current Sensing and E-Fuse
- moved on the sheet: U15

Commit message: Added connectors to schematic
Parts:
- C66: renamed from C73; footprint (none) -> Capacitor_SMD:C_0603_1608Metric; MANUFACTURER (none) -> DigiKey; MANUFACTURER_PART_NUMBER (none) -> 06035C104K4T2A
- C67: renamed from C77; footprint (none) -> Capacitor_SMD:C_0603_1608Metric; MANUFACTURER (none) -> DigiKey; MANUFACTURER_PART_NUMBER (none) -> 06035C104K4T2A
- C68: renamed from C74; footprint (none) -> Capacitor_SMD:C_0603_1608Metric; MANUFACTURER (none) -> DigiKey; MANUFACTURER_PART_NUMBER (none) -> CL10B105KQ8NNNC
- C69: renamed from C75; footprint (none) -> Capacitor_SMD:C_0603_1608Metric; MANUFACTURER (none) -> DigiKey; MANUFACTURER_PART_NUMBER (none) -> CL10B105KQ8NNNC
- C70: renamed from C76; footprint (none) -> Capacitor_SMD:C_0603_1608Metric; MANUFACTURER (none) -> DigiKey; MANUFACTURER_PART_NUMBER (none) -> CL10B105KQ8NNNC
- C71: renamed from C81; footprint Capacitor_SMD:C_1210_3225Metric -> zLibrary:CAP_C1210C_X7R_2S_FW_KEM-M; MANUFACTURER_PART_NUMBER CL32B226KAJNFNE -> C1210C106M5R2C7186
- C72: renamed from C89; footprint Capacitor_SMD:C_1210_3225Metric -> zLibrary:CAP_C1210C_X7R_2S_FW_KEM-M; MANUFACTURER_PART_NUMBER CL32B226KAJNFNE -> C1210C106M5R2C7186
- C73: renamed from C78; footprint Capacitor_SMD:C_1210_3225Metric -> Capacitor_SMD:C_0603_1608Metric; MANUFACTURER_PART_NUMBER CL32B226KAJNFNE -> 06035C104K4T2A
- C74: renamed from C86; footprint Capacitor_SMD:C_1210_3225Metric -> Capacitor_SMD:C_0603_1608Metric; MANUFACTURER_PART_NUMBER CL32B226KAJNFNE -> 06035C104K4T2A
- C75: renamed from C85; footprint Capacitor_SMD:C_1210_3225Metric -> zLibrary:CAP_C1210C_X7R_2S_FW_KEM-M; MANUFACTURER_PART_NUMBER CL32B226KAJNFNE -> C1210C106M5R2C7186
- C76: renamed from C82; footprint Capacitor_SMD:C_1210_3225Metric -> Capacitor_SMD:C_0603_1608Metric; MANUFACTURER_PART_NUMBER CL32B226KAJNFNE -> 06035C104K4T2A
- C77: renamed from C79; footprint Capacitor_SMD:C_1210_3225Metric -> Capacitor_SMD:C_0603_1608Metric; MANUFACTURER_PART_NUMBER CL32B226KAJNFNE -> GCM1885C1H222FA16D
- C78: renamed from C80; footprint Capacitor_SMD:C_1210_3225Metric -> Capacitor_SMD:C_0603_1608Metric; MANUFACTURER_PART_NUMBER CL32B226KAJNFNE -> 885342206001
- C79: renamed from C87; footprint Capacitor_SMD:C_1210_3225Metric -> Capacitor_SMD:C_0603_1608Metric; MANUFACTURER_PART_NUMBER CL32B226KAJNFNE -> GCM1885C1H222FA16D
- C80: renamed from C88; footprint Capacitor_SMD:C_1210_3225Metric -> Capacitor_SMD:C_0603_1608Metric; MANUFACTURER_PART_NUMBER CL32B226KAJNFNE -> 885342206001
- C81: renamed from C83; footprint Capacitor_SMD:C_1210_3225Metric -> Capacitor_SMD:C_0603_1608Metric; MANUFACTURER_PART_NUMBER CL32B226KAJNFNE -> GCM1885C1H222FA16D
- C82: renamed from C84; footprint Capacitor_SMD:C_1210_3225Metric -> Capacitor_SMD:C_0603_1608Metric; MANUFACTURER_PART_NUMBER CL32B226KAJNFNE -> 885342206001
- Q12: footprint (none) -> Package_TO_SOT_SMD:LFPAK56; MANUFACTURER_PART_NUMBER (none) -> PSMN4R0-40YS,115
- Q13: renamed from Q14; footprint (none) -> Package_TO_SOT_SMD:LFPAK56; MANUFACTURER_PART_NUMBER (none) -> PSMN4R0-40YS,115
- Q14: renamed from Q13; footprint (none) -> Package_TO_SOT_SMD:LFPAK56; MANUFACTURER_PART_NUMBER (none) -> PSMN4R0-40YS,115
- R57: renamed from R69; footprint (none) -> Resistor_SMD:R_0805_2012Metric; MANUFACTURER (none) -> Digikey; MANUFACTURER_PART_NUMBER (none) -> TNPW080510R0BEEA
- R58: renamed from R61; footprint (none) -> Resistor_SMD:R_0815_2038Metric; MANUFACTURER (none) -> Digikey; MANUFACTURER_PART_NUMBER (none) -> RL3720WT-R004-F
- R59: renamed from R78; footprint (none) -> Resistor_SMD:R_0805_2012Metric; MANUFACTURER (none) -> Digikey; MANUFACTURER_PART_NUMBER (none) -> TNPW080510K0FEEA
- R60: renamed from R77; footprint (none) -> Resistor_SMD:R_0805_2012Metric; MANUFACTURER (none) -> Digikey; MANUFACTURER_PART_NUMBER (none) -> TNPW080510K0FEEA
- R61: renamed from R76; footprint (none) -> Resistor_SMD:R_0805_2012Metric; MANUFACTURER (none) -> Digikey; MANUFACTURER_PART_NUMBER (none) -> TNPW080510K0FEEA
- R62: renamed from R67; footprint (none) -> Resistor_SMD:R_0805_2012Metric; MANUFACTURER (none) -> Digikey; MANUFACTURER_PART_NUMBER (none) -> TNPW080510K0FEEA
- R63: renamed from R68; footprint (none) -> Resistor_SMD:R_0805_2012Metric; MANUFACTURER (none) -> Digikey; MANUFACTURER_PART_NUMBER (none) -> TNPW080510K0FEEA
- R64: renamed from R71; footprint (none) -> Resistor_SMD:R_0805_2012Metric; MANUFACTURER (none) -> Digikey; MANUFACTURER_PART_NUMBER (none) -> TNPW080510R0BEEA
- R65: renamed from R70; footprint (none) -> Resistor_SMD:R_0805_2012Metric; MANUFACTURER (none) -> Digikey; MANUFACTURER_PART_NUMBER (none) -> TNPW080510R0BEEA
- R66: renamed from R65; footprint (none) -> Resistor_SMD:R_0815_2038Metric; MANUFACTURER (none) -> Digikey; MANUFACTURER_PART_NUMBER (none) -> RL3720WT-R004-F
- R67: renamed from R72; footprint (none) -> Resistor_SMD:R_0805_2012Metric; MANUFACTURER (none) -> Digikey; MANUFACTURER_PART_NUMBER (none) -> TNPW080510R0BEEA
- R68: renamed from R73; footprint (none) -> Resistor_SMD:R_0805_2012Metric; MANUFACTURER (none) -> Digikey; MANUFACTURER_PART_NUMBER (none) -> TNPW080510R0BEEA
- R69: renamed from R66; footprint (none) -> Resistor_SMD:R_0815_2038Metric; MANUFACTURER (none) -> Digikey; MANUFACTURER_PART_NUMBER (none) -> RL3720WT-R004-F
- R70: renamed from R74; footprint (none) -> Resistor_SMD:R_0805_2012Metric; MANUFACTURER (none) -> Digikey; MANUFACTURER_PART_NUMBER (none) -> TNPW080510R0BEEA
- R71: renamed from R80; footprint (none) -> Resistor_SMD:R_0603_1608Metric; MANUFACTURER (none) -> Digikey; MANUFACTURER_PART_NUMBER (none) -> AT0603FRE07100KL
- R72: renamed from R92; footprint (none) -> Resistor_SMD:R_0603_1608Metric; MANUFACTURER (none) -> Digikey; MANUFACTURER_PART_NUMBER (none) -> AT0603FRE07100KL
- R73: renamed from R87; footprint (none) -> Resistor_SMD:R_0603_1608Metric; MANUFACTURER (none) -> Digikey; MANUFACTURER_PART_NUMBER (none) -> AT0603FRE07100KL
- R74: renamed from R79; footprint (none) -> Resistor_SMD:R_0603_1608Metric
- R75: renamed from R89; footprint (none) -> Resistor_SMD:R_0603_1608Metric
- R76: renamed from R84; footprint (none) -> Resistor_SMD:R_0603_1608Metric
- R77: renamed from R82; footprint (none) -> Resistor_SMD:R_0603_1608Metric
- R78: renamed from R90; footprint (none) -> Resistor_SMD:R_0603_1608Metric
- R79: renamed from R85; footprint (none) -> Resistor_SMD:R_0603_1608Metric
- R80: renamed from R81; footprint (none) -> Resistor_SMD:R_0805_2012Metric; MANUFACTURER (none) -> Digikey; MANUFACTURER_PART_NUMBER (none) -> TNPW080510K0FEEA
- R81: renamed from R93; value 5kk -> 5k; footprint (none) -> Resistor_SMD:R_0603_1608Metric; MANUFACTURER (none) -> Digikey; MANUFACTURER_PART_NUMBER (none) -> RN73R1JTTD4991F100
- R82: renamed from R83; footprint (none) -> Resistor_SMD:R_0603_1608Metric; MANUFACTURER (none) -> Digikey; MANUFACTURER_PART_NUMBER (none) -> AT0603FRE07100KL
- R83: renamed from R88; footprint (none) -> Resistor_SMD:R_0805_2012Metric; MANUFACTURER (none) -> Digikey; MANUFACTURER_PART_NUMBER (none) -> TNPW080510K0FEEA
- R84: renamed from R91; footprint (none) -> Resistor_SMD:R_0603_1608Metric; MANUFACTURER (none) -> Digikey; MANUFACTURER_PART_NUMBER (none) -> AT0603FRE07100KL
- R85: renamed from R86; footprint (none) -> Resistor_SMD:R_0603_1608Metric; MANUFACTURER (none) -> Digikey; MANUFACTURER_PART_NUMBER (none) -> AT0603FRE07100KL
- R86: renamed from R94; footprint (none) -> Resistor_SMD:R_0805_2012Metric; MANUFACTURER (none) -> Digikey; MANUFACTURER_PART_NUMBER (none) -> TNPW080510K0FEEA
- R87: renamed from R96; footprint (none) -> Resistor_SMD:R_0805_2012Metric; MANUFACTURER (none) -> Digikey; MANUFACTURER_PART_NUMBER (none) -> TNPW080510K0FEEA
- R88: renamed from R95; footprint (none) -> Resistor_SMD:R_0805_2012Metric; MANUFACTURER (none) -> Digikey; MANUFACTURER_PART_NUMBER (none) -> TNPW080510K0FEEA
- U16: renamed from U17; footprint RPW0010A-MFG -> zLibrary:RPW0010A-MFG
- U17: renamed from U19; footprint RPW0010A-MFG -> zLibrary:RPW0010A-MFG
- U18: footprint RPW0010A-MFG -> zLibrary:RPW0010A-MFG
Connections:
- net ADCS_5V_Line_Out: now reaches C72.1, U17.6 (OUT)
- net OBC_3V3_Line_Out: now reaches C71.1, U16.6 (OUT)
- net ADCS_3V3_Line_Out: now reaches C75.1, U18.6 (OUT)
Other:
- moved on the sheet: C71, C75

Commit message: A bunch of misc schematic changes
Parts:
- renumbered C66 to C30, C67 to C31, C68 to C32, C69 to C33, C70 to C34, C71 to C35, C72 to C36, C73 to C37, C74 to C38, C75 to C39, C76 to C40, C77 to C41, C78 to C42, C79 to C43, C80 to C44, C81 to C45, C82 to C46, Q12 to Q4, Q13 to Q5, Q14 to Q6, R57 to R29, R58 to R30, R59 to R31, R60 to R32, R61 to R33, R62 to R34, R63 to R35, R64 to R36, R65 to R37, R66 to R38, R67 to R39, R68 to R40, R69 to R41, R70 to R42, R71 to R43, R72 to R44, R73 to R45, R74 to R46, R75 to R47, R76 to R48, R77 to R49, R78 to R50, R79 to R51, R80 to R52, R81 to R53, R82 to R54, R83 to R55, R84 to R56, R85 to R57, R86 to R58, R87 to R59, R88 to R60, U15 to U11, U16 to U12, U17 to U13, U18 to U14

Commit message: Small schematic changes
Connections:
- net OBC3V3 is gone; now on net OBC_3V3: C37.1, R46.1, U12.5 (IN)
Changed lines of the file:
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@@
 	)
 	(label "OBC_3V3"
-		(at 191.77 69.85 180)
+		(at 24.13 179.07 180)
 		(effects
 			(font
@@
 		)
 	)
-	(label "ADCS_5V"
-		(at 186.69 109.22 180)
+	(label "OBC_3V3"
+		(at 191.77 69.85 180)
 		(effects
 			(font
@@
 		)
 	)
-	(label "ADCS_3V3"
-		(at 156.21 88.9 180)
+	(label "ADCS_5V"
+		(at 186.69 109.22 180)
 		(effects
 			(font
@@
 		)
 	)
-	(label "OBC3V3"
-		(at 24.13 179.07 180)
+	(label "ADCS_3V3"
+		(at 156.21 88.9 180)
 		(effects
 			(font
@@
 					(size 1.27 1.27)
 				)
+				(hide yes)
 			)
 		)
@@
 					(size 1.27 1.27)
 				)
+				(hide yes)
 			)
 		)
@@
 					(size 1.27 1.27)
 				)
+				(hide yes)
 			)
 		)
@@
 					(size 1.27 1.27)
 				)
+				(hide yes)
 			)
 		)
@@
 					(size 1.27 1.27)
 				)
+				(hide yes)
 			)
 		)
@@
 					(size 1.27 1.27)
 				)
+				(hide yes)
 			)
 		)
@@
 					(size 1.27 1.27)
 				)
+				(hide yes)
 			)
 		)
@@
 					(size 1.27 1.27)
 				)
+				(hide yes)
 			)
 		)
@@
 					(size 1.27 1.27)
 				)
+				(hide yes)
 			)
 		)
@@
 					(size 1.27 1.27)
 				)
+				(hide yes)
 			)
 		)
@@
 					(size 1.27 1.27)
 				)
+				(hide yes)
 			)
 		)
@@
 					(size 1.27 1.27)
 				)
+				(hide yes)
 			)
 		)
@@
 					(size 1.27 1.27)
 				)
+				(hide yes)
 			)
 		)
@@
 					(size 1.27 1.27)
 				)
+				(hide yes)
 			)
 		)
@@
 					(size 1.27 1.27)
 				)
+				(hide yes)
 			)
 		)
@@
 					(size 1.27 1.27)
 				)
+				(hide yes)
 			)
 		)
@@
 					(size 1.27 1.27)
 				)
+				(hide yes)
 			)
 		)
@@
 					(size 1.27 1.27)
 				)
+				(hide yes)
 			)
 		)
@@
 					(size 1.27 1.27)
 				)
+				(hide yes)
 			)
 		)
@@
 					(size 1.27 1.27)
 				)
+				(hide yes)
 			)
 		)
@@
 					(size 1.27 1.27)
 				)
+				(hide yes)
 			)
 		)
@@
 					(size 1.27 1.27)
 				)
+				(hide yes)
 			)
 		)
@@
 					(size 1.27 1.27)
 				)
+				(hide yes)
 			)
 		)
@@
 					(size 1.27 1.27)
 				)
+				(hide yes)
 			)
 		)
@@
 					(size 1.27 1.27)
 				)
+				(hide yes)
 			)
 		)
@@
 					(size 1.27 1.27)
 				)
+				(hide yes)
 			)
 		)
@@
 					(size 1.27 1.27)
 				)
+				(hide yes)
 			)
 		)
@@
 					(size 1.27 1.27)
 				)
+				(hide yes)
 			)
 		)
@@
 					(size 1.27 1.27)
 				)
+				(hide yes)
 			)
 		)
@@
 					(size 1.27 1.27)
 				)
+				(hide yes)
 			)
 		)
@@
 					(size 1.27 1.27)
 				)
+				(hide yes)
 			)
 		)
@@
 					(size 1.27 1.27)
 				)
+				(hide yes)
 			)
 		)
@@
 					(size 1.27 1.27)
 				)
+				(hide yes)
 			)
 		)
@@
 					(size 1.27 1.27)
 				)
+				(hide yes)
 			)
 		)
@@
 					(size 1.27 1.27)
 				)
+				(hide yes)
 			)
 		)
@@
 					(size 1.27 1.27)
 				)
+				(hide yes)
 			)
 		)
@@
 					(size 1.27 1.27)
 				)
+				(hide yes)
 			)
 		)
@@
 					(size 1.27 1.27)
 				)
+				(hide yes)
 			)
 		)
@@
 					(size 1.27 1.27)
 				)
+				(hide yes)
 			)
 		)
@@
 					(size 1.27 1.27)
 				)
+				(hide yes)
 			)
 		)
@@
 					(size 1.27 1.27)
 				)
+				(hide yes)
 			)
 		)
@@
 					(size 1.27 1.27)
 				)
+				(hide yes)
 			)
 		)
@@
 					(size 1.27 1.27)
 				)
+				(hide yes)
 			)
 		)
@@
 					(size 1.27 1.27)
 				)
+				(hide yes)
 			)
 		)
@@
 					(size 1.27 1.27)
 				)
+				(hide yes)
 			)
 		)
@@
 					(size 1.27 1.27)
 				)
+				(hide yes)
 			)
 		)
@@
 					(size 1.27 1.27)
 				)
+				(hide yes)
 			)
 		)
@@
 					(size 1.27 1.27)
 				)
+				(hide yes)
 			)
 		)
@@
 					(size 1.27 1.27)
 				)
+				(hide yes)
 			)
 		)
@@
 					(size 1.27 1.27)
 				)
+				(hide yes)
 			)
 		)
@@
 					(size 1.27 1.27)
 				)
+				(hide yes)
 			)
 		)
@@
 					(size 1.27 1.27)
 				)
+				(hide yes)
 			)
 		)
@@
 					(size 1.27 1.27)
 				)
+				(hide yes)
 			)
 		)
@@
 					(size 1.27 1.27)
 				)
+				(hide yes)
 			)
 		)
@@
 					(size 1.27 1.27)
 				)
+				(hide yes)
 			)
 		)
@@
 					(size 1.27 1.27)
 				)
+				(hide yes)
 			)
 		)
@@
 					(size 1.27 1.27)
 				)
+				(hide yes)
 			)
 		)
@@
 					(size 1.27 1.27)
 				)
+				(hide yes)
 			)
 		)
@@
 					(size 1.27 1.27)
 				)
+				(hide yes)
 			)
 		)
@@
 					(size 1.27 1.27)
 				)
+				(hide yes)
 			)
 		)
@@
 					(size 1.27 1.27)
 				)
+				(hide yes)
 			)
 		)
@@
 					(size 1.27 1.27)
 				)
+				(hide yes)
 			)
 		)
@@
 					(size 1.27 1.27)
 				)
+				(hide yes)
 			)
 		)
@@
 					(size 1.27 1.27)
 				)
+				(hide yes)
 			)
 		)

Commit message: Changed LTC 4412 to 4417, still kinks to work out
Parts:
- Q5: renamed from Q4; footprint Package_TO_SOT_SMD:LFPAK56 -> Package_TO_SOT_SMD:TSOT-23; MANUFACTURER (none) -> Digikey; MANUFACTURER_PART_NUMBER PSMN4R0-40YS,115 -> AO3400A
- Q6: footprint Package_TO_SOT_SMD:LFPAK56 -> Package_TO_SOT_SMD:TSOT-23; MANUFACTURER (none) -> Digikey; MANUFACTURER_PART_NUMBER PSMN4R0-40YS,115 -> AO3400A
- Q7: renamed from Q5; footprint Package_TO_SOT_SMD:LFPAK56 -> Package_TO_SOT_SMD:TSOT-23; MANUFACTURER (none) -> Digikey; MANUFACTURER_PART_NUMBER PSMN4R0-40YS,115 -> AO3400A
- renumbered C37 to C33, C41 to C34, C42 to C35, C35 to C36, C40 to C37, C33 to C38, C32 to C39, C34 to C40, C45 to C41, C46 to C42, C30 to C43, C31 to C44, C39 to C45, C38 to C46, C43 to C47, C44 to C48, C36 to C49, R58 to R39, R46 to R40, R49 to R41, R54 to R42, R52 to R44, R38 to R45, R36 to R46, R39 to R47, R41 to R48, R60 to R49, R30 to R50, R48 to R51, R51 to R52, R57 to R53, R29 to R54, R37 to R55, R40 to R56, R42 to R57, R45 to R58, R31 to R59, R55 to R60, R32 to R61, R33 to R62, R34 to R63, R35 to R64, R59 to R65, R47 to R66, R50 to R67, R56 to R68, R44 to R69, R53 to R70, U12 to U10, U14 to U11, U11 to U12
