File: Sensing.kicad_sch (KiCad schematic)
At the start: 56 parts, among them Q5 Q_NMOS, Q6 Q_NMOS, Q7 Q_NMOS, U10 TPS259470ARPWR, U11 TPS259470ARPWR, U12 INA3221, U13 TPS259470ARPWR

Commit message: Efuses for this board and Battery board
Parts:
- C41: renamed from C36; footprint zLibrary:CAP_C1210C_X7R_2S_FW_KEM-M -> Capacitor_SMD:C_1206_3216Metric; MANUFACTURER_PART_NUMBER C1210C106M5R2C7186 -> AVX, 04025C104KAT2A
- C50: renamed from C45; footprint zLibrary:CAP_C1210C_X7R_2S_FW_KEM-M -> Capacitor_SMD:C_1206_3216Metric; MANUFACTURER_PART_NUMBER C1210C106M5R2C7186 -> AVX, 04025C104KAT2A
- C54: renamed from C49; footprint zLibrary:CAP_C1210C_X7R_2S_FW_KEM-M -> Capacitor_SMD:C_1206_3216Metric; MANUFACTURER_PART_NUMBER C1210C106M5R2C7186 -> AVX, 04025C104KAT2A
- renumbered C33 to C38, C34 to C39, C35 to C40, C37 to C42, C38 to C43, C39 to C44, C40 to C45, C41 to C46, C42 to C47, C43 to C48, C44 to C49, C46 to C51, C47 to C52, C48 to C53, R39 to R34, R40 to R35, R41 to R36, R42 to R37, R43 to R38, R44 to R39, R45 to R40, R46 to R41, R47 to R42, R48 to R43, R49 to R44, R50 to R45, R51 to R46, R52 to R47, R53 to R48, R54 to R49, R55 to R50, R56 to R51, R57 to R52, R58 to R53, R59 to R54, R60 to R55, R61 to R56, R62 to R57, R63 to R58, R64 to R59, R65 to R60, R66 to R61, R67 to R62, R68 to R63, R69 to R64, R70 to R65
