File: _autosave-EPS_mppt_board.kicad_pcb (KiCad board)
At the start: 6 copper layers, 90.2 x 95.9 mm, 284 parts, among them J1 Conn_01x04_Pin, J2 M80-5400642, J3 M80-5400642, J4 M80-5400642, J5 M80-5400642, J6 ESQ-126-39-G-D, J7 ESQ-126-39-G-D, Q1 SIR5607DP-T1-RE3, Q10 Q_NMOS, Q11 Q_NMOS, Q12 Q_NMOS, Q13 Q_NMOS, Q14 Q_NMOS, Q15 Q_NMOS, Q2 SIR5607DP-T1-RE3, Q3 SIR5607DP-T1-RE3, Q4 SIR5607DP-T1-RE3, Q5 Q_NMOS, Q6 Q_NMOS, Q7 Q_NMOS, Q8 Q_NMOS, Q9 Q_NMOS, U1 LTC4417HUF, U10 TPS259470ARPWR, U11 TPS259470ARPWR, U12 INA3221, U13 TPS259470ARPWR, U14 LTC3633AIUFDPBF, U15 LTC4162IUFD-LADM_PBF, U16 LTC4162IUFD-LADM_PBF, U17 LTC4162IUFD-LADM_PBF, U18 LTC4162IUFD-LADM_PBF, U2 TPS259470ARPWR, U3 TPS62177DQCR, U4 TPS3823A-33DBVR, U5 MR20H40, U6 STM32L496RGTx, U7 TCAN334GDCNT, U8 TCAN334GDCNT, U9 TCA9548AMRGER, Y1 8 MHZ Oscillator

Commit message: Started layout of the Ideal diode input (LTC4417)
I'm considering getting rid of the second 3V3 buck but will need to weigh the pros and cons a little more before commiting
Parts:
- C1, C10, C2, C3, C4, C8, C9: footprint Capacitor_SMD:C_0603_1608Metric -> Capacitor_SMD:C_0402_1005Metric
- C16, D2, JP1, Q5, Q6, R19, U4: moved to B.Cu
- C7, J1: moved to F.Cu
- moved C16 297.5 mm to (211.2, 92.6), turned to 180 degrees
- moved R19 271.5 mm to (183.2, 85.0)
- moved U4 267.0 mm to (181.2, 88.8), turned to 90 degrees
- moved D2 261.9 mm to (183.8, 91.1), turned to -90 degrees
- moved JP1 260.9 mm to (178.9, 93.7), turned to 90 degrees
- moved U3 259.3 mm to (133.6, 96.9)
- moved C9 253.2 mm to (129.2, 97.0)
- moved U2 248.2 mm to (126.7, 95.9), turned to -90 degrees
- moved R16 247.7 mm to (127.5, 98.9), turned to -90 degrees
- moved C10 238.7 mm to (125.7, 98.2), turned to -90 degrees
- moved U8 236.5 mm to (196.1, 108.3)
- moved C8 233.4 mm to (123.6, 95.5), turned to 180 degrees
- moved C24 232.6 mm to (174.2, 87.0), turned to 0 degrees
- moved C23 224.0 mm to (171.9, 95.4), turned to -90 degrees
- moved D3 222.9 mm to (168.4, 76.6), turned to -90 degrees
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Routing:
- net +3.3V: track 37.8 -> 32.4 mm
- net /MPPT IC/+Y_MPPT/VOUT: track 72.4 -> 73.9 mm
