File: STM32L4.kicad_sch (KiCad schematic)
At the start: 42 parts, among them J1 Conn_01x04_Pin, U19 LMK1C1106PWR, U20 TCAN337G, U21 TCAN337G, U5 MR20H40, U6 STM32L496RGTx, Y1 8 MHZ Oscillator

Commit message: Added Batt 1 and Batt 2 charging
Parts:
- JP2: footprint Jumper:SolderJumper-2_P1.3mm_Open_TrianglePad1.0x1.5mm -> Jumper:SolderJumper-3_P1.3mm_Open_RoundedPad1.0x1.5mm_NumberLabels
Changed lines of the file:
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@@
 			)
 		)
-		(property "Footprint" "Jumper:SolderJumper-2_P1.3mm_Open_TrianglePad1.0x1.5mm"
+		(property "Footprint" "Jumper:SolderJumper-3_P1.3mm_Open_RoundedPad1.0x1.5mm_NumberLabels"
 			(at 39.37 92.71 0)
 			(effects
